Commit message: more urdf

File: rover_description/rover.urdf (robot description, URDF)
Before this commit: robot mrover_arm, 1 links, 0 joints
Links:
- removed link chassis
- added link back_left_wheel_link; collision cylinder length=0.2 radius=0.2; visual cylinder length=0.2 radius=0.2
- added link back_right_wheel_link; collision cylinder length=0.2 radius=0.2; visual cylinder length=0.2 radius=0.2
- added link chassis_link; collision box size=0.8 0.6 0.4; visual box size=0.8 0.6 0.4
Joints:
- added joint back_left_wheel_joint: type continuous, parent chassis_link, child back_left_wheel_link, origin xyz=0.00 0.30 -0.1 rpy=1.570796 0 0, axis 0 0 1, limit effort=10000 velocity=1000
- added joint back_right_wheel_joint: type continuous, parent chassis_link, child back_right_wheel_link, origin xyz=0.00 -0.30 -0.1 rpy=1.570796 0 0, axis 0 0 1, limit effort=10000 velocity=1000

Commit message: inertial data

File: rover_description/rover.urdf (robot description, URDF)
Before this commit: robot mrover_arm, 3 links, 2 joints
Links:
- link back_left_wheel_link: mass None -> 10
- link back_right_wheel_link: mass None -> 10
- link chassis_link: mass None -> 10

Commit message: Caster wheel

File: rover_description/rover.urdf (robot description, URDF)
Before this commit: robot mrover_arm, 3 links, 2 joints
Links:
- added link caster_link, mass 10; collision cylinder length=0.2 radius=0.2; visual cylinder length=0.2 radius=0.2
Joints:
- added joint caster_joint: type continuous, parent chassis_link, child caster_link, origin xyz=0.10 0.0 -0.1 rpy=1.570796 0 0, axis 0 0 1, limit effort=10000 velocity=1000
- joint back_left_wheel_joint: origin xyz=0.00 0.30 -0.1 rpy=1.570796 0 0 -> xyz=-0.20 0.30 -0.1 rpy=1.570796 0 0
- joint back_right_wheel_joint: origin xyz=0.00 -0.30 -0.1 rpy=1.570796 0 0 -> xyz=-0.20 -0.30 -0.1 rpy=1.570796 0 0

Commit message: Change to xacro, turning works

File: rover_description/rover.urdf (robot description, URDF)
Before this commit: robot rover, 4 links, 3 joints
Links:
- removed link back_left_wheel_link
- removed link back_right_wheel_link
- removed link caster_link
- removed link chassis_link
- added link base_footprint, mass 10; visual box size=0.001 0.001 0.001
- added link base_link, mass 10; collision box size=0.16 0.16 0.01; visual box size=0.16 0.16 0.01
- added link caster_wheel, mass 10; collision sphere radius=0.0175; visual sphere radius=0.0175
- added link left_wheel, mass 10; collision cylinder length=0.005 radius=0.035; visual cylinder length=0.005 radius=0.035
- added link right_wheel, mass 10; collision cylinder length=0.005 radius=0.035; visual cylinder length=0.005 radius=0.035
Joints:
- removed joint back_left_wheel_joint
- removed joint back_right_wheel_joint
- removed joint caster_joint
- added joint base_link_joint: type fixed, parent base_footprint, child base_link, origin xyz=0 0 0.04 rpy=0 0 0
- added joint caster_wheel_joint: type continuous, parent base_link, child caster_wheel, origin xyz=-0.052 0 -0.022500000000000003 rpy=0 0 0, axis 0 1 0
- added joint left_wheel_joint: type continuous, parent base_link, child left_wheel, origin xyz=0.02 0.08700000000000001 -0.005 rpy=0 0 0, axis 0 1 0
- added joint right_wheel_joint: type continuous, parent base_link, child right_wheel, origin xyz=0.02 -0.08700000000000001 -0.005 rpy=0 0 0, axis 0 1 0

Commit message: new urdf

File: rover_description/rover.urdf (robot description, URDF)
Before this commit: robot rover, 5 links, 4 joints
Links:
- added link right_rocker_link, mass 3.0; collision box size=0.563 0.1 0.305; visual mesh filename=package://mrover/rover_description/meshes/right_rocker.stl scale=0.0254 0.0254 0.0254
- link base_link: mass 10 -> 45.0; geometry collision box size=0.563 0.6357 0.305; visual mesh filename=package://mrover/rover_description/meshes/chassis.stl scale=0.0254 0.0254 0.0254
Joints:
- added joint base_right_rocker_joint: type fixed, parent base_link, child right_rocker_link, origin xyz=0 -0.31785 0 rpy=0 0 0
- joint left_wheel_joint: origin xyz=0.02 0.08700000000000001 -0.005 rpy=0 0 0 -> xyz=0.02 0.32485 -0.005 rpy=0 0 0
- joint right_wheel_joint: origin xyz=0.02 -0.08700000000000001 -0.005 rpy=0 0 0 -> xyz=0.02 -0.32485 -0.005 rpy=0 0 0

File: rover_description/rover.xacro (robot description, xacro)
@@ -1,6 +1,7 @@
 <?xml version="1.0"?>
 <robot xmlns:xacro="http://www.ros.org/wiki/xacro" name="rover">
-  <xacro:property name="base_width" value="0.16" />
-  <xacro:property name="base_len" value="0.16" />
+  <xacro:property name="base_width" value="0.6357" />
+  <xacro:property name="base_len" value="0.563" />
+  <xacro:property name="base_height" value="0.305" />
   <xacro:property name="wheel_radius" value="0.035" />
   <xacro:property name="base_wheel_gap" value="0.007" />
@@ -10,4 +11,6 @@
   <xacro:property name="caster_wheel_mass" value="0.001" />
   <xacro:property name="caster_wheel_joint_offset" value="-0.052" />
+  <xacro:property name="mesh_scale" value="0.0254 0.0254 0.0254" />
+  <xacro:property name="PI" value="3.141592" />
   <!--Color Properties-->
   <material name="blue">
@@ -54,17 +57,38 @@
   <!--Base link-->
   <link name="base_link">
-    <xacro:box_inertia m="10" w="${base_len}" h="${base_width}" d="0.01" />
+    <xacro:box_inertia m="45.0" w="${base_len}" h="${base_width}" d="${base_height}" />
     <visual>
+      <origin rpy="0 0 0" xyz="${base_len/2.0 + 0.05} ${-base_width/2.0 + 0.05} -0.03"/>
       <geometry>
-        <box size="${base_len} ${base_width} 0.01" />
+        <mesh filename="package://mrover/rover_description/meshes/chassis.stl" scale="${mesh_scale}"/>
       </geometry>
-      <material name="black" />
+      <material name="blue" />
     </visual>
     <collision>
       <geometry>
-        <box size="${base_len} ${base_width} 0.01" />
+        <box size="${base_len} ${base_width} ${base_height}" />
       </geometry>
     </collision>
   </link>
+  <link name="right_rocker_link">
+    <xacro:box_inertia m="3.0" w="${base_len}" h="${base_width}" d="${base_height}" />
+    <visual>
+      <origin rpy="${PI/2} 0 ${PI/2}" xyz="0.13 0.17 -0.5"/>
+      <geometry>
+        <mesh filename="package://mrover/rover_description/meshes/right_rocker.stl" scale="${mesh_scale}"/>
+      </geometry>
+      <material name="red" />
+    </visual>
+    <collision>
+      <geometry>
+        <box size="${base_len} 0.1 ${base_height}" />
+      </geometry>
+    </collision>
+  </link>
+  <joint name="base_right_rocker_joint" type="fixed">
+    <origin xyz="0 ${-base_width/2.0} 0" rpy="0 0 0" />
+    <parent link="base_link" />
+    <child link="right_rocker_link" />
+  </joint>
   <!--base_link to base_footprint Joint-->
   <joint name="base_link_joint" type="fixed">

Commit message: more urdf

File: rover_description/rover.urdf (robot description, URDF)
Before this commit: robot rover, 6 links, 5 joints
Links:
- link right_rocker_link: geometry collision box size=0.733 0.05 0.505; visual mesh filename=package://mrover/rover_description/meshes/right_rocker.stl scale=0.0254 0.0254 0.0254
Joints:
- joint base_right_rocker_joint: origin xyz=0 -0.31785 0 rpy=0 0 0 -> xyz=0.01 -0.36785 -0.2 rpy=0 0 0

File: rover_description/rover.xacro (robot description, xacro)
@@ -74,5 +74,5 @@
     <xacro:box_inertia m="3.0" w="${base_len}" h="${base_width}" d="${base_height}" />
     <visual>
-      <origin rpy="${PI/2} 0 ${PI/2}" xyz="0.13 0.17 -0.5"/>
+      <origin rpy="${PI/2} 0 ${PI/2}" xyz="0.11 0.22 -0.3"/>
       <geometry>
         <mesh filename="package://mrover/rover_description/meshes/right_rocker.stl" scale="${mesh_scale}"/>
@@ -82,10 +82,10 @@
     <collision>
       <geometry>
-        <box size="${base_len} 0.1 ${base_height}" />
+        <box size="${base_len + 0.17} 0.05 ${base_height + 0.2}" />
       </geometry>
     </collision>
   </link>
   <joint name="base_right_rocker_joint" type="fixed">
-    <origin xyz="0 ${-base_width/2.0} 0" rpy="0 0 0" />
+    <origin xyz="0.01 ${-base_width/2.0 - 0.05} -0.2" rpy="0 0 0" />
     <parent link="base_link" />
     <child link="right_rocker_link" />

Commit message: urdf

File: rover_description/rover.urdf (robot description, URDF)
Before this commit: robot rover, 6 links, 5 joints
Links:
- added link left_rocker_link, mass 3.0; collision box size=0.733 0.05 0.505; visual mesh filename=package://mrover/rover_description/meshes/left_rocker.stl scale=0.0254 0.0254 0.0254
Joints:
- added joint base_left_rocker_joint: type fixed, parent base_link, child left_rocker_link, origin xyz=0.01 0.36785 -0.2 rpy=0 0 0

File: rover_description/rover.xacro (robot description, xacro)
@@ -91,4 +91,24 @@
     <child link="right_rocker_link" />
   </joint>
+  <link name="left_rocker_link">
+    <xacro:box_inertia m="3.0" w="${base_len}" h="${base_width}" d="${base_height}" />
+    <visual>
+      <origin rpy="${-PI/8} ${1.1*PI} ${-PI/7}" xyz="0.0 0.0 0.0"/>
+      <geometry>
+        <mesh filename="package://mrover/rover_description/meshes/left_rocker.stl" scale="${mesh_scale}"/>
+      </geometry>
+      <material name="white" />
+    </visual>
+    <collision>
+      <geometry>
+        <box size="${base_len + 0.17} 0.05 ${base_height + 0.2}" />
+      </geometry>
+    </collision>
+  </link>
+  <joint name="base_left_rocker_joint" type="fixed">
+    <origin xyz="0.01 ${base_width/2.0 + 0.05} -0.2" rpy="0 0 0" />
+    <parent link="base_link" />
+    <child link="left_rocker_link" />
+  </joint>
   <!--base_link to base_footprint Joint-->
   <joint name="base_link_joint" type="fixed">
