Commit message: Normalize all STL files

File: rover_description/rover.xacro (robot description, xacro)
@@ -11,5 +11,5 @@
   <xacro:property name="caster_wheel_mass" value="0.001" />
   <xacro:property name="caster_wheel_joint_offset" value="-0.052" />
-  <xacro:property name="mesh_scale" value="0.0254 0.0254 0.0254" />
+  <!-- <xacro:property name="mesh_scale" value="0.0254 0.0254 0.0254" /> -->
   <xacro:property name="PI" value="3.141592" />
   <!--Color Properties-->
@@ -59,7 +59,7 @@
     <xacro:box_inertia m="45.0" w="${base_len}" h="${base_width}" d="${base_height}" />
     <visual>
-      <origin rpy="0 0 0" xyz="${base_len/2.0 + 0.05} ${-base_width/2.0 + 0.05} -0.03"/>
+      <origin rpy="0 0 0" xyz="0 0 -0.03"/>
       <geometry>
-        <mesh filename="package://mrover/rover_description/meshes/chassis.stl" scale="${mesh_scale}"/>
+        <mesh filename="package://mrover/rover_description/meshes/chassis.stl" scale="1 1 1"/>
       </geometry>
       <material name="blue" />
@@ -74,7 +74,7 @@
     <xacro:box_inertia m="3.0" w="${base_len}" h="${base_width}" d="${base_height}" />
     <visual>
-      <origin rpy="${PI/2} 0 ${PI/2}" xyz="0.11 0.22 -0.3"/>
+      <origin rpy="0 0 0" xyz="0.0 0.0 0.0"/>
       <geometry>
-        <mesh filename="package://mrover/rover_description/meshes/right_rocker.stl" scale="${mesh_scale}"/>
+        <mesh filename="package://mrover/rover_description/meshes/right_rocker.stl" />
       </geometry>
       <material name="red" />
@@ -96,5 +96,5 @@
       <origin rpy="0.0 0.0 0.0" xyz="0.0 0.0 0.0"/>
       <geometry>
-        <mesh filename="package://mrover/rover_description/meshes/left_rocker.stl" scale="${mesh_scale}"/>
+        <mesh filename="package://mrover/rover_description/meshes/left_rocker.stl"/>
       </geometry>
       <material name="white" />

Commit message: Add bogies to xacro

File: rover_description/rover.xacro (robot description, xacro)
@@ -110,4 +110,44 @@
     <parent link="base_link" />
     <child link="left_rocker_link" />
+  </joint>
+  <link name="left_bogie_link">
+    <xacro:box_inertia m="3.0" w="${base_len}" h="${base_width}" d="${base_height}" />
+    <visual>
+      <origin rpy="0.0 0.0 0.0" xyz="0.0 0.0 0.0"/>
+      <geometry>
+        <mesh filename="package://mrover/rover_description/meshes/left_bogie.stl"/>
+      </geometry>
+      <material name="white" />
+    </visual>
+    <collision>
+      <geometry>
+        <box size="${base_len + 0.17} 0.05 ${base_height + 0.2}" />
+      </geometry>
+    </collision>
+  </link>
+  <joint name="base_left_bogie_joint" type="fixed">
+    <origin xyz="0.01 ${base_width/2.0 + 0.05} -0.2" rpy="0 0 0" />
+    <parent link="base_link" />
+    <child link="left_bogie_link" />
+  </joint>
+  <link name="right_bogie_link">
+    <xacro:box_inertia m="3.0" w="${base_len}" h="${base_width}" d="${base_height}" />
+    <visual>
+      <origin rpy="0.0 0.0 0.0" xyz="0.0 0.0 0.0"/>
+      <geometry>
+        <mesh filename="package://mrover/rover_description/meshes/right_bogie.stl"/>
+      </geometry>
+      <material name="white" />
+    </visual>
+    <collision>
+      <geometry>
+        <box size="${base_len + 0.17} 0.05 ${base_height + 0.2}" />
+      </geometry>
+    </collision>
+  </link>
+  <joint name="base_rught_bogie_joint" type="fixed">
+    <origin xyz="0.01 ${-base_width/2.0 - 0.05} -0.2" rpy="0 0 0" />
+    <parent link="base_link" />
+    <child link="right_bogie_link" />
   </joint>
   <!--base_link to base_footprint Joint-->

Commit message: updates to xacro

File: rover_description/rover.xacro (robot description, xacro)
@@ -59,5 +59,5 @@
     <xacro:box_inertia m="45.0" w="${base_len}" h="${base_width}" d="${base_height}" />
     <visual>
-      <origin rpy="0 0 0" xyz="0 0 -0.03"/>
+      <origin rpy="0 0 0" xyz="0.1 0.0 -0.1"/>
       <geometry>
         <mesh filename="package://mrover/rover_description/meshes/chassis.stl" scale="1 1 1"/>
@@ -74,5 +74,5 @@
     <xacro:box_inertia m="3.0" w="${base_len}" h="${base_width}" d="${base_height}" />
     <visual>
-      <origin rpy="0 0 0" xyz="0.0 0.0 0.0"/>
+      <origin rpy="0 0 0" xyz="0.1 0.03 0.1"/>
       <geometry>
         <mesh filename="package://mrover/rover_description/meshes/right_rocker.stl" />
@@ -94,5 +94,5 @@
     <xacro:box_inertia m="3.0" w="${base_len}" h="${base_width}" d="${base_height}" />
     <visual>
-      <origin rpy="0.0 0.0 0.0" xyz="0.0 0.0 0.0"/>
+      <origin rpy="0.0 0.0 0.0" xyz="0.1 -0.04 0.1"/>
       <geometry>
         <mesh filename="package://mrover/rover_description/meshes/left_rocker.stl"/>
@@ -114,5 +114,5 @@
     <xacro:box_inertia m="3.0" w="${base_len}" h="${base_width}" d="${base_height}" />
     <visual>
-      <origin rpy="0.0 0.0 0.0" xyz="0.0 0.0 0.0"/>
+      <origin rpy="0.0 0.0 0.0" xyz="0.0 0.0 0.04"/>
       <geometry>
         <mesh filename="package://mrover/rover_description/meshes/left_bogie.stl"/>
@@ -122,11 +122,11 @@
     <collision>
       <geometry>
-        <box size="${base_len + 0.17} 0.05 ${base_height + 0.2}" />
-      </geometry>
-    </collision>
-  </link>
-  <joint name="base_left_bogie_joint" type="fixed">
-    <origin xyz="0.01 ${base_width/2.0 + 0.05} -0.2" rpy="0 0 0" />
-    <parent link="base_link" />
+        <box size="0.32 0.05 0.2" />
+      </geometry>
+    </collision>
+  </link>
+  <joint name="left_bogie_joint" type="fixed">
+    <origin xyz="0.31 -0.01 -0.09" rpy="0 0 0" />
+    <parent link="left_rocker_link" />
     <child link="left_bogie_link" />
   </joint>

Commit message: added point cloud and image simulation

File: rover_description/rover.xacro (robot description, xacro)
@@ -1,6 +1,7 @@
 <?xml version="1.0"?>
 <robot xmlns:xacro="http://www.ros.org/wiki/xacro" name="rover">
-  <xacro:property name="base_width" value="0.16" />
-  <xacro:property name="base_len" value="0.16" />
+  <xacro:property name="base_width" value="0.6357" />
+  <xacro:property name="base_len" value="0.563" />
+  <xacro:property name="base_height" value="0.305" />
   <xacro:property name="wheel_radius" value="0.035" />
   <xacro:property name="base_wheel_gap" value="0.007" />
@@ -10,4 +11,6 @@
   <xacro:property name="caster_wheel_mass" value="0.001" />
   <xacro:property name="caster_wheel_joint_offset" value="-0.052" />
+  <!-- <xacro:property name="mesh_scale" value="0.0254 0.0254 0.0254" /> -->
+  <xacro:property name="PI" value="3.141592" />
   <!--Color Properties-->
   <material name="blue">
@@ -54,17 +57,98 @@
   <!--Base link-->
   <link name="base_link">
-    <xacro:box_inertia m="10" w="${base_len}" h="${base_width}" d="0.01" />
-    <visual>
-      <geometry>
-        <box size="${base_len} ${base_width} 0.01" />
-      </geometry>
-      <material name="black" />
-    </visual>
-    <collision>
-      <geometry>
-        <box size="${base_len} ${base_width} 0.01" />
-      </geometry>
-    </collision>
-  </link>
+    <xacro:box_inertia m="45.0" w="${base_len}" h="${base_width}" d="${base_height}" />
+    <visual>
+      <origin rpy="0 0 0" xyz="0.1 0.0 -0.1"/>
+      <geometry>
+        <mesh filename="package://mrover/rover_description/meshes/chassis.stl" scale="1 1 1"/>
+      </geometry>
+      <material name="blue" />
+    </visual>
+    <collision>
+      <geometry>
+        <box size="${base_len} ${base_width} ${base_height}" />
+      </geometry>
+    </collision>
+  </link>
+  <link name="right_rocker_link">
+    <xacro:box_inertia m="3.0" w="${base_len}" h="${base_width}" d="${base_height}" />
+    <visual>
+      <origin rpy="0 0 0" xyz="0.1 0.03 0.1"/>
+      <geometry>
+        <mesh filename="package://mrover/rover_description/meshes/right_rocker.stl" />
+      </geometry>
+      <material name="red" />
+    </visual>
+    <collision>
+      <geometry>
+        <box size="${base_len + 0.17} 0.05 ${base_height + 0.2}" />
+      </geometry>
+    </collision>
+  </link>
+  <joint name="base_right_rocker_joint" type="fixed">
+    <origin xyz="0.01 ${-base_width/2.0 - 0.05} -0.2" rpy="0 0 0" />
+    <parent link="base_link" />
+    <child link="right_rocker_link" />
+  </joint>
+  <link name="left_rocker_link">
+    <xacro:box_inertia m="3.0" w="${base_len}" h="${base_width}" d="${base_height}" />
+    <visual>
+      <origin rpy="0.0 0.0 0.0" xyz="0.1 -0.04 0.1"/>
+      <geometry>
+        <mesh filename="package://mrover/rover_description/meshes/left_rocker.stl"/>
+      </geometry>
+      <material name="white" />
+    </visual>
+    <collision>
+      <geometry>
+        <box size="${base_len + 0.17} 0.05 ${base_height + 0.2}" />
+      </geometry>
+    </collision>
+  </link>
+  <joint name="base_left_rocker_joint" type="fixed">
+    <origin xyz="0.01 ${base_width/2.0 + 0.05} -0.2" rpy="0 0 0" />
+    <parent link="base_link" />
+    <child link="left_rocker_link" />
+  </joint>
+  <link name="left_bogie_link">
+    <xacro:box_inertia m="3.0" w="${base_len}" h="${base_width}" d="${base_height}" />
+    <visual>
+      <origin rpy="0.0 0.0 0.0" xyz="0.0 0.0 0.04"/>
+      <geometry>
+        <mesh filename="package://mrover/rover_description/meshes/left_bogie.stl"/>
+      </geometry>
+      <material name="white" />
+    </visual>
+    <collision>
+      <geometry>
+        <box size="0.32 0.05 0.2" />
+      </geometry>
+    </collision>
+  </link>
+  <joint name="left_bogie_joint" type="fixed">
+    <origin xyz="0.31 -0.01 -0.09" rpy="0 0 0" />
+    <parent link="left_rocker_link" />
+    <child link="left_bogie_link" />
+  </joint>
+  <link name="right_bogie_link">
+    <xacro:box_inertia m="3.0" w="${base_len}" h="${base_width}" d="${base_height}" />
+    <visual>
+      <origin rpy="0.0 0.0 0.0" xyz="0.0 0.0 0.0"/>
+      <geometry>
+        <mesh filename="package://mrover/rover_description/meshes/right_bogie.stl"/>
+      </geometry>
+      <material name="white" />
+    </visual>
+    <collision>
+      <geometry>
+        <box size="${base_len + 0.17} 0.05 ${base_height + 0.2}" />
+      </geometry>
+    </collision>
+  </link>
+  <joint name="base_rught_bogie_joint" type="fixed">
+    <origin xyz="0.01 ${-base_width/2.0 - 0.05} -0.2" rpy="0 0 0" />
+    <parent link="base_link" />
+    <child link="right_bogie_link" />
+  </joint>
   <!--base_link to base_footprint Joint-->
   <joint name="base_link_joint" type="fixed">
@@ -125,4 +209,32 @@
     <origin xyz="${caster_wheel_joint_offset} 0 -${caster_wheel_radius+0.005}" rpy="0 0 0" />
   </joint>
+  <!--Camera Joint-->
+  <joint name="camera_joint" type="fixed">
+    <axis xyz="0 1 0" />
+    <origin xyz="0 0 0.2" rpy="0 0 0"/>
+    <parent link="base_link"/>
+    <child link="camera_link"/>
+  </joint>
+  <!-- Camera -->
+  <link name="camera_link">
+    <collision>
+      <origin xyz="0 0 0" rpy="0 0 0"/>
+      <geometry>
+    <box size="0.01 0.1 0.01"/>
+      </geometry>
+    </collision>
+    <visual>
+      <origin xyz="0 0 0" rpy="0 0 0"/>
+      <geometry>
+    <box size="0.01 0.1 0.01"/>
+      </geometry>
+      <material name="red"/>
+    </visual>
+    <inertial>
+      <mass value="1e-5" />
+      <origin xyz="0 0 0" rpy="0 0 0"/>
+      <inertia ixx="1e-6" ixy="0" ixz="0" iyy="1e-6" iyz="0" izz="1e-6" />
+    </inertial>
+  </link>
   <xacro:include filename="$(find mrover)/rover_description/rover_gazebo_plugins.xacro" />
 </robot>

File: rover_description/rover_gazebo_plugins.xacro (robot description, xacro)
@@ -55,3 +55,45 @@
         </sensor>
     </gazebo>
+    <!-- camera -->
+    <gazebo reference="camera_link">
+    <sensor name="camera_link_camera" type="depth">
+        <update_rate>20</update_rate>
+        <camera>
+        <horizontal_fov>1.919862</horizontal_fov>
+        <image>
+            <width>1920</width>
+            <height>1080</height>
+            <format>R8G8B8</format>
+        </image>
+        <clip>
+            <near>0.3</near>
+            <far>20</far>
+        </clip>
+        </camera>
+        <plugin name="camera_link_controller" filename="libgazebo_ros_openni_kinect.so">
+        <baseline>0.2</baseline>
+        <alwaysOn>true</alwaysOn>
+        <updateRate>1.0</updateRate>
+        <cameraName>camera_link_ir</cameraName>
+        <imageTopicName>/camera_link/color/image_raw</imageTopicName>
+        <cameraInfoTopicName>/camera_link/color/camera_info</cameraInfoTopicName>
+        <depthImageTopicName>/camera_link/depth/image_raw</depthImageTopicName>
+        <depthImageInfoTopicName>/camera_link/depth/camera_info</depthImageInfoTopicName>
+        <pointCloudTopicName>/camera_link/depth/points</pointCloudTopicName>
+        <frameName>camera_link</frameName>
+        <pointCloudCutoff>0.3</pointCloudCutoff>
+        <pointCloudCutoffMax>20.0</pointCloudCutoffMax>
+        <distortionK1>0.00000001</distortionK1>
+        <distortionK2>0.00000001</distortionK2>
+        <distortionK3>0.00000001</distortionK3>
+        <distortionT1>0.00000001</distortionT1>
+        <distortionT2>0.00000001</distortionT2>
+        <CxPrime>0</CxPrime>
+        <Cx>0</Cx>
+        <Cy>0</Cy>
+        <focalLength>0.00212</focalLength>
+        <hackBaseline>0</hackBaseline>
+        </plugin>
+    </sensor>
+    </gazebo>
 </robot>

Commit message: fix mesh

File: rover_description/rover.xacro (robot description, xacro)
@@ -1,7 +1,7 @@
 <?xml version="1.0"?>
 <robot xmlns:xacro="http://www.ros.org/wiki/xacro" name="rover">
-  <xacro:property name="base_width" value="0.6357" />
-  <xacro:property name="base_len" value="0.563" />
-  <xacro:property name="base_height" value="0.305" />
+  <xacro:property name="base_width" value="0.7357" />
+  <xacro:property name="base_len" value="1.0" />
+  <xacro:property name="base_height" value="0.6" />
   <xacro:property name="wheel_radius" value="0.035" />
   <xacro:property name="base_wheel_gap" value="0.007" />
@@ -59,7 +59,7 @@
     <xacro:box_inertia m="45.0" w="${base_len}" h="${base_width}" d="${base_height}" />
     <visual>
-      <origin rpy="0 0 0" xyz="0.1 0.0 -0.1"/>
+      <origin rpy="0 0 0" xyz="-0.25 0.0 0.2"/>
       <geometry>
-        <mesh filename="package://mrover/rover_description/meshes/chassis.stl" scale="1 1 1"/>
+        <mesh filename="package://mrover/rover_description/meshes/rover.stl" scale="1 1 1"/>
       </geometry>
       <material name="blue" />
@@ -71,84 +71,4 @@
     </collision>
   </link>
-  <link name="right_rocker_link">
-    <xacro:box_inertia m="3.0" w="${base_len}" h="${base_width}" d="${base_height}" />
-    <visual>
-      <origin rpy="0 0 0" xyz="0.1 0.03 0.1"/>
-      <geometry>
-        <mesh filename="package://mrover/rover_description/meshes/right_rocker.stl" />
-      </geometry>
-      <material name="red" />
-    </visual>
-    <collision>
-      <geometry>
-        <box size="${base_len + 0.17} 0.05 ${base_height + 0.2}" />
-      </geometry>
-    </collision>
-  </link>
-  <joint name="base_right_rocker_joint" type="fixed">
-    <origin xyz="0.01 ${-base_width/2.0 - 0.05} -0.2" rpy="0 0 0" />
-    <parent link="base_link" />
-    <child link="right_rocker_link" />
-  </joint>
-  <link name="left_rocker_link">
-    <xacro:box_inertia m="3.0" w="${base_len}" h="${base_width}" d="${base_height}" />
-    <visual>
-      <origin rpy="0.0 0.0 0.0" xyz="0.1 -0.04 0.1"/>
-      <geometry>
-        <mesh filename="package://mrover/rover_description/meshes/left_rocker.stl"/>
-      </geometry>
-      <material name="white" />
-    </visual>
-    <collision>
-      <geometry>
-        <box size="${base_len + 0.17} 0.05 ${base_height + 0.2}" />
-      </geometry>
-    </collision>
-  </link>
-  <joint name="base_left_rocker_joint" type="fixed">
-    <origin xyz="0.01 ${base_width/2.0 + 0.05} -0.2" rpy="0 0 0" />
-    <parent link="base_link" />
-    <child link="left_rocker_link" />
-  </joint>
-  <link name="left_bogie_link">
-    <xacro:box_inertia m="3.0" w="${base_len}" h="${base_width}" d="${base_height}" />
-    <visual>
-      <origin rpy="0.0 0.0 0.0" xyz="0.0 0.0 0.04"/>
-      <geometry>
-        <mesh filename="package://mrover/rover_description/meshes/left_bogie.stl"/>
-      </geometry>
-      <material name="white" />
-    </visual>
-    <collision>
-      <geometry>
-        <box size="0.32 0.05 0.2" />
-      </geometry>
-    </collision>
-  </link>
-  <joint name="left_bogie_joint" type="fixed">
-    <origin xyz="0.31 -0.01 -0.09" rpy="0 0 0" />
-    <parent link="left_rocker_link" />
-    <child link="left_bogie_link" />
-  </joint>
-  <link name="right_bogie_link">
-    <xacro:box_inertia m="3.0" w="${base_len}" h="${base_width}" d="${base_height}" />
-    <visual>
-      <origin rpy="0.0 0.0 0.0" xyz="0.0 0.0 0.0"/>
-      <geometry>
-        <mesh filename="package://mrover/rover_description/meshes/right_bogie.stl"/>
-      </geometry>
-      <material name="white" />
-    </visual>
-    <collision>
-      <geometry>
-        <box size="${base_len + 0.17} 0.05 ${base_height + 0.2}" />
-      </geometry>
-    </collision>
-  </link>
-  <joint name="base_rught_bogie_joint" type="fixed">
-    <origin xyz="0.01 ${-base_width/2.0 - 0.05} -0.2" rpy="0 0 0" />
-    <parent link="base_link" />
-    <child link="right_bogie_link" />
-  </joint>
   <!--base_link to base_footprint Joint-->
   <joint name="base_link_joint" type="fixed">
@@ -157,56 +77,4 @@
     <child link="base_link" />
   </joint>
-  <!--Wheel link & joint macro-->
-  <xacro:macro name="wheel" params="prefix reflect">
-    <link name="${prefix}_wheel">
-      <visual>
-        <origin xyz="0 0 0" rpy="${pi/2} 0 0" />
-        <geometry>
-          <cylinder radius="${wheel_radius}" length="0.005" />
-        </geometry>
-        <material name="red" />
-      </visual>
-      <collision>
-        <origin xyz="0 0 0" rpy="${pi/2} 0 0" />
-        <geometry>
-          <cylinder radius="${wheel_radius}" length="0.005" />
-        </geometry>
-      </collision>
-      <xacro:cylinder_inertia m="10" r="${wheel_radius}" h="0.005" />
-    </link>
-    <joint name="${prefix}_wheel_joint" type="continuous">
-      <axis xyz="0 1 0" rpy="0 0 0" />
-      <parent link="base_link" />
-      <child link="${prefix}_wheel" />
-      <origin xyz="${wheel_joint_offset} ${((base_width/2)+base_wheel_gap)*reflect} -0.005" rpy="0 0 0" />
-    </joint>
-  </xacro:macro>
-  <!--Create Left & Right Wheel links/joints-->
-  <xacro:wheel prefix="left" reflect="1" />
-  <xacro:wheel prefix="right" reflect="-1" />
-  <!--Caster Wheel Link-->
-  <link name="caster_wheel">
-    <visual>
-      <origin xyz="0 0 0" rpy="0 0 0" />
-      <geometry>
-        <sphere radius="${caster_wheel_radius}" />
-      </geometry>
-      <material name="blue" />
-    </visual>
-    <collision>
-      <origin xyz="0 0 0" rpy="0 0 0" />
-      <geometry>
-        <sphere radius="${caster_wheel_radius}" />
-      </geometry>
-    </collision>
-    <xacro:sphere_inertia m="10" r="${caster_wheel_radius}" />
-  </link>
-  <!--Caster Wheel Joint-->
-  <joint name="caster_wheel_joint" type="continuous">
-    <axis xyz="0 1 0" rpy="0 0 0" />
-    <parent link="base_link" />
-    <child link="caster_wheel" />
-    <origin xyz="${caster_wheel_joint_offset} 0 -${caster_wheel_radius+0.005}" rpy="0 0 0" />
-  </joint>
   <xacro:include filename="$(find mrover)/rover_description/rover_gazebo_plugins.xacro" />
 </robot>

Commit message: center wheels

File: rover_description/rover.xacro (robot description, xacro)
@@ -4,11 +4,7 @@
   <xacro:property name="base_len" value="1.0" />
   <xacro:property name="base_height" value="0.6" />
-  <xacro:property name="wheel_radius" value="0.035" />
-  <xacro:property name="base_wheel_gap" value="0.007" />
-  <xacro:property name="wheel_separation" value="0.15" />
-  <xacro:property name="wheel_joint_offset" value="0.02" />
-  <xacro:property name="caster_wheel_radius" value="${wheel_radius/2}" />
-  <xacro:property name="caster_wheel_mass" value="0.001" />
-  <xacro:property name="caster_wheel_joint_offset" value="-0.052" />
+  <xacro:property name="wheel_radius" value="0.13" />
+  <xacro:property name="wheel_width" value="0.1" />
+  <xacro:property name="wheel_mass" value="2" />
   <!-- <xacro:property name="mesh_scale" value="0.0254 0.0254 0.0254" /> -->
   <xacro:property name="PI" value="3.141592" />
@@ -45,14 +41,4 @@
     </inertial>
   </xacro:macro>
-  <!--Base Footprint-->
-  <link name="base_footprint">
-    <xacro:box_inertia m="10" w="0.001" h="0.001" d="0.001" />
-    <visual>
-      <origin xyz="0 0 0" rpy="0 0 0" />
-      <geometry>
-        <box size="0.001 0.001 0.001" />
-      </geometry>
-    </visual>
-  </link>
   <!--Base link-->
   <link name="base_link">
@@ -71,9 +57,45 @@
     </collision>
   </link>
-  <!--base_link to base_footprint Joint-->
-  <joint name="base_link_joint" type="fixed">
-    <origin xyz="0 0 ${wheel_radius + 0.005}" rpy="0 0 0" />
-    <parent link="base_footprint" />
-    <child link="base_link" />
+  <link name="front_left_wheel_link">
+    <xacro:cylinder_inertia m="2.0" r="${wheel_radius}" h="${wheel_width}" />
+    <visual>
+      <origin rpy="${PI/2} 0 0" xyz="0.0 0.0 0.0"/>
+      <geometry>
+        <mesh filename="package://mrover/rover_description/meshes/wheel.stl" scale="1 1 1"/>
+      </geometry>
+      <material name="red" />
+    </visual>
+    <collision>
+      <geometry>
+        <cylinder length="${wheel_width}" radius="${wheel_radius}"/>
+      </geometry>
+    </collision>
+  </link>
+  <joint name="front_left_wheel_joint" type="continuous">
+    <parent link="base_link"/>
+    <child link="front_left_wheel_link"/>
+    <origin xyz="0 ${base_width/2 + 0.06} -0.27" rpy="${-PI/2} 0 0" />
+    <axis xyz="0 0 1"/>
+  </joint>
+  <link name="front_right_wheel_link">
+    <xacro:cylinder_inertia m="2.0" r="${wheel_radius}" h="${wheel_width}" />
+    <visual>
+      <origin rpy="${PI/2} 0 0" xyz="0.0 0.0 0.0"/>
+      <geometry>
+        <mesh filename="package://mrover/rover_description/meshes/wheel.stl" scale="1 1 1"/>
+      </geometry>
+      <material name="red" />
+    </visual>
+    <collision>
+      <geometry>
+        <cylinder length="${wheel_width}" radius="${wheel_radius}"/>
+      </geometry>
+    </collision>
+  </link>
+  <joint name="front_right_wheel_joint" type="continuous">
+    <parent link="base_link"/>
+    <child link="front_right_wheel_link"/>
+    <origin xyz="0 ${-base_width/2 - 0.06} -0.27" rpy="${PI/2} 0 0" />
+    <axis xyz="0 0 1"/>
   </joint>
   <xacro:include filename="$(find mrover)/rover_description/rover_gazebo_plugins.xacro" />

File: rover_description/rover_gazebo_plugins.xacro (robot description, xacro)
@@ -8,5 +8,5 @@
             <leftJoint>left_wheel_joint</leftJoint>
             <rightJoint>right_wheel_joint</rightJoint>
-            <wheelSeparation>${wheel_separation}</wheelSeparation>
+            <wheelSeparation>${base_width}</wheelSeparation>
             <wheelDiameter>${wheel_radius * 2}</wheelDiameter>
             <torque>20</torque>
