Commit message: Attempt to use multicamera plugin

File: rover_description/rover.xacro (robot description, xacro)
@@ -137,4 +137,56 @@
     </inertial>
   </link>
+  <!-- Left Stereoscopic Camera -->
+  <joint name="left_camera_joint" type="fixed">
+    <origin xyz="0 0.05 0.2" />
+    <parent link="base_link" />
+    <child link="left_camera_link" />
+  </joint>
+  <link name="left_camera_link">
+    <collision>
+      <origin xyz="0 0 0" rpy="0 0 0" />
+      <geometry>
+        <box size="0.06 0.01 0.06" />
+      </geometry>
+    </collision>
+    <visual>
+      <origin xyz="0 0 0" rpy="0 0 0" />
+      <geometry>
+        <box size="0.06 0.01 0.06" />
+      </geometry>
+      <material name="red"/>
+    </visual>
+    <inertial>
+      <mass value="1e-5" />
+      <origin xyz="0 0 0" rpy="0 0 0" />
+      <inertia ixx="1e-6" ixy="0" ixz="0" iyy="1e-6" iyz="0" izz="1e-6" />
+    </inertial>
+  </link>
+  <!-- Right Stereoscopic Camera -->
+  <joint name="right_camera_joint" type="fixed">
+    <origin xyz="0 -0.05 0.2" />
+    <parent link="base_link" />
+    <child link="right_camera_link" />
+  </joint>
+  <link name="right_camera_link">
+    <collision>
+      <origin xyz="0 0 0" rpy="0 0 0" />
+      <geometry>
+        <box size="0.06 0.01 0.06" />
+      </geometry>
+    </collision>
+    <visual>
+      <origin xyz="0 0 0" rpy="0 0 0" />
+      <geometry>
+        <box size="0.06 0.01 0.06" />
+      </geometry>
+      <material name="red"/>
+    </visual>
+    <inertial>
+      <mass value="1e-5" />
+      <origin xyz="0 0 0" rpy="0 0 0" />
+      <inertia ixx="1e-6" ixy="0" ixz="0" iyy="1e-6" iyz="0" izz="1e-6" />
+    </inertial>
+  </link>
   <xacro:include filename="$(find mrover)/rover_description/rover_gazebo_plugins.xacro" />
   <xacro:wheel side="left" reflect="1" />

File: rover_description/rover_gazebo_plugins.xacro (robot description, xacro)
@@ -113,3 +113,143 @@
     </sensor>
   </gazebo>
+  <gazebo reference="left_camera_frame">
+    <sensor type="multicamera" name="stereo_camera">
+      <update_rate>30.0</update_rate>
+      <camera name="left">
+        <horizontal_fov>1.3962634</horizontal_fov>
+        <image>
+          <width>800</width>
+          <height>800</height>
+          <format>R8G8B8</format>
+        </image>
+        <clip>
+          <near>0.02</near>
+          <far>300</far>
+        </clip>
+        <noise>
+          <type>gaussian</type>
+          <mean>0.0</mean>
+          <stddev>0.007</stddev>
+        </noise>
+      </camera>
+      <camera name="right">
+        <pose>0 -0.07 0 0 0 0</pose>
+        <horizontal_fov>1.3962634</horizontal_fov>
+        <image>
+          <width>800</width>
+          <height>800</height>
+          <format>R8G8B8</format>
+        </image>
+        <clip>
+          <near>0.02</near>
+          <far>300</far>
+        </clip>
+        <noise>
+          <type>gaussian</type>
+          <mean>0.0</mean>
+          <stddev>0.007</stddev>
+        </noise>
+      </camera>
+      <plugin name="stereo_camera_controller" filename="libgazebo_ros_multicamera.so">
+        <alwaysOn>true</alwaysOn>
+        <updateRate>0.0</updateRate>
+        <cameraName>stereo_cam</cameraName>
+        <imageTopicName>image_raw</imageTopicName>
+        <cameraInfoTopicName>camera_info</cameraInfoTopicName>
+        <frameName>left_camera_optical_frame</frameName>
+        <rightFrameName>right_camera_optical_frame</rightFrameName>
+        <hackBaseline>0.07</hackBaseline>
+        <distortionK1>0.0</distortionK1>
+        <distortionK2>0.0</distortionK2>
+        <distortionK3>0.0</distortionK3>
+        <distortionT1>0.0</distortionT1>
+        <distortionT2>0.0</distortionT2>
+      </plugin>
+    </sensor>
+  </gazebo>
+  <!--
+  <gazebo reference="left_camera_link">
+    <sensor name="left_camera_link_camera" type="camera">
+      <update_rate>20</update_rate>
+      <camera>
+        <horizontal_fov>1.919862</horizontal_fov>
+        <image>
+          <width>640</width>
+          <height>480</height>
+          <format>R8G8B8</format>
+        </image>
+        <clip>
+          <near>0.2</near>
+          <far>20</far>
+        </clip>
+      </camera>
+      <plugin name="left_camera_controller" filename="libgazebo_ros_camera.so">
+        <alwaysOn>true</alwaysOn>
+        <updateRate>0.0</updateRate>
+        <cameraName>left</cameraName>
+        <imageTopicName>image_rect</imageTopicName>
+        <cameraInfoTopicName>camera_info</cameraInfoTopicName>
+        <frameName>base_link</frameName>
+        <hackBaseline>0.07</hackBaseline>
+        <distortionK1>0.0</distortionK1>
+        <distortionK2>0.0</distortionK2>
+        <distortionK3>0.0</distortionK3>
+        <distortionT1>0.0</distortionT1>
+        <distortionT2>0.0</distortionT2>
+      </plugin>
+    </sensor>
+  </gazebo>
+  <gazebo reference="right_camera_link">
+    <sensor name="right_camera_link_camera" type="camera">
+      <update_rate>20</update_rate>
+      <camera>
+        <horizontal_fov>1.919862</horizontal_fov>
+        <image>
+          <width>640</width>
+          <height>480</height>
+          <format>R8G8B8</format>
+        </image>
+        <clip>
+          <near>0.2</near>
+          <far>20</far>
+        </clip>
+      </camera>
+      <plugin name="right_camera_controller" filename="libgazebo_ros_camera.so">
+        <alwaysOn>true</alwaysOn>
+        <updateRate>0.0</updateRate>
+        <cameraName>right</cameraName>
+        <imageTopicName>image_rect</imageTopicName>
+        <cameraInfoTopicName>camera_info</cameraInfoTopicName>
+        <frameName>base_link</frameName>
+        <hackBaseline>0.07</hackBaseline>
+        <distortionK1>0.0</distortionK1>
+        <distortionK2>0.0</distortionK2>
+        <distortionK3>0.0</distortionK3>
+        <distortionT1>0.0</distortionT1>
+        <distortionT2>0.0</distortionT2>
+      </plugin>
+    </sensor>
+  </gazebo>
+  <gazebo>
+    <sensor name="stereo_camera" type="camera">
+      <plugin name="stereo_controller" filename="libros_stereo_camera.so">
+          <alwaysOn>true</alwaysOn>
+          <updateRate>20.0</updateRate>
+          <leftCamera>left_camera_link_camera</leftCamera>
+          <rightCamera>right_camera_link_camera</rightCamera>
+          <topicName>raw_stereo</topicName>
+          <frameName>optical_frame</frameName>
+          <CxPrime>320</CxPrime>
+          <Cx>320</Cx>
+          <Cy>240</Cy>
+          <focal_length>320</focal_length>
+          <distortion_k1>0</distortion_k1>
+          <distortion_k2>0</distortion_k2>
+          <distortion_k3>0</distortion_k3>
+          <distortion_t1>0</distortion_t1>
+          <distortion_t2>0</distortion_t2>
+          <baseline>1</baseline>
+        </plugin>
+    </sensor>
+  </gazebo> -->
 </robot>

Commit message: Formatting, update ci to use flat world

File: rover_description/rover.xacro (robot description, xacro)
@@ -1,43 +1,43 @@
 <?xml version="1.0"?>
 <robot xmlns:xacro="http://www.ros.org/wiki/xacro" name="rover">
-  <xacro:property name="base_width" value="0.7357" />
-  <xacro:property name="base_len" value="1.0" />
-  <xacro:property name="base_height" value="0.6" />
-  <xacro:property name="wheel_radius" value="0.13" />
-  <xacro:property name="wheel_width" value="0.1" />
-  <xacro:property name="wheel_mass" value="2" />
+  <xacro:property name="base_width" value="0.7357"/>
+  <xacro:property name="base_len" value="1.0"/>
+  <xacro:property name="base_height" value="0.6"/>
+  <xacro:property name="wheel_radius" value="0.13"/>
+  <xacro:property name="wheel_width" value="0.1"/>
+  <xacro:property name="wheel_mass" value="2"/>
   <!-- <xacro:property name="mesh_scale" value="0.0254 0.0254 0.0254" /> -->
-  <xacro:property name="PI" value="3.141592" />
+  <xacro:property name="PI" value="3.141592"/>
   <!--Interial macros-->
   <xacro:macro name="cylinder_inertia" params="m r h">
     <inertial>
-      <mass value="${m}" />
-      <inertia ixx="${m*(3*r*r+h*h)/12}" ixy="0" ixz="0" iyy="${m*(3*r*r+h*h)/12}" iyz="0" izz="${m*r*r/2}" />
+      <mass value="${m}"/>
+      <inertia ixx="${m*(3*r*r+h*h)/12}" ixy="0" ixz="0" iyy="${m*(3*r*r+h*h)/12}" iyz="0" izz="${m*r*r/2}"/>
     </inertial>
   </xacro:macro>
   <xacro:macro name="box_inertia" params="m w h d">
     <inertial>
-      <mass value="${m}" />
-      <inertia ixx="${m / 12.0 * (d*d + h*h)}" ixy="0.0" ixz="0.0" iyy="${m / 12.0 * (w*w + h*h)}" iyz="0.0" izz="${m / 12.0 * (w*w + d*d)}" />
+      <mass value="${m}"/>
+      <inertia ixx="${m / 12.0 * (d*d + h*h)}" ixy="0.0" ixz="0.0" iyy="${m / 12.0 * (w*w + h*h)}" iyz="0.0" izz="${m / 12.0 * (w*w + d*d)}"/>
     </inertial>
   </xacro:macro>
   <xacro:macro name="sphere_inertia" params="m r">
     <inertial>
-      <mass value="${m}" />
-      <inertia ixx="${2.0*m*(r*r)/5.0}" ixy="0.0" ixz="0.0" iyy="${2.0*m*(r*r)/5.0}" iyz="0.0" izz="${2.0*m*(r*r)/5.0}" />
+      <mass value="${m}"/>
+      <inertia ixx="${2.0*m*(r*r)/5.0}" ixy="0.0" ixz="0.0" iyy="${2.0*m*(r*r)/5.0}" iyz="0.0" izz="${2.0*m*(r*r)/5.0}"/>
     </inertial>
   </xacro:macro>
   <!--Base link-->
   <link name="base_link">
-    <xacro:box_inertia m="3.0" w="${base_len}" h="${base_width}" d="${base_height}" />
+    <xacro:box_inertia m="3.0" w="${base_len}" h="${base_width}" d="${base_height}"/>
     <visual>
-      <origin rpy="0 0 0" xyz="-0.25 0.0 0.2" />
+      <origin rpy="0 0 0" xyz="-0.25 0.0 0.2"/>
       <geometry>
-        <mesh filename="package://mrover/rover_description/meshes/rover.dae" scale="1 1 1" />
+        <mesh filename="package://mrover/rover_description/meshes/rover.dae" scale="1 1 1"/>
       </geometry>
     </visual>
     <collision>
       <geometry>
-        <box size="${base_len} ${base_width} ${base_height}" />
+        <box size="${base_len} ${base_width} ${base_height}"/>
       </geometry>
     </collision>
@@ -45,150 +45,148 @@
   <xacro:macro name="wheel" params="side reflect">
     <link name="front_${side}_wheel_link">
-      <xacro:sphere_inertia m="${wheel_mass}" r="${wheel_radius}" />
+      <xacro:sphere_inertia m="${wheel_mass}" r="${wheel_radius}"/>
       <visual>
-        <origin rpy="${reflect * PI/2} 0 0" xyz="0.0 0.0 0.0" />
+        <origin rpy="${reflect * PI/2} 0 0" xyz="0.0 0.0 0.0"/>
         <geometry>
-          <mesh filename="package://mrover/rover_description/meshes/wheel.dae" scale="1 1 1" />
+          <mesh filename="package://mrover/rover_description/meshes/wheel.dae" scale="1 1 1"/>
         </geometry>
       </visual>
       <collision>
         <geometry>
-          <sphere radius="${wheel_radius}" />
+          <sphere radius="${wheel_radius}"/>
         </geometry>
       </collision>
     </link>
     <link name="center_${side}_wheel_link">
-      <xacro:cylinder_inertia m="${wheel_mass}" r="${wheel_radius}" h="${wheel_width}" />
+      <xacro:cylinder_inertia m="${wheel_mass}" r="${wheel_radius}" h="${wheel_width}"/>
       <visual>
-        <origin rpy="${reflect * PI/2} 0 0" xyz="0.0 0.0 0.0" />
+        <origin rpy="${reflect * PI/2} 0 0" xyz="0.0 0.0 0.0"/>
         <geometry>
-          <mesh filename="package://mrover/rover_description/meshes/wheel.dae" scale="1 1 1" />
+          <mesh filename="package://mrover/rover_description/meshes/wheel.dae" scale="1 1 1"/>
         </geometry>
       </visual>
       <collision>
         <geometry>
-          <cylinder length="${wheel_width}" radius="${wheel_radius}" />
+          <cylinder length="${wheel_width}" radius="${wheel_radius}"/>
         </geometry>
       </collision>
     </link>
     <link name="back_${side}_wheel_link">
-      <xacro:sphere_inertia m="${wheel_mass}" r="${wheel_radius}" />
+      <xacro:sphere_inertia m="${wheel_mass}" r="${wheel_radius}"/>
       <visual>
-        <origin rpy="${reflect * PI/2} 0 0" xyz="0.0 0.0 0.0" />
+        <origin rpy="${reflect * PI/2} 0 0" xyz="0.0 0.0 0.0"/>
         <geometry>
-          <mesh filename="package://mrover/rover_description/meshes/wheel.dae" scale="1 1 1" />
+          <mesh filename="package://mrover/rover_description/meshes/wheel.dae" scale="1 1 1"/>
         </geometry>
       </visual>
       <collision>
         <geometry>
-          <sphere radius="${wheel_radius}" />
+          <sphere radius="${wheel_radius}"/>
         </geometry>
       </collision>
     </link>
     <joint name="front_${side}_wheel_joint" type="continuous">
-      <parent link="base_link" />
-      <child link="front_${side}_wheel_link" />
-      <origin xyz="0.42 ${reflect * (base_width/2 + 0.06)} -0.27" rpy="${-PI/2} 0 0" />
-      <axis xyz="0 0 1" />
+      <parent link="base_link"/>
+      <child link="front_${side}_wheel_link"/>
+      <origin xyz="0.42 ${reflect * (base_width/2 + 0.06)} -0.27" rpy="${-PI/2} 0 0"/>
+      <axis xyz="0 0 1"/>
     </joint>
     <joint name="center_${side}_wheel_joint" type="continuous">
-      <parent link="base_link" />
-      <child link="center_${side}_wheel_link" />
-      <origin xyz="0 ${reflect * (base_width/2 + 0.06)} -0.27" rpy="${-PI/2} 0 0" />
-      <axis xyz="0 0 1" />
+      <parent link="base_link"/>
+      <child link="center_${side}_wheel_link"/>
+      <origin xyz="0 ${reflect * (base_width/2 + 0.06)} -0.27" rpy="${-PI/2} 0 0"/>
+      <axis xyz="0 0 1"/>
     </joint>
     <joint name="back_${side}_wheel_joint" type="continuous">
-      <parent link="base_link" />
-      <child link="back_${side}_wheel_link" />
-      <origin xyz="-0.42 ${reflect*(base_width/2 + 0.06)} -0.27" rpy="${-PI/2} 0 0" />
-      <axis xyz="0 0 1" />
+      <parent link="base_link"/>
+      <child link="back_${side}_wheel_link"/>
+      <origin xyz="-0.42 ${reflect*(base_width/2 + 0.06)} -0.27" rpy="${-PI/2} 0 0"/>
+      <axis xyz="0 0 1"/>
     </joint>
   </xacro:macro>
   <!-- IMU -->
   <joint name="imu_joint" type="fixed">
-    <origin xyz="0 0 0.2" />
-    <parent link="base_link" />
-    <child link="imu_link" />
+    <origin xyz="0 0 0.2"/>
+    <parent link="base_link"/>
+    <child link="imu_link"/>
   </joint>
   <link name="imu_link"></link>
   <!-- Camera -->
   <joint name="camera_joint" type="fixed">
-    <origin xyz="0 0 0.2" />
-    <parent link="base_link" />
-    <child link="camera_link" />
+    <origin xyz="0 0 0.2"/>
+    <parent link="base_link"/>
+    <child link="camera_link"/>
   </joint>
   <link name="camera_link">
     <collision>
-      <origin xyz="0 0 0" rpy="0 0 0" />
+      <origin xyz="0 0 0" rpy="0 0 0"/>
       <geometry>
-        <box size="0.01 0.1 0.01" />
+        <box size="0.01 0.1 0.01"/>
       </geometry>
     </collision>
     <visual>
-      <origin xyz="0 0 0" rpy="0 0 0" />
+      <origin xyz="0 0 0" rpy="0 0 0"/>
       <geometry>
-        <mesh filename="package://mrover/rover_description/meshes/ZED2i.dae" scale="1 1 1" />
+        <mesh filename="package://mrover/rover_description/meshes/ZED2i.dae" scale="1 1 1"/>
       </geometry>
     </visual>
     <inertial>
-      <mass value="1e-5" />
-      <origin xyz="0 0 0" rpy="0 0 0" />
-      <inertia ixx="1e-6" ixy="0" ixz="0" iyy="1e-6" iyz="0" izz="1e-6" />
+      <mass value="1e-5"/>
+      <origin xyz="0 0 0" rpy="0 0 0"/>
+      <inertia ixx="1e-6" ixy="0" ixz="0" iyy="1e-6" iyz="0" izz="1e-6"/>
     </inertial>
   </link>
   <!-- Left Stereoscopic Camera -->
   <joint name="left_camera_joint" type="fixed">
-    <origin xyz="0 0.05 0.2" />
-    <parent link="base_link" />
-    <child link="left_camera_link" />
+    <origin xyz="0 0.05 0.2"/>
+    <parent link="base_link"/>
+    <child link="left_camera_link"/>
   </joint>
   <link name="left_camera_link">
     <collision>
-      <origin xyz="0 0 0" rpy="0 0 0" />
+      <origin xyz="0 0 0" rpy="0 0 0"/>
       <geometry>
-        <box size="0.06 0.01 0.06" />
+        <box size="0.06 0.01 0.06"/>
       </geometry>
     </collision>
     <visual>
-      <origin xyz="0 0 0" rpy="0 0 0" />
+      <origin xyz="0 0 0" rpy="0 0 0"/>
       <geometry>
-        <box size="0.06 0.01 0.06" />
+        <box size="0.06 0.01 0.06"/>
       </geometry>
-      <material name="red"/>
     </visual>
     <inertial>
-      <mass value="1e-5" />
-      <origin xyz="0 0 0" rpy="0 0 0" />
-      <inertia ixx="1e-6" ixy="0" ixz="0" iyy="1e-6" iyz="0" izz="1e-6" />
+      <mass value="1e-5"/>
+      <origin xyz="0 0 0" rpy="0 0 0"/>
+      <inertia ixx="1e-6" ixy="0" ixz="0" iyy="1e-6" iyz="0" izz="1e-6"/>
     </inertial>
   </link>
   <!-- Right Stereoscopic Camera -->
   <joint name="right_camera_joint" type="fixed">
-    <origin xyz="0 -0.05 0.2" />
-    <parent link="base_link" />
-    <child link="right_camera_link" />
+    <origin xyz="0 -0.05 0.2"/>
+    <parent link="base_link"/>
+    <child link="right_camera_link"/>
   </joint>
   <link name="right_camera_link">
     <collision>
-      <origin xyz="0 0 0" rpy="0 0 0" />
+      <origin xyz="0 0 0" rpy="0 0 0"/>
       <geometry>
-        <box size="0.06 0.01 0.06" />
+        <box size="0.06 0.01 0.06"/>
       </geometry>
     </collision>
     <visual>
-      <origin xyz="0 0 0" rpy="0 0 0" />
+      <origin xyz="0 0 0" rpy="0 0 0"/>
       <geometry>
-        <box size="0.06 0.01 0.06" />
+        <box size="0.06 0.01 0.06"/>
       </geometry>
-      <material name="red"/>
     </visual>
     <inertial>
-      <mass value="1e-5" />
-      <origin xyz="0 0 0" rpy="0 0 0" />
-      <inertia ixx="1e-6" ixy="0" ixz="0" iyy="1e-6" iyz="0" izz="1e-6" />
+      <mass value="1e-5"/>
+      <origin xyz="0 0 0" rpy="0 0 0"/>
+      <inertia ixx="1e-6" ixy="0" ixz="0" iyy="1e-6" iyz="0" izz="1e-6"/>
     </inertial>
   </link>
-  <xacro:include filename="$(find mrover)/rover_description/rover_gazebo_plugins.xacro" />
-  <xacro:wheel side="left" reflect="1" />
-  <xacro:wheel side="right" reflect="-1" />
+  <xacro:include filename="$(find mrover)/rover_description/rover_gazebo_plugins.xacro"/>
+  <xacro:wheel side="left" reflect="1"/>
+  <xacro:wheel side="right" reflect="-1"/>
 </robot>
