Commit message: Add visual odometry to simulator (#401)
* RTAB map and zed ros wrapper visual odom

* started sensor fusion using robot_localization

* test vis odom sdk

* Attempt to use multicamera plugin

* rtabmap in sim working

* Add ERC terrain model

* Work on launch files

* Actually use argument

* Enable odom and change arg format

* Delete test files

* Update sim

* Cleanup

* Style

* Formatting, update ci to use flat world

* moved to auton launch

* Remove

* Re-remove meshes_orig

* Move vis odom launch to auton sim

---------

Co-authored-by: umroverPerception <umroverPerception@gmail.com>
Co-authored-by: qhdwight <qhdwight@gmail.com>
Co-authored-by: Riley Bridges <rlybrdgs@gmail.com>

File: rover_description/rover.xacro (robot description, xacro)
@@ -1,43 +1,43 @@
 <?xml version="1.0"?>
 <robot xmlns:xacro="http://www.ros.org/wiki/xacro" name="rover">
-  <xacro:property name="base_width" value="0.7357" />
-  <xacro:property name="base_len" value="1.0" />
-  <xacro:property name="base_height" value="0.6" />
-  <xacro:property name="wheel_radius" value="0.13" />
-  <xacro:property name="wheel_width" value="0.1" />
-  <xacro:property name="wheel_mass" value="2" />
+  <xacro:property name="base_width" value="0.7357"/>
+  <xacro:property name="base_len" value="1.0"/>
+  <xacro:property name="base_height" value="0.6"/>
+  <xacro:property name="wheel_radius" value="0.13"/>
+  <xacro:property name="wheel_width" value="0.1"/>
+  <xacro:property name="wheel_mass" value="2"/>
   <!-- <xacro:property name="mesh_scale" value="0.0254 0.0254 0.0254" /> -->
-  <xacro:property name="PI" value="3.141592" />
+  <xacro:property name="PI" value="3.141592"/>
   <!--Interial macros-->
   <xacro:macro name="cylinder_inertia" params="m r h">
     <inertial>
-      <mass value="${m}" />
-      <inertia ixx="${m*(3*r*r+h*h)/12}" ixy="0" ixz="0" iyy="${m*(3*r*r+h*h)/12}" iyz="0" izz="${m*r*r/2}" />
+      <mass value="${m}"/>
+      <inertia ixx="${m*(3*r*r+h*h)/12}" ixy="0" ixz="0" iyy="${m*(3*r*r+h*h)/12}" iyz="0" izz="${m*r*r/2}"/>
     </inertial>
   </xacro:macro>
   <xacro:macro name="box_inertia" params="m w h d">
     <inertial>
-      <mass value="${m}" />
-      <inertia ixx="${m / 12.0 * (d*d + h*h)}" ixy="0.0" ixz="0.0" iyy="${m / 12.0 * (w*w + h*h)}" iyz="0.0" izz="${m / 12.0 * (w*w + d*d)}" />
+      <mass value="${m}"/>
+      <inertia ixx="${m / 12.0 * (d*d + h*h)}" ixy="0.0" ixz="0.0" iyy="${m / 12.0 * (w*w + h*h)}" iyz="0.0" izz="${m / 12.0 * (w*w + d*d)}"/>
     </inertial>
   </xacro:macro>
   <xacro:macro name="sphere_inertia" params="m r">
     <inertial>
-      <mass value="${m}" />
-      <inertia ixx="${2.0*m*(r*r)/5.0}" ixy="0.0" ixz="0.0" iyy="${2.0*m*(r*r)/5.0}" iyz="0.0" izz="${2.0*m*(r*r)/5.0}" />
+      <mass value="${m}"/>
+      <inertia ixx="${2.0*m*(r*r)/5.0}" ixy="0.0" ixz="0.0" iyy="${2.0*m*(r*r)/5.0}" iyz="0.0" izz="${2.0*m*(r*r)/5.0}"/>
     </inertial>
   </xacro:macro>
   <!--Base link-->
   <link name="base_link">
-    <xacro:box_inertia m="3.0" w="${base_len}" h="${base_width}" d="${base_height}" />
+    <xacro:box_inertia m="3.0" w="${base_len}" h="${base_width}" d="${base_height}"/>
     <visual>
-      <origin rpy="0 0 0" xyz="-0.25 0.0 0.2" />
+      <origin rpy="0 0 0" xyz="-0.25 0.0 0.2"/>
       <geometry>
-        <mesh filename="package://mrover/rover_description/meshes/rover.dae" scale="1 1 1" />
+        <mesh filename="package://mrover/rover_description/meshes/rover.dae" scale="1 1 1"/>
       </geometry>
     </visual>
     <collision>
       <geometry>
-        <box size="${base_len} ${base_width} ${base_height}" />
+        <box size="${base_len} ${base_width} ${base_height}"/>
       </geometry>
     </collision>
@@ -45,98 +45,148 @@
   <xacro:macro name="wheel" params="side reflect">
     <link name="front_${side}_wheel_link">
-      <xacro:sphere_inertia m="${wheel_mass}" r="${wheel_radius}" />
+      <xacro:sphere_inertia m="${wheel_mass}" r="${wheel_radius}"/>
       <visual>
-        <origin rpy="${reflect * PI/2} 0 0" xyz="0.0 0.0 0.0" />
+        <origin rpy="${reflect * PI/2} 0 0" xyz="0.0 0.0 0.0"/>
         <geometry>
-          <mesh filename="package://mrover/rover_description/meshes/wheel.dae" scale="1 1 1" />
+          <mesh filename="package://mrover/rover_description/meshes/wheel.dae" scale="1 1 1"/>
         </geometry>
       </visual>
       <collision>
         <geometry>
-          <sphere radius="${wheel_radius}" />
+          <sphere radius="${wheel_radius}"/>
         </geometry>
       </collision>
     </link>
     <link name="center_${side}_wheel_link">
-      <xacro:cylinder_inertia m="${wheel_mass}" r="${wheel_radius}" h="${wheel_width}" />
+      <xacro:cylinder_inertia m="${wheel_mass}" r="${wheel_radius}" h="${wheel_width}"/>
       <visual>
-        <origin rpy="${reflect * PI/2} 0 0" xyz="0.0 0.0 0.0" />
+        <origin rpy="${reflect * PI/2} 0 0" xyz="0.0 0.0 0.0"/>
         <geometry>
-          <mesh filename="package://mrover/rover_description/meshes/wheel.dae" scale="1 1 1" />
+          <mesh filename="package://mrover/rover_description/meshes/wheel.dae" scale="1 1 1"/>
         </geometry>
       </visual>
       <collision>
         <geometry>
-          <cylinder length="${wheel_width}" radius="${wheel_radius}" />
+          <cylinder length="${wheel_width}" radius="${wheel_radius}"/>
         </geometry>
       </collision>
     </link>
     <link name="back_${side}_wheel_link">
-      <xacro:sphere_inertia m="${wheel_mass}" r="${wheel_radius}" />
+      <xacro:sphere_inertia m="${wheel_mass}" r="${wheel_radius}"/>
       <visual>
-        <origin rpy="${reflect * PI/2} 0 0" xyz="0.0 0.0 0.0" />
+        <origin rpy="${reflect * PI/2} 0 0" xyz="0.0 0.0 0.0"/>
         <geometry>
-          <mesh filename="package://mrover/rover_description/meshes/wheel.dae" scale="1 1 1" />
+          <mesh filename="package://mrover/rover_description/meshes/wheel.dae" scale="1 1 1"/>
         </geometry>
       </visual>
       <collision>
         <geometry>
-          <sphere radius="${wheel_radius}" />
+          <sphere radius="${wheel_radius}"/>
         </geometry>
       </collision>
     </link>
     <joint name="front_${side}_wheel_joint" type="continuous">
-      <parent link="base_link" />
-      <child link="front_${side}_wheel_link" />
-      <origin xyz="0.42 ${reflect * (base_width/2 + 0.06)} -0.27" rpy="${-PI/2} 0 0" />
-      <axis xyz="0 0 1" />
+      <parent link="base_link"/>
+      <child link="front_${side}_wheel_link"/>
+      <origin xyz="0.42 ${reflect * (base_width/2 + 0.06)} -0.27" rpy="${-PI/2} 0 0"/>
+      <axis xyz="0 0 1"/>
     </joint>
     <joint name="center_${side}_wheel_joint" type="continuous">
-      <parent link="base_link" />
-      <child link="center_${side}_wheel_link" />
-      <origin xyz="0 ${reflect * (base_width/2 + 0.06)} -0.27" rpy="${-PI/2} 0 0" />
-      <axis xyz="0 0 1" />
+      <parent link="base_link"/>
+      <child link="center_${side}_wheel_link"/>
+      <origin xyz="0 ${reflect * (base_width/2 + 0.06)} -0.27" rpy="${-PI/2} 0 0"/>
+      <axis xyz="0 0 1"/>
     </joint>
     <joint name="back_${side}_wheel_joint" type="continuous">
-      <parent link="base_link" />
-      <child link="back_${side}_wheel_link" />
-      <origin xyz="-0.42 ${reflect*(base_width/2 + 0.06)} -0.27" rpy="${-PI/2} 0 0" />
-      <axis xyz="0 0 1" />
+      <parent link="base_link"/>
+      <child link="back_${side}_wheel_link"/>
+      <origin xyz="-0.42 ${reflect*(base_width/2 + 0.06)} -0.27" rpy="${-PI/2} 0 0"/>
+      <axis xyz="0 0 1"/>
     </joint>
   </xacro:macro>
   <!-- IMU -->
   <joint name="imu_joint" type="fixed">
-    <origin xyz="0 0 0.2" />
-    <parent link="base_link" />
-    <child link="imu_link" />
+    <origin xyz="0 0 0.2"/>
+    <parent link="base_link"/>
+    <child link="imu_link"/>
   </joint>
   <link name="imu_link"></link>
   <!-- Camera -->
   <joint name="camera_joint" type="fixed">
-    <origin xyz="0 0 0.2" />
-    <parent link="base_link" />
-    <child link="camera_link" />
+    <origin xyz="0 0 0.2"/>
+    <parent link="base_link"/>
+    <child link="camera_link"/>
   </joint>
   <link name="camera_link">
     <collision>
-      <origin xyz="0 0 0" rpy="0 0 0" />
+      <origin xyz="0 0 0" rpy="0 0 0"/>
       <geometry>
-        <box size="0.01 0.1 0.01" />
+        <box size="0.01 0.1 0.01"/>
       </geometry>
     </collision>
     <visual>
-      <origin xyz="0 0 0" rpy="0 0 0" />
+      <origin xyz="0 0 0" rpy="0 0 0"/>
       <geometry>
-        <mesh filename="package://mrover/rover_description/meshes/ZED2i.dae" scale="1 1 1" />
+        <mesh filename="package://mrover/rover_description/meshes/ZED2i.dae" scale="1 1 1"/>
       </geometry>
     </visual>
     <inertial>
-      <mass value="1e-5" />
-      <origin xyz="0 0 0" rpy="0 0 0" />
-      <inertia ixx="1e-6" ixy="0" ixz="0" iyy="1e-6" iyz="0" izz="1e-6" />
+      <mass value="1e-5"/>
+      <origin xyz="0 0 0" rpy="0 0 0"/>
+      <inertia ixx="1e-6" ixy="0" ixz="0" iyy="1e-6" iyz="0" izz="1e-6"/>
     </inertial>
   </link>
-  <xacro:include filename="$(find mrover)/rover_description/rover_gazebo_plugins.xacro" />
-  <xacro:wheel side="left" reflect="1" />
-  <xacro:wheel side="right" reflect="-1" />
+  <!-- Left Stereoscopic Camera -->
+  <joint name="left_camera_joint" type="fixed">
+    <origin xyz="0 0.05 0.2"/>
+    <parent link="base_link"/>
+    <child link="left_camera_link"/>
+  </joint>
+  <link name="left_camera_link">
+    <collision>
+      <origin xyz="0 0 0" rpy="0 0 0"/>
+      <geometry>
+        <box size="0.06 0.01 0.06"/>
+      </geometry>
+    </collision>
+    <visual>
+      <origin xyz="0 0 0" rpy="0 0 0"/>
+      <geometry>
+        <box size="0.06 0.01 0.06"/>
+      </geometry>
+    </visual>
+    <inertial>
+      <mass value="1e-5"/>
+      <origin xyz="0 0 0" rpy="0 0 0"/>
+      <inertia ixx="1e-6" ixy="0" ixz="0" iyy="1e-6" iyz="0" izz="1e-6"/>
+    </inertial>
+  </link>
+  <!-- Right Stereoscopic Camera -->
+  <joint name="right_camera_joint" type="fixed">
+    <origin xyz="0 -0.05 0.2"/>
+    <parent link="base_link"/>
+    <child link="right_camera_link"/>
+  </joint>
+  <link name="right_camera_link">
+    <collision>
+      <origin xyz="0 0 0" rpy="0 0 0"/>
+      <geometry>
+        <box size="0.06 0.01 0.06"/>
+      </geometry>
+    </collision>
+    <visual>
+      <origin xyz="0 0 0" rpy="0 0 0"/>
+      <geometry>
+        <box size="0.06 0.01 0.06"/>
+      </geometry>
+    </visual>
+    <inertial>
+      <mass value="1e-5"/>
+      <origin xyz="0 0 0" rpy="0 0 0"/>
+      <inertia ixx="1e-6" ixy="0" ixz="0" iyy="1e-6" iyz="0" izz="1e-6"/>
+    </inertial>
+  </link>
+  <xacro:include filename="$(find mrover)/rover_description/rover_gazebo_plugins.xacro"/>
+  <xacro:wheel side="left" reflect="1"/>
+  <xacro:wheel side="right" reflect="-1"/>
 </robot>

File: rover_description/rover_gazebo_plugins.xacro (robot description, xacro)
@@ -116,3 +116,65 @@
     </sensor>
   </gazebo>
+  <gazebo reference="left_camera_link">
+    <sensor name="left_camera_link_camera" type="camera">
+      <update_rate>20</update_rate>
+      <camera>
+        <horizontal_fov>1.919862</horizontal_fov>
+        <image>
+          <width>640</width>
+          <height>480</height>
+          <format>R8G8B8</format>
+        </image>
+        <clip>
+          <near>0.2</near>
+          <far>20</far>
+        </clip>
+      </camera>
+      <plugin name="left_camera_controller" filename="libgazebo_ros_camera.so">
+        <alwaysOn>true</alwaysOn>
+        <updateRate>20</updateRate>
+        <cameraName>left</cameraName>
+        <imageTopicName>image_rect</imageTopicName>
+        <cameraInfoTopicName>camera_info</cameraInfoTopicName>
+        <frameName>base_link</frameName>
+        <hackBaseline>0.02</hackBaseline>
+        <distortionK1>0.0</distortionK1>
+        <distortionK2>0.0</distortionK2>
+        <distortionK3>0.0</distortionK3>
+        <distortionT1>0.0</distortionT1>
+        <distortionT2>0.0</distortionT2>
+      </plugin>
+    </sensor>
+  </gazebo>
+  <gazebo reference="right_camera_link">
+    <sensor name="right_camera_link_camera" type="camera">
+      <update_rate>20</update_rate>
+      <camera>
+        <horizontal_fov>1.919862</horizontal_fov>
+        <image>
+          <width>640</width>
+          <height>480</height>
+          <format>R8G8B8</format>
+        </image>
+        <clip>
+          <near>0.2</near>
+          <far>20</far>
+        </clip>
+      </camera>
+      <plugin name="right_camera_controller" filename="libgazebo_ros_camera.so">
+        <alwaysOn>true</alwaysOn>
+        <updateRate>20</updateRate>
+        <cameraName>right</cameraName>
+        <imageTopicName>image_rect</imageTopicName>
+        <cameraInfoTopicName>camera_info</cameraInfoTopicName>
+        <frameName>base_link</frameName>
+        <hackBaseline>0.07</hackBaseline>
+        <distortionK1>0.0</distortionK1>
+        <distortionK2>0.0</distortionK2>
+        <distortionK3>0.0</distortionK3>
+        <distortionT1>0.0</distortionT1>
+        <distortionT2>0.0</distortionT2>
+      </plugin>
+    </sensor>
+  </gazebo>
 </robot>

Commit message: Fix perception im sim (topic mismatch oops). rtabmap also changed their nodelet name

File: rover_description/rover.xacro (robot description, xacro)
@@ -128,5 +128,5 @@
       <origin xyz="0 0 0" rpy="0 0 0"/>
       <geometry>
-        <mesh filename="package://mrover/rover_description/meshes/ZED2i.dae" scale="1 1 1"/>
+        <mesh filename="package://mrover/rover_description/meshes/zed2i.dae" scale="1 1 1"/>
       </geometry>
     </visual>

File: rover_description/rover_gazebo_plugins.xacro (robot description, xacro)
@@ -94,10 +94,10 @@
         <alwaysOn>true</alwaysOn>
         <updateRate>1.0</updateRate>
-        <cameraName>camera</cameraName>
-        <imageTopicName>color/image_raw</imageTopicName>
-        <cameraInfoTopicName>color/camera_info</cameraInfoTopicName>
-        <depthImageTopicName>depth/image_raw</depthImageTopicName>
-        <depthImageInfoTopicName>depth/camera_info</depthImageInfoTopicName>
-        <pointCloudTopicName>depth/points</pointCloudTopicName>
+        <cameraName>camera/left</cameraName>
+        <imageTopicName>image</imageTopicName>
+        <cameraInfoTopicName>camera_info</cameraInfoTopicName>
+        <depthImageTopicName>depth_image</depthImageTopicName>
+        <depthImageInfoTopicName>camera_info</depthImageInfoTopicName>
+        <pointCloudTopicName>points</pointCloudTopicName>
         <frameName>camera_link</frameName>
         <pointCloudCutoff>0.3</pointCloudCutoff>
@@ -134,6 +134,6 @@
         <alwaysOn>true</alwaysOn>
         <updateRate>20</updateRate>
-        <cameraName>left</cameraName>
-        <imageTopicName>image_rect</imageTopicName>
+        <cameraName>camera/left</cameraName>
+        <imageTopicName>image</imageTopicName>
         <cameraInfoTopicName>camera_info</cameraInfoTopicName>
         <frameName>base_link</frameName>
@@ -165,6 +165,6 @@
         <alwaysOn>true</alwaysOn>
         <updateRate>20</updateRate>
-        <cameraName>right</cameraName>
-        <imageTopicName>image_rect</imageTopicName>
+        <cameraName>camera/right</cameraName>
+        <imageTopicName>image</imageTopicName>
         <cameraInfoTopicName>camera_info</cameraInfoTopicName>
         <frameName>base_link</frameName>
