Commit message: use xacro in launch file

File: deprecated/rover.urdf (robot description, URDF)
Before this commit: robot rover, 7 links, 6 joints
Links:
- removed link left_rocker_link
- removed link right_rocker_link
- link base_link: mass 45.0 -> 10; geometry collision box size=0.16 0.16 0.01; visual box size=0.16 0.16 0.01
Joints:
- removed joint base_left_rocker_joint
- removed joint base_right_rocker_joint
- joint left_wheel_joint: origin xyz=0.02 0.32485 -0.005 rpy=0 0 0 -> xyz=0.02 0.08700000000000001 -0.005 rpy=0 0 0
- joint right_wheel_joint: origin xyz=0.02 -0.32485 -0.005 rpy=0 0 0 -> xyz=0.02 -0.08700000000000001 -0.005 rpy=0 0 0

File: deprecated/rover.xacro (robot description, xacro)
@@ -1,7 +1,6 @@
 <?xml version="1.0"?>
 <robot xmlns:xacro="http://www.ros.org/wiki/xacro" name="rover">
-  <xacro:property name="base_width" value="0.6357" />
-  <xacro:property name="base_len" value="0.563" />
-  <xacro:property name="base_height" value="0.305" />
+  <xacro:property name="base_width" value="0.16" />
+  <xacro:property name="base_len" value="0.16" />
   <xacro:property name="wheel_radius" value="0.035" />
   <xacro:property name="base_wheel_gap" value="0.007" />
@@ -11,6 +10,4 @@
   <xacro:property name="caster_wheel_mass" value="0.001" />
   <xacro:property name="caster_wheel_joint_offset" value="-0.052" />
-  <xacro:property name="mesh_scale" value="0.0254 0.0254 0.0254" />
-  <xacro:property name="PI" value="3.141592" />
   <!--Color Properties-->
   <material name="blue">
@@ -57,58 +54,17 @@
   <!--Base link-->
   <link name="base_link">
-    <xacro:box_inertia m="45.0" w="${base_len}" h="${base_width}" d="${base_height}" />
+    <xacro:box_inertia m="10" w="${base_len}" h="${base_width}" d="0.01" />
     <visual>
-      <origin rpy="0 0 0" xyz="${base_len/2.0 + 0.05} ${-base_width/2.0 + 0.05} -0.03"/>
       <geometry>
-        <mesh filename="package://mrover/rover_description/meshes/chassis.stl" scale="${mesh_scale}"/>
+        <box size="${base_len} ${base_width} 0.01" />
       </geometry>
-      <material name="blue" />
+      <material name="black" />
     </visual>
     <collision>
       <geometry>
-        <box size="${base_len} ${base_width} ${base_height}" />
+        <box size="${base_len} ${base_width} 0.01" />
       </geometry>
     </collision>
   </link>
-  <link name="right_rocker_link">
-    <xacro:box_inertia m="3.0" w="${base_len}" h="${base_width}" d="${base_height}" />
-    <visual>
-      <origin rpy="${PI/2} 0 ${PI/2}" xyz="0.11 0.22 -0.3"/>
-      <geometry>
-        <mesh filename="package://mrover/rover_description/meshes/right_rocker.stl" scale="${mesh_scale}"/>
-      </geometry>
-      <material name="red" />
-    </visual>
-    <collision>
-      <geometry>
-        <box size="${base_len + 0.17} 0.05 ${base_height + 0.2}" />
-      </geometry>
-    </collision>
-  </link>
-  <joint name="base_right_rocker_joint" type="fixed">
-    <origin xyz="0.01 ${-base_width/2.0 - 0.05} -0.2" rpy="0 0 0" />
-    <parent link="base_link" />
-    <child link="right_rocker_link" />
-  </joint>
-  <link name="left_rocker_link">
-    <xacro:box_inertia m="3.0" w="${base_len}" h="${base_width}" d="${base_height}" />
-    <visual>
-      <origin rpy="0.0 0.0 0.0" xyz="0.0 0.0 0.0"/>
-      <geometry>
-        <mesh filename="package://mrover/rover_description/meshes/left_rocker.stl" scale="${mesh_scale}"/>
-      </geometry>
-      <material name="white" />
-    </visual>
-    <collision>
-      <geometry>
-        <box size="${base_len + 0.17} 0.05 ${base_height + 0.2}" />
-      </geometry>
-    </collision>
-  </link>
-  <joint name="base_left_rocker_joint" type="fixed">
-    <origin xyz="0.01 ${base_width/2.0 + 0.05} -0.2" rpy="0 0 0" />
-    <parent link="base_link" />
-    <child link="left_rocker_link" />
-  </joint>
   <!--base_link to base_footprint Joint-->
   <joint name="base_link_joint" type="fixed">
