Commit message: Align all visual geometry

File: rover_description/new_arm/arm.xacro (robot description, xacro)
@@ -64,7 +64,7 @@
         </collision>
     </xacro:macro>
-    <xacro:macro name="joints" params="name type:=revolute parent child origin_x origin_y origin_z axis_x:=0 axis_y:=0 axis_z:=0 lower upper damp:=1.0">
+    <xacro:macro name="joints" params="name type:=revolute parent child roll:=0 pitch:=0 yaw:=0 origin_x origin_y origin_z axis_x:=0 axis_y:=0 axis_z:=0 lower upper damp:=1.0" >
         <joint name="${name}" type="${type}">
-            <origin xyz="${origin_x} ${origin_y} ${origin_z}" rpy="0 0 0" />
+            <origin xyz="${origin_x} ${origin_y} ${origin_z}" rpy="${roll} ${pitch} ${yaw}" />
             <parent link="${parent}" />
             <child link="${child}" />
@@ -98,5 +98,5 @@
     <!-- <link name=x -->
     <link name="chassisToa">
-        <xacro:link-visual fileName="chassis-a.stl" x="0" y="0" z="0" col="red" r="1" g="0" b="0" roll="${-1.0*PI/2.0}"/>
+        <xacro:link-visual fileName="chassis-a.stl" x="0" y="0" z="0" col="red" r="1" g="0" b="0"/>
         <xacro:link-collision-cylinder radius="3.75" x1="0" y1="0" z1="-1.25" x2="0" y2="0" z2="-3.75" />
         <xacro:link-collision-cylinder radius="1.75" x1="-3.6467207" y1="3.6590503" z1="-0.6913988" x2="-3.6467207" y2="3.6590503" z2="-2.6913988" />
@@ -110,6 +110,6 @@
         <xacro:link-inertial y="-1.75" z="3" mass="0.5" ixx="1.9" iyy="0.7" izz="0.5" />
     </link>
-    <!--link name="bToc">
-        <xacro:link-visual fileName="b-c.stl" x="0" y="0" z="0" col="yellow" r="1" g="1" b="0" roll="0"/>
+    <link name="bToc">
+        <xacro:link-visual fileName="b-c-blender.stl" x="0" y="0" z="0" col="yellow" r="1" g="1" b="0" roll="0"/>
         <xacro:link-collision-box y="12" lx="3" ly="24" lz="3" />
         <xacro:link-collision-cylinder radius="1" x1="0" y1="23" z1="0" x2="5" y2="23" z2="0" />
@@ -123,5 +123,5 @@
     </link>
     <link name="dToe">
-        <xacro:link-visual fileName="d-e-blender.stl" x="0" y="0" z="0" col="blue" r="0" g="0" b="1"/>
+        <xacro:link-visual fileName="d-e-blender.stl" x="0" y="0" z="0" col="blue" r="0" g="0" b="1" pitch="0" roll="0"/>
         <xacro:link-collision-box y="-7.6324" z="4.7693" lx="2.5" ly="20" lz="2.5" roll="-0.558505" />
         <xacro:link-collision-box x="1" y="-13.75" z="9.5" lx="3" ly="3" lz="6" roll="-0.558505" />
@@ -129,15 +129,15 @@
     </link>
     <link name="eTof">
-        <xacro:link-visual fileName="e-f-blender.stl" x="0" y="0" z="0" col="violet" r="0.5" g="0" b="1" roll="1.67552" />
+        <xacro:link-visual fileName="e-f-blender2.stl" x="0" y="0" z="0" col="violet" r="0.5" g="0" b="1" roll="0" />
         <xacro:link-collision-cylinder radius="1" x1="-0.75" y1="0" z1="0" x2="-0.75" y2="0" z2="-6" />
         <xacro:link-inertial z="-3" mass="0.5" ixx="1.6" iyy="1.6" izz="0.25" />
     </link>
     <link name="hand">
-        <xacro:link-visual fileName="hand.stl" x="0" y="0" z="0" col="pink" r="1" g="0" b="1" yaw="${PI}" roll="-1.67552"/>
+        <xacro:link-visual fileName="hand-blender2.stl" x="0" y="0" z="0" col="pink" r="1" g="0" b="1"/>
         <xacro:link-collision-box z="-2.5" lx="7" ly="2" lz="7" />
         <xacro:link-collision-box y="-8" lx="3" ly="2" lz="4" />
         <xacro:link-collision-cylinder radius="0.75" x1="-1.5" y1="0" z1="-0.5" x2="-1.5" y2="-9" z2="-0.5" />
         <xacro:link-inertial z="-2.5" mass="0.5" ixx="2.2" iyy="4" izz="2.2" />
-    </link> -->
+    </link>
     <link name="world" />
     <joint name="virtual_joint" type="fixed">
@@ -146,10 +146,16 @@
         <origin xyz="0 0 ${base_height/2.0}" rpy="0 0 0" />
     </joint>
+    <!-- <xacro:joints name="joint_c" parent="bToc" child="cTod" origin_x="-4.59961" origin_y="22.83397" origin_z="0.38119" axis_x="1" lower="-3.01" upper="2.73" /> -->
+    <!-- /home/joe/Desktop/mrover_catkin_ws/src/mrover/rover_description/new_arm -->
     <xacro:joints name="joint_a" type="continuous" parent="chassisToa" child="aTob" origin_x="0" origin_y="0" origin_z="0" axis_z="1" lower="-3.14" upper="3.14" />
-    <!-- <xacro:joints name="joint_b" parent="aTob" child="bToc" origin_x="0" origin_y="1.41293" origin_z="1.13303" axis_x="1" lower="0.035" upper="1.09" />
-    <xacro:joints name="joint_c" parent="bToc" child="cTod" origin_x="-4.59961" origin_y="22.83397" origin_z="0.38119" axis_x="1" lower="-3.01" upper="2.73" />
-    <xacro:joints name="joint_d" parent="cTod" child="dToe" origin_x="0" origin_y="-1.4699" origin_z="0.963976" axis_z="-0.52992" axis_y="0.84805" lower="-3.14" upper="3.14" />
-    <xacro:joints name="joint_e" parent="dToe" child="eTof" origin_x="-2.30884" origin_y="-14.2085" origin_z="9.01643" axis_x="1" lower="-2.68" upper="2.68" />
-    <xacro:joints name="joint_f" parent="eTof" child="hand" origin_x="-0.817441" origin_y="0.678501" origin_z="-6.45623" axis_z="1" lower="-3.14" upper="3.14" /> -->
+    <xacro:joints name="joint_b" parent="aTob" child="bToc" origin_x="0" origin_y="1.33" origin_z="0.99" axis_x="1" lower="-0.48079632679" upper="1.09" />
+    <xacro:joints name="joint_c" parent="bToc" child="cTod" origin_x="0" origin_y="20.11" origin_z="10.75" axis_x="1" lower="-3.01" upper="2.73" />
+    <xacro:joints name="joint_d" parent="cTod" child="dToe" origin_x="-4.4" origin_y="-0.42" origin_z="-2.535" axis_z="1" axis_y="0" lower="-3.14" upper="3.14" roll="-0.15708" pitch="-0.0174533" />
+    <!-- <xacro:joints name="joint_e" parent="dToe" child="eTof" origin_x="-2.30884" origin_y="-14.2085" origin_z="9.01643" axis_x="1" lower="-2.68" upper="2.68" /> -->
+    <!-- <xacro:joints name="joint_e" parent="dToe" child="eTof" origin_x="-7.78" origin_y="20.05" origin_z="-10.385" axis_x="1" lower="-2.68" upper="2.68" /> -->
+    <!-- pitch="-0.4694936" -->
+    <xacro:joints name="joint_e" parent="dToe" child="eTof" origin_x="0.75" origin_y="2.5" origin_z="-17" axis_y="1" lower="-2.68" upper="2.68" roll="0" pitch="0" yaw="-0.471239"/>
+    <xacro:joints name="joint_f" parent="eTof" child="hand" origin_x="-6.3" origin_y="1.75" origin_z="0" axis_x="1" lower="-3.14" upper="3.14" />
+    <!-- x 0.16 m y -0.47 m z -0.09 m -->
     <!-- <xacro:transmissions name="joint_a" />
     <xacro:transmissions name="joint_b" />
