Commit message: Got arm components to display in rviz, still messed up, need to blenderize stl files bc axes are weird

File: rover_description/arm/arm.xacro (robot description, xacro)
@@ -2,9 +2,10 @@
 <robot xmlns:xacro="http://www.ros.org/wiki/xacro" name="mrover_arm">
     <virtual_joint name="" type="fixed" parent_frame="world" child_link="chassis-a" />
-    <xacro:macro name="link-visual" params="x y z col r g b">
+    <xacro:property name="scale_factor" value="0.7357" />
+    <xacro:macro name="link-visual" params="fileName x y z col r g b">
         <visual>
             <origin xyz="${x} ${y} ${z}" rpy="0 0 0" />
             <geometry>
-                <mesh filename="package://mrover/rover_description/arm/${name}.stl" />
+                <mesh filename="package://mrover/rover_description/arm/${fileName}.stl" />
             </geometry>
             <material name="${col}">
@@ -64,33 +65,33 @@
     </xacro:macro>
     <link name="chassis-a">
-        <xacro:link-visual name="chassis-a" x="0" y="0" z="0" col="red" r="1" g="0" b="0" />
+        <xacro:link-visual fileName="chassis-a" x="0" y="0" z="0" col="red" r="1" g="0" b="0" />
         <!-- TODO: fill in collision objects for all links -->
+        <!-- <xacro:link-collision radius="" x1="" y1="" z1="" x2="" y2="" z2="" />
         <xacro:link-collision radius="" x1="" y1="" z1="" x2="" y2="" z2="" />
-        <xacro:link-collision radius="" x1="" y1="" z1="" x2="" y2="" z2="" />
-        <xacro:link-collision radius="" x1="" y1="" z1="" x2="" y2="" z2="" />
+        <xacro:link-collision radius="" x1="" y1="" z1="" x2="" y2="" z2="" /> -->
     </link>
     <link name="a-b">
-        <xacro:link-visual name="a-b" x="0" y="0" z="0" col="orange" r="1" g="0.43" b="0" />
+        <xacro:link-visual fileName="a-b" x="0" y="0" z="0" col="orange" r="1" g="0.43" b="0" />
     </link>
     <link name="b-c">
-        <xacro:link-visual name="b-c" x="0" y="0.03429" z="0.02858" col="yellow" r="1" g="1" b="0" />
+        <xacro:link-visual fileName="b-c" x="0" y="30" z="1" col="yellow" r="1" g="1" b="0" />
     </link>
-    <link name="c-d">
-        <xacro:link-visual name="c-d" x="-0.0584" y="0.58039" z="0.009525" col="green" r="0.43" g="1" b="0" />
+    <!-- <link name="c-d">
+        <xacro:link-visual fileName="c-d" x="0" y="${0.5393*scale_factor}" z="${0*scale_factor}" col="green" r="0.43" g="1" b="0" />
     </link>
     <link name="d-e">
-        <xacro:link-visual name="d-e" x="-0.044323" y="0.0583946" z="0" col="blue" r="0" g="0" b="1" />
+        <xacro:link-visual fileName="d-e" x="0" y="${-1*scale_factor}" z="${5*scale_factor}" col="blue" r="0" g="0" b="1" />
     </link>
     <link name="e-f">
-        <xacro:link-visual name="e-f" x="0.0583946" y="0.426847" z="0" col="violet" r="0.5" g="0" b="1" />
+        <xacro:link-visual fileName="e-f" x="${1.002*scale_factor}" y="${-2.7240*scale_factor}" z="${-22.6051*scale_factor}" col="violet" r="0.5" g="0" b="1" />
     </link>
     <link name="hand">
-        <xacro:link-visual name="hand" x="0.0206502" y="0.1647444" z="-0.028575" col="pink" r="1" g="0" b="1" />
-    </link>
+        <xacro:link-visual fileName="hand" x="${2.5166*scale_factor}" y="${-2.7226*scale_factor}" z="${-34.3566*scale_factor}" col="pink" r="1" g="0" b="1" />
+    </link> -->
     <xacro:joints name="joint_a" type="continuous" parent="chassis-a" child="a-b" origin_x="0" origin_y="0" origin_z="0" axis_z="1" lower="-3.14" upper="3.14" />
     <xacro:joints name="joint_b" parent="a-b" child="b-c" origin_x="0" origin_y="0.03429" origin_z="0.028575" axis_x="1" lower="0.035" upper="1.09" />
-    <xacro:joints name="joint_c" parent="b-c" child="c-d" origin_x="-0.0584" origin_y="0.58039" origin_z="0.009525" axis_x="1" lower="-3.01" upper="2.73" />
+    <!-- <xacro:joints name="joint_c" parent="b-c" child="c-d" origin_x="-0.0584" origin_y="0.58039" origin_z="0.009525" axis_x="1" lower="-3.01" upper="2.73" />
     <xacro:joints name="joint_d" parent="c-d" child="d-e" origin_x="-0.044" origin_y="0.05840025" origin_z="0" axis_y="1" lower="-3.14" upper="3.14" />
     <xacro:joints name="joint_e" parent="d-e" child="e-f" origin_x="0.058401009944" origin_y="0.427" origin_z="0" axis_x="1" lower="-2.68" upper="2.68" />
-    <xacro:joints name="joint_f" parent="e-f" child="hand" origin_x="0.021" origin_y="0.164741225" origin_z="0" axis_z="1" lower="-3.14" upper="3.14" />
+    <xacro:joints name="joint_f" parent="e-f" child="hand" origin_x="0.021" origin_y="0.164741225" origin_z="0" axis_z="1" lower="-3.14" upper="3.14" /> -->
 </robot>

Commit message: Commit progress

File: rover_description/arm/arm.xacro (robot description, xacro)
@@ -2,10 +2,10 @@
 <robot xmlns:xacro="http://www.ros.org/wiki/xacro" name="mrover_arm">
     <virtual_joint name="" type="fixed" parent_frame="world" child_link="chassis-a" />
-    <xacro:property name="scale_factor" value="0.7357" />
-    <xacro:macro name="link-visual" params="fileName x y z col r g b">
+    <xacro:property name="PI" value="3.141592" />
+    <xacro:macro name="link-visual" params="fileName x y z col r g b roll:=0 pitch:=0 yaw:=0">
         <visual>
-            <origin xyz="${x} ${y} ${z}" rpy="0 0 0" />
+            <origin xyz="${x} ${y} ${z}" rpy="${roll} ${pitch} ${yaw}" />
             <geometry>
-                <mesh filename="package://mrover/rover_description/arm/${fileName}.stl" />
+                <mesh filename="package://mrover/rover_description/arm/${fileName}" />
             </geometry>
             <material name="${col}">
@@ -65,5 +65,5 @@
     </xacro:macro>
     <link name="chassis-a">
-        <xacro:link-visual fileName="chassis-a" x="0" y="0" z="0" col="red" r="1" g="0" b="0" />
+        <xacro:link-visual fileName="chassis-a.stl" x="0" y="0" z="0" col="red" r="1" g="0" b="0" />
         <!-- TODO: fill in collision objects for all links -->
         <!-- <xacro:link-collision radius="" x1="" y1="" z1="" x2="" y2="" z2="" />
@@ -72,8 +72,8 @@
     </link>
     <link name="a-b">
-        <xacro:link-visual fileName="a-b" x="0" y="0" z="0" col="orange" r="1" g="0.43" b="0" />
+        <xacro:link-visual fileName="a-b.stl" x="0" y="0" z="0" col="orange" r="1" g="0.43" b="0" />
     </link>
     <link name="b-c">
-        <xacro:link-visual fileName="b-c" x="0" y="30" z="1" col="yellow" r="1" g="1" b="0" />
+        <xacro:link-visual fileName="b-c-blender.stl" x="0" y="1.5" z="0" col="yellow" r="1" g="1" b="0" roll="0.558505"/>
     </link>
     <!-- <link name="c-d">

Commit message: Urdf up to joint E

File: rover_description/arm/arm.xacro (robot description, xacro)
@@ -75,23 +75,23 @@
     </link>
     <link name="b-c">
-        <xacro:link-visual fileName="b-c-blender.stl" x="0" y="1.5" z="0" col="yellow" r="1" g="1" b="0" roll="0.558505"/>
+        <xacro:link-visual fileName="b-c.stl" x="0" y="0" z="0" col="yellow" r="1" g="1" b="0" roll="0"/>
     </link>
-    <!-- <link name="c-d">
-        <xacro:link-visual fileName="c-d" x="0" y="${0.5393*scale_factor}" z="${0*scale_factor}" col="green" r="0.43" g="1" b="0" />
+    <link name="c-d">
+        <xacro:link-visual fileName="c-d-blender.stl" x="0" y="0" z="0" col="green" r="0.43" g="1" b="0"/>
     </link>
     <link name="d-e">
-        <xacro:link-visual fileName="d-e" x="0" y="${-1*scale_factor}" z="${5*scale_factor}" col="blue" r="0" g="0" b="1" />
+        <xacro:link-visual fileName="d-e-blender.stl" x="0" y="0" z="0" col="blue" r="0" g="0" b="1"/>
     </link>
-    <link name="e-f">
-        <xacro:link-visual fileName="e-f" x="${1.002*scale_factor}" y="${-2.7240*scale_factor}" z="${-22.6051*scale_factor}" col="violet" r="0.5" g="0" b="1" />
+     <link name="e-f">
+        <xacro:link-visual fileName="e-f-blender.stl" x="0" y="0" z="0" col="violet" r="0.5" g="0" b="1" roll="1.67552" />
     </link>
-    <link name="hand">
+    <!--<link name="hand">
         <xacro:link-visual fileName="hand" x="${2.5166*scale_factor}" y="${-2.7226*scale_factor}" z="${-34.3566*scale_factor}" col="pink" r="1" g="0" b="1" />
     </link> -->
     <xacro:joints name="joint_a" type="continuous" parent="chassis-a" child="a-b" origin_x="0" origin_y="0" origin_z="0" axis_z="1" lower="-3.14" upper="3.14" />
-    <xacro:joints name="joint_b" parent="a-b" child="b-c" origin_x="0" origin_y="0.03429" origin_z="0.028575" axis_x="1" lower="0.035" upper="1.09" />
-    <!-- <xacro:joints name="joint_c" parent="b-c" child="c-d" origin_x="-0.0584" origin_y="0.58039" origin_z="0.009525" axis_x="1" lower="-3.01" upper="2.73" />
-    <xacro:joints name="joint_d" parent="c-d" child="d-e" origin_x="-0.044" origin_y="0.05840025" origin_z="0" axis_y="1" lower="-3.14" upper="3.14" />
-    <xacro:joints name="joint_e" parent="d-e" child="e-f" origin_x="0.058401009944" origin_y="0.427" origin_z="0" axis_x="1" lower="-2.68" upper="2.68" />
-    <xacro:joints name="joint_f" parent="e-f" child="hand" origin_x="0.021" origin_y="0.164741225" origin_z="0" axis_z="1" lower="-3.14" upper="3.14" /> -->
+    <xacro:joints name="joint_b" parent="a-b" child="b-c" origin_x="0" origin_y="1.41293" origin_z="1.13303" axis_x="1" lower="0.035" upper="1.09" />
+    <xacro:joints name="joint_c" parent="b-c" child="c-d" origin_x="-4.59961" origin_y="22.83397" origin_z="0.38119" axis_x="1" lower="-3.01" upper="2.73" />
+    <xacro:joints name="joint_d" parent="c-d" child="d-e" origin_x="0" origin_y="-1.4699" origin_z="0.963976" axis_z="-0.52992" axis_y="0.84805" lower="-3.14" upper="3.14" />
+    <xacro:joints name="joint_e" parent="d-e" child="e-f" origin_x="-2.30884" origin_y="-14.2085" origin_z="9.01643" axis_x="1" lower="-2.68" upper="2.68" />
+    <!--<xacro:joints name="joint_f" parent="e-f" child="hand" origin_x="0.021" origin_y="0.164741225" origin_z="0" axis_z="1" lower="-3.14" upper="3.14" /> -->
 </robot>

Commit message: visuals of URDF complete

File: rover_description/arm/arm.xacro (robot description, xacro)
@@ -86,7 +86,7 @@
         <xacro:link-visual fileName="e-f-blender.stl" x="0" y="0" z="0" col="violet" r="0.5" g="0" b="1" roll="1.67552" />
     </link>
-    <!--<link name="hand">
-        <xacro:link-visual fileName="hand" x="${2.5166*scale_factor}" y="${-2.7226*scale_factor}" z="${-34.3566*scale_factor}" col="pink" r="1" g="0" b="1" />
-    </link> -->
+    <link name="hand">
+        <xacro:link-visual fileName="hand.stl" x="0" y="0" z="0" col="pink" r="1" g="0" b="1" yaw="${PI}" roll="-1.67552"/>
+    </link>
     <xacro:joints name="joint_a" type="continuous" parent="chassis-a" child="a-b" origin_x="0" origin_y="0" origin_z="0" axis_z="1" lower="-3.14" upper="3.14" />
     <xacro:joints name="joint_b" parent="a-b" child="b-c" origin_x="0" origin_y="1.41293" origin_z="1.13303" axis_x="1" lower="0.035" upper="1.09" />
@@ -94,4 +94,4 @@
     <xacro:joints name="joint_d" parent="c-d" child="d-e" origin_x="0" origin_y="-1.4699" origin_z="0.963976" axis_z="-0.52992" axis_y="0.84805" lower="-3.14" upper="3.14" />
     <xacro:joints name="joint_e" parent="d-e" child="e-f" origin_x="-2.30884" origin_y="-14.2085" origin_z="9.01643" axis_x="1" lower="-2.68" upper="2.68" />
-    <!--<xacro:joints name="joint_f" parent="e-f" child="hand" origin_x="0.021" origin_y="0.164741225" origin_z="0" axis_z="1" lower="-3.14" upper="3.14" /> -->
+    <xacro:joints name="joint_f" parent="e-f" child="hand" origin_x="-0.817441" origin_y="0.678501" origin_z="-6.45623" axis_z="1" lower="-3.14" upper="3.14" />
 </robot>

Commit message: Define cylinder and box collision xacros

File: rover_description/arm/arm.xacro (robot description, xacro)
@@ -14,20 +14,16 @@
         </visual>
     </xacro:macro>
-    <!-- defines a capsule collision object -->
-    <xacro:macro name="link-collision" params="radius x1 y1 z1 x2 y2 z2">
+    <!-- defines a cylinder collision object with two endpoints -->
+    <xacro:macro name="link-collision-cylinder" params="radius x1 y1 z1 x2 y2 z2">
         <xacro:property name="dx" value="${x2-x1}" />
         <xacro:property name="dy" value="${y2-y1}" />
         <xacro:property name="dz" value="${z2-z1}" />
-        <xacro:property name="mx" value="${x1+dx/2}" />
-        <xacro:property name="my" value="${y1+dy/2}" />
-        <xacro:property name="mz" value="${z1+dz/2}" />
-        <xacro:property name="pi" value="3.1415926" />
         <xacro:if value="${dx != 0}">
             <xacro:property name="length" value="${dx}" />
-            <xacro:property name="rpy" value="0 ${pi/2} 0" />
+            <xacro:property name="rpy" value="0 ${PI/2} 0" />
         </xacro:if>
         <xacro:if value="${dy != 0}">
             <xacro:property name="length" value="${dy}" />
-            <xacro:property name="rpy" value="${pi/2} 0 0" />
+            <xacro:property name="rpy" value="${PI/2} 0 0" />
         </xacro:if>
         <xacro:if value="${dz != 0}">
@@ -38,17 +34,14 @@
             <origin xyz="${x1+dx/2} ${y1+dy/2} ${z1+dz/2}" rpy="${rpy}" />
             <geometry>
-                <cylinder radius="${radius}" length="length" />
+                <cylinder radius="${radius}" length="${length}" />
             </geometry>
         </collision>
+    </xacro:macro>
+    <!-- defines a box collision object with the center and dimensions -->
+    <xacro:macro name="link-collision-box" params="x:=0 y:=0 z:=0 lx ly lz">
         <collision>
-            <origin xyz="${x1} ${y1} ${z1}" rpy="0 0 0" />
+            <origin xyz="${x} ${y} ${z}" rpy="0 0 0" />
             <geometry>
-                <sphere radius="${radius}" />
-            </geometry>
-        </collision>
-        <collision>
-            <origin xyz="${x2} ${y2} ${z2}" rpy="0 0 0" />
-            <geometry>
-                <sphere radius="${radius}" />
+                <box size="${lx} ${ly} ${lz}" />
             </geometry>
         </collision>
@@ -76,4 +69,6 @@
     <link name="b-c">
         <xacro:link-visual fileName="b-c.stl" x="0" y="0" z="0" col="yellow" r="1" g="1" b="0" roll="0"/>
+        <!-- <xacro:link-collision radius="2" x1="0" y1="0" z1="0" x2="0" y2="25" z2="0" /> -->
+        <xacro:link-collision-box y="12" lx="4" ly="24" lz="4" />
     </link>
     <link name="c-d">

Commit message: Add collision models

File: rover_description/arm/arm.xacro (robot description, xacro)
@@ -15,19 +15,19 @@
     </xacro:macro>
     <!-- defines a cylinder collision object with two endpoints -->
-    <xacro:macro name="link-collision-cylinder" params="radius x1 y1 z1 x2 y2 z2">
+    <xacro:macro name="link-collision-cylinder" params="radius x1 y1 z1 x2 y2 z2 roll:=0 pitch:=0 yaw:=0">
         <xacro:property name="dx" value="${x2-x1}" />
         <xacro:property name="dy" value="${y2-y1}" />
         <xacro:property name="dz" value="${z2-z1}" />
         <xacro:if value="${dx != 0}">
-            <xacro:property name="length" value="${dx}" />
-            <xacro:property name="rpy" value="0 ${PI/2} 0" />
+            <xacro:property name="length" value="${fabs(dx)}" />
+            <xacro:property name="rpy" value="${roll} ${pitch+PI/2} ${yaw}" />
         </xacro:if>
         <xacro:if value="${dy != 0}">
-            <xacro:property name="length" value="${dy}" />
-            <xacro:property name="rpy" value="${PI/2} 0 0" />
+            <xacro:property name="length" value="${fabs(dy)}" />
+            <xacro:property name="rpy" value="${roll+PI/2} ${pitch} ${yaw}" />
         </xacro:if>
         <xacro:if value="${dz != 0}">
-            <xacro:property name="length" value="${dz}" />
-            <xacro:property name="rpy" value="0 0 0" />
+            <xacro:property name="length" value="${fabs(dz)}" />
+            <xacro:property name="rpy" value="${roll} ${pitch} ${yaw}" />
         </xacro:if>
         <collision>
@@ -39,7 +39,7 @@
     </xacro:macro>
     <!-- defines a box collision object with the center and dimensions -->
-    <xacro:macro name="link-collision-box" params="x:=0 y:=0 z:=0 lx ly lz">
+    <xacro:macro name="link-collision-box" params="x:=0 y:=0 z:=0 lx ly lz roll:=0 pitch:=0 yaw:=0">
         <collision>
-            <origin xyz="${x} ${y} ${z}" rpy="0 0 0" />
+            <origin xyz="${x} ${y} ${z}" rpy="${roll} ${pitch} ${yaw}" />
             <geometry>
                 <box size="${lx} ${ly} ${lz}" />
@@ -59,28 +59,34 @@
     <link name="chassis-a">
         <xacro:link-visual fileName="chassis-a.stl" x="0" y="0" z="0" col="red" r="1" g="0" b="0" />
-        <!-- TODO: fill in collision objects for all links -->
-        <!-- <xacro:link-collision radius="" x1="" y1="" z1="" x2="" y2="" z2="" />
-        <xacro:link-collision radius="" x1="" y1="" z1="" x2="" y2="" z2="" />
-        <xacro:link-collision radius="" x1="" y1="" z1="" x2="" y2="" z2="" /> -->
+        <xacro:link-collision-cylinder radius="3.75" x1="0" y1="0" z1="-1.25" x2="0" y2="0" z2="-3.75" />
+        <xacro:link-collision-cylinder radius="1.75" x1="-3.6467207" y1="3.6590503" z1="-0.6913988" x2="-3.6467207" y2="3.6590503" z2="-2.6913988" />
     </link>
     <link name="a-b">
         <xacro:link-visual fileName="a-b.stl" x="0" y="0" z="0" col="orange" r="1" g="0.43" b="0" />
+        <xacro:link-collision-box y="-1.75" z="3" lx="2" ly="3" lz="6" />
+        <xacro:link-collision-cylinder radius="2" x1="0" y1="0" z1="-0.25" x2="0" y2="0" z2="0.75" />
     </link>
     <link name="b-c">
         <xacro:link-visual fileName="b-c.stl" x="0" y="0" z="0" col="yellow" r="1" g="1" b="0" roll="0"/>
-        <!-- <xacro:link-collision radius="2" x1="0" y1="0" z1="0" x2="0" y2="25" z2="0" /> -->
-        <xacro:link-collision-box y="12" lx="4" ly="24" lz="4" />
+        <xacro:link-collision-box y="12" lx="3" ly="24" lz="3" />
+        <xacro:link-collision-cylinder radius="1" x1="0" y1="23" z1="0" x2="5" y2="23" z2="0" />
     </link>
     <link name="c-d">
         <xacro:link-visual fileName="c-d-blender.stl" x="0" y="0" z="0" col="green" r="0.43" g="1" b="0"/>
+        <xacro:link-collision-cylinder radius="2" x1="3" y1="0" z1="0" x2="-5" y2="0" z2="0" />
     </link>
     <link name="d-e">
         <xacro:link-visual fileName="d-e-blender.stl" x="0" y="0" z="0" col="blue" r="0" g="0" b="1"/>
+        <xacro:link-collision-box y="-7.6324" z="4.7693" lx="2.5" ly="20" lz="2.5" roll="-0.558505" />
     </link>
-     <link name="e-f">
+    <link name="e-f">
         <xacro:link-visual fileName="e-f-blender.stl" x="0" y="0" z="0" col="violet" r="0.5" g="0" b="1" roll="1.67552" />
+        <xacro:link-collision-cylinder radius="1" x1="-0.75" y1="0" z1="0" x2="-0.75" y2="0" z2="-6" />
     </link>
     <link name="hand">
         <xacro:link-visual fileName="hand.stl" x="0" y="0" z="0" col="pink" r="1" g="0" b="1" yaw="${PI}" roll="-1.67552"/>
+        <xacro:link-collision-box z="-2.5" lx="5" ly="2" lz="7" />
+        <xacro:link-collision-box y="-8" lx="3" ly="2" lz="4" />
+        <xacro:link-collision-cylinder radius="0.75" x1="-1.5" y1="0" z1="-0.5" x2="-1.5" y2="-9" z2="-0.5" />
     </link>
     <xacro:joints name="joint_a" type="continuous" parent="chassis-a" child="a-b" origin_x="0" origin_y="0" origin_z="0" axis_z="1" lower="-3.14" upper="3.14" />
