Commit message: xacro link name changes

File: rover_description/arm/arm.xacro (robot description, xacro)
@@ -57,15 +57,15 @@
         </joint>
     </xacro:macro>
-    <link name="chassis-a">
+    <link name="chassisToa">
         <xacro:link-visual fileName="chassis-a.stl" x="0" y="0" z="0" col="red" r="1" g="0" b="0" />
         <xacro:link-collision-cylinder radius="3.75" x1="0" y1="0" z1="-1.25" x2="0" y2="0" z2="-3.75" />
         <xacro:link-collision-cylinder radius="1.75" x1="-3.6467207" y1="3.6590503" z1="-0.6913988" x2="-3.6467207" y2="3.6590503" z2="-2.6913988" />
     </link>
-    <link name="a-b">
+    <link name="aTob">
         <xacro:link-visual fileName="a-b.stl" x="0" y="0" z="0" col="orange" r="1" g="0.43" b="0" />
         <xacro:link-collision-box y="-1.75" z="3" lx="2" ly="3" lz="6" />
         <xacro:link-collision-cylinder radius="2" x1="0" y1="0" z1="-0.25" x2="0" y2="0" z2="0.75" />
     </link>
-    <link name="b-c">
+    <link name="bToc">
         <xacro:link-visual fileName="b-c.stl" x="0" y="0" z="0" col="yellow" r="1" g="1" b="0" roll="0"/>
         <xacro:link-collision-box y="12" lx="3" ly="24" lz="3" />
@@ -73,14 +73,14 @@
         <xacro:link-collision-cylinder radius="1" x1="0" y1="0" z1="3.75" x2="0" y2="17" z2="3.75" roll="-0.3"/>
     </link>
-    <link name="c-d">
+    <link name="cTod">
         <xacro:link-visual fileName="c-d-blender.stl" x="0" y="0" z="0" col="green" r="0.43" g="1" b="0"/>
         <xacro:link-collision-cylinder radius="2" x1="3" y1="0" z1="0" x2="-5" y2="0" z2="0" />
     </link>
-    <link name="d-e">
+    <link name="dToe">
         <xacro:link-visual fileName="d-e-blender.stl" x="0" y="0" z="0" col="blue" r="0" g="0" b="1"/>
         <xacro:link-collision-box y="-7.6324" z="4.7693" lx="2.5" ly="20" lz="2.5" roll="-0.558505" />
         <xacro:link-collision-box x="1" y="-13.75" z="9.5" lx="3" ly="3" lz="6" roll="-0.558505" />
     </link>
-    <link name="e-f">
+    <link name="eTof">
         <xacro:link-visual fileName="e-f-blender.stl" x="0" y="0" z="0" col="violet" r="0.5" g="0" b="1" roll="1.67552" />
         <xacro:link-collision-cylinder radius="1" x1="-0.75" y1="0" z1="0" x2="-0.75" y2="0" z2="-6" />
@@ -92,9 +92,9 @@
         <xacro:link-collision-cylinder radius="0.75" x1="-1.5" y1="0" z1="-0.5" x2="-1.5" y2="-9" z2="-0.5" />
     </link>
-    <xacro:joints name="joint_a" type="continuous" parent="chassis-a" child="a-b" origin_x="0" origin_y="0" origin_z="0" axis_z="1" lower="-3.14" upper="3.14" />
-    <xacro:joints name="joint_b" parent="a-b" child="b-c" origin_x="0" origin_y="1.41293" origin_z="1.13303" axis_x="1" lower="0.035" upper="1.09" />
-    <xacro:joints name="joint_c" parent="b-c" child="c-d" origin_x="-4.59961" origin_y="22.83397" origin_z="0.38119" axis_x="1" lower="-3.01" upper="2.73" />
-    <xacro:joints name="joint_d" parent="c-d" child="d-e" origin_x="0" origin_y="-1.4699" origin_z="0.963976" axis_z="-0.52992" axis_y="0.84805" lower="-3.14" upper="3.14" />
-    <xacro:joints name="joint_e" parent="d-e" child="e-f" origin_x="-2.30884" origin_y="-14.2085" origin_z="9.01643" axis_x="1" lower="-2.68" upper="2.68" />
-    <xacro:joints name="joint_f" parent="e-f" child="hand" origin_x="-0.817441" origin_y="0.678501" origin_z="-6.45623" axis_z="1" lower="-3.14" upper="3.14" />
+    <xacro:joints name="joint_a" type="continuous" parent="chassisToa" child="aTob" origin_x="0" origin_y="0" origin_z="0" axis_z="1" lower="-3.14" upper="3.14" />
+    <xacro:joints name="joint_b" parent="aTob" child="bToc" origin_x="0" origin_y="1.41293" origin_z="1.13303" axis_x="1" lower="0.035" upper="1.09" />
+    <xacro:joints name="joint_c" parent="bToc" child="cTod" origin_x="-4.59961" origin_y="22.83397" origin_z="0.38119" axis_x="1" lower="-3.01" upper="2.73" />
+    <xacro:joints name="joint_d" parent="cTod" child="dToe" origin_x="0" origin_y="-1.4699" origin_z="0.963976" axis_z="-0.52992" axis_y="0.84805" lower="-3.14" upper="3.14" />
+    <xacro:joints name="joint_e" parent="dToe" child="eTof" origin_x="-2.30884" origin_y="-14.2085" origin_z="9.01643" axis_x="1" lower="-2.68" upper="2.68" />
+    <xacro:joints name="joint_f" parent="eTof" child="hand" origin_x="-0.817441" origin_y="0.678501" origin_z="-6.45623" axis_z="1" lower="-3.14" upper="3.14" />
 </robot>

Commit message: define urdf macro for inertial

File: rover_description/arm/arm.xacro (robot description, xacro)
@@ -13,4 +13,10 @@
             </material>
         </visual>
+    </xacro:macro>
+    <xacro:macro name="link-inertial" params="x:=0 y:=0 z:=0 roll:=0 pitch:=0 yaw:=0 mass ixx iyy izz ixy:=0 iyz:=0 ixz:=0">
+        <origin xyz="${x} ${y} ${z}" rpy="${roll} ${pitch} ${yaw}" />
+        <!-- mass in kg -->
+        <mass value="${mass}" />
+        <inertia ixx="${ixx}" iyy="${iyy}" izz="${izz}" ixy="${ixy}" iyz="${iyz}" ixz="${ixz}" />
     </xacro:macro>
     <!-- defines a cylinder collision object with two endpoints -->

Commit message: define transmissions in urdf

File: rover_description/arm/arm.xacro (robot description, xacro)
@@ -63,4 +63,16 @@
         </joint>
     </xacro:macro>
+    <xacro:macro name="transmissions" params="name">
+        <transmission name="trans_${name}">
+            <type>transmission_interface/SimpleTransmission</type>
+            <joint name="${name}">
+                <hardwareInterface>hardware_interface/EffortJointInterface</hardwareInterface>
+            </joint>
+            <actuator name="${name}_motor">
+                <hardwareInterface>hardware_interface/EffortJointInterface</hardwareInterface>
+                <mechanicalReduction>1</mechanicalReduction>
+            </actuator>
+        </transmission>
+    </xacro:macro>
     <link name="chassisToa">
         <xacro:link-visual fileName="chassis-a.stl" x="0" y="0" z="0" col="red" r="1" g="0" b="0" />
@@ -104,3 +116,14 @@
     <xacro:joints name="joint_e" parent="dToe" child="eTof" origin_x="-2.30884" origin_y="-14.2085" origin_z="9.01643" axis_x="1" lower="-2.68" upper="2.68" />
     <xacro:joints name="joint_f" parent="eTof" child="hand" origin_x="-0.817441" origin_y="0.678501" origin_z="-6.45623" axis_z="1" lower="-3.14" upper="3.14" />
+    <xacro:transmissions name="joint_a" />
+    <xacro:transmissions name="joint_b" />
+    <xacro:transmissions name="joint_c" />
+    <xacro:transmissions name="joint_d" />
+    <xacro:transmissions name="joint_e" />
+    <xacro:transmissions name="joint_f" />
+    <gazebo>
+        <plugin name="gazebo_ros_control">
+            <robotNamespace>/</robotNamespace>
+        </plugin>
+    </gazebo>
 </robot>

Commit message: gazebo integration with arm

File: rover_description/arm/arm.xacro (robot description, xacro)
@@ -15,8 +15,10 @@
     </xacro:macro>
     <xacro:macro name="link-inertial" params="x:=0 y:=0 z:=0 roll:=0 pitch:=0 yaw:=0 mass ixx iyy izz ixy:=0 iyz:=0 ixz:=0">
-        <origin xyz="${x} ${y} ${z}" rpy="${roll} ${pitch} ${yaw}" />
-        <!-- mass in kg -->
-        <mass value="${mass}" />
-        <inertia ixx="${ixx}" iyy="${iyy}" izz="${izz}" ixy="${ixy}" iyz="${iyz}" ixz="${ixz}" />
+        <inertial>
+            <origin xyz="${x} ${y} ${z}" rpy="${roll} ${pitch} ${yaw}" />
+            <!-- mass in kg -->
+            <mass value="${mass}" />
+            <inertia ixx="${ixx}" iyy="${iyy}" izz="${izz}" ixy="${ixy}" iyz="${iyz}" ixz="${ixz}" />
+        </inertial>
     </xacro:macro>
     <!-- defines a cylinder collision object with two endpoints -->
@@ -53,5 +55,5 @@
         </collision>
     </xacro:macro>
-    <xacro:macro name="joints" params="name type:=revolute parent child origin_x origin_y origin_z axis_x:=0 axis_y:=0 axis_z:=0 lower upper">
+    <xacro:macro name="joints" params="name type:=revolute parent child origin_x origin_y origin_z axis_x:=0 axis_y:=0 axis_z:=0 lower upper damp:=1">
         <joint name="${name}" type="${type}">
             <origin xyz="${origin_x} ${origin_y} ${origin_z}" rpy="0 0 0" />
@@ -61,6 +63,15 @@
             <!-- effort in N-m, velocity in rad/s -->
             <limit lower="${lower}" upper="${upper}" effort="30" velocity="1" />
+            <!-- damping in N-m-s/rad -->
+            <dynamics damping="${damp}" />
         </joint>
     </xacro:macro>
+    <xacro:macro name="gazebo_friction" params="link">
+      <gazebo reference="${link}">
+         <material>Gazebo/White</material>
+         <mu1>0.2</mu1>
+         <mu2>0.2</mu2>
+      </gazebo>
+   </xacro:macro>
     <xacro:macro name="transmissions" params="name">
         <transmission name="trans_${name}">
@@ -79,4 +90,5 @@
         <xacro:link-collision-cylinder radius="3.75" x1="0" y1="0" z1="-1.25" x2="0" y2="0" z2="-3.75" />
         <xacro:link-collision-cylinder radius="1.75" x1="-3.6467207" y1="3.6590503" z1="-0.6913988" x2="-3.6467207" y2="3.6590503" z2="-2.6913988" />
+        <xacro:link-inertial mass="2" ixx="0.3" iyy="0.3" izz="0.3" />
     </link>
     <link name="aTob">
@@ -84,4 +96,5 @@
         <xacro:link-collision-box y="-1.75" z="3" lx="2" ly="3" lz="6" />
         <xacro:link-collision-cylinder radius="2" x1="0" y1="0" z1="-0.25" x2="0" y2="0" z2="0.75" />
+        <xacro:link-inertial mass="2" ixx="0.3" iyy="0.3" izz="0.3" />
     </link>
     <link name="bToc">
@@ -90,8 +103,10 @@
         <xacro:link-collision-cylinder radius="1" x1="0" y1="23" z1="0" x2="5" y2="23" z2="0" />
         <xacro:link-collision-cylinder radius="1" x1="0" y1="0" z1="3.75" x2="0" y2="17" z2="3.75" roll="-0.3"/>
+        <xacro:link-inertial mass="2" ixx="0.3" iyy="0.3" izz="0.3" />
     </link>
     <link name="cTod">
         <xacro:link-visual fileName="c-d-blender.stl" x="0" y="0" z="0" col="green" r="0.43" g="1" b="0"/>
         <xacro:link-collision-cylinder radius="2" x1="3" y1="0" z1="0" x2="-5" y2="0" z2="0" />
+        <xacro:link-inertial mass="2" ixx="0.3" iyy="0.3" izz="0.3" />
     </link>
     <link name="dToe">
@@ -99,8 +114,10 @@
         <xacro:link-collision-box y="-7.6324" z="4.7693" lx="2.5" ly="20" lz="2.5" roll="-0.558505" />
         <xacro:link-collision-box x="1" y="-13.75" z="9.5" lx="3" ly="3" lz="6" roll="-0.558505" />
+        <xacro:link-inertial mass="2" ixx="0.3" iyy="0.3" izz="0.3" />
     </link>
     <link name="eTof">
         <xacro:link-visual fileName="e-f-blender.stl" x="0" y="0" z="0" col="violet" r="0.5" g="0" b="1" roll="1.67552" />
         <xacro:link-collision-cylinder radius="1" x1="-0.75" y1="0" z1="0" x2="-0.75" y2="0" z2="-6" />
+        <xacro:link-inertial mass="2" ixx="0.3" iyy="0.3" izz="0.3" />
     </link>
     <link name="hand">
@@ -109,5 +126,12 @@
         <xacro:link-collision-box y="-8" lx="3" ly="2" lz="4" />
         <xacro:link-collision-cylinder radius="0.75" x1="-1.5" y1="0" z1="-0.5" x2="-1.5" y2="-9" z2="-0.5" />
+        <xacro:link-inertial mass="2" ixx="0.3" iyy="0.3" izz="0.3" />
     </link>
+    <link name="world" />
+    <joint name="virtual_joint" type="fixed">
+        <parent link="world" />
+        <child link="chassisToa" />
+        <origin xyz="0 0 0" rpy="0 0 0" />
+    </joint>
     <xacro:joints name="joint_a" type="continuous" parent="chassisToa" child="aTob" origin_x="0" origin_y="0" origin_z="0" axis_z="1" lower="-3.14" upper="3.14" />
     <xacro:joints name="joint_b" parent="aTob" child="bToc" origin_x="0" origin_y="1.41293" origin_z="1.13303" axis_x="1" lower="0.035" upper="1.09" />
@@ -122,8 +146,13 @@
     <xacro:transmissions name="joint_e" />
     <xacro:transmissions name="joint_f" />
+    <xacro:gazebo_friction link="chassisToa" />
+    <xacro:gazebo_friction link="aTob" />
+    <xacro:gazebo_friction link="bToc" />
+    <xacro:gazebo_friction link="cTod" />
+    <xacro:gazebo_friction link="dToe" />
+    <xacro:gazebo_friction link="eTof" />
+    <xacro:gazebo_friction link="hand" />
     <gazebo>
-        <plugin name="gazebo_ros_control">
-            <robotNamespace>/</robotNamespace>
-        </plugin>
+        <plugin name="gazebo_ros_control" filename="libgazebo_ros_control.so" />
     </gazebo>
 </robot>

Commit message: disable self collision gazebo

File: rover_description/arm/arm.xacro (robot description, xacro)
@@ -67,10 +67,11 @@
         </joint>
     </xacro:macro>
-    <xacro:macro name="gazebo_friction" params="link">
-      <gazebo reference="${link}">
-         <material>Gazebo/White</material>
-         <mu1>0.2</mu1>
-         <mu2>0.2</mu2>
-      </gazebo>
+    <xacro:macro name="gazebo_ref" params="link">
+        <gazebo reference="${link}">
+            <material>Gazebo/White</material>
+            <mu1>0.2</mu1>
+            <mu2>0.2</mu2>
+            <selfCollide>false</selfCollide>
+        </gazebo>
    </xacro:macro>
     <xacro:macro name="transmissions" params="name">
@@ -146,11 +147,11 @@
     <xacro:transmissions name="joint_e" />
     <xacro:transmissions name="joint_f" />
-    <xacro:gazebo_friction link="chassisToa" />
-    <xacro:gazebo_friction link="aTob" />
-    <xacro:gazebo_friction link="bToc" />
-    <xacro:gazebo_friction link="cTod" />
-    <xacro:gazebo_friction link="dToe" />
-    <xacro:gazebo_friction link="eTof" />
-    <xacro:gazebo_friction link="hand" />
+    <xacro:gazebo_ref link="chassisToa" />
+    <xacro:gazebo_ref link="aTob" />
+    <xacro:gazebo_ref link="bToc" />
+    <xacro:gazebo_ref link="cTod" />
+    <xacro:gazebo_ref link="dToe" />
+    <xacro:gazebo_ref link="eTof" />
+    <xacro:gazebo_ref link="hand" />
     <gazebo>
         <plugin name="gazebo_ros_control" filename="libgazebo_ros_control.so" />

Commit message: Update arm.xacro with box and no collision with world link, regenerate package, set up position control in gazebo with action server

File: rover_description/arm/arm.xacro (robot description, xacro)
@@ -3,4 +3,7 @@
     <virtual_joint name="" type="fixed" parent_frame="world" child_link="chassis-a" />
     <xacro:property name="PI" value="3.141592" />
+    <xacro:property name="base_width" value="7" />
+    <xacro:property name="base_len" value="7" />
+    <xacro:property name="base_height" value="7" />
     <xacro:macro name="link-visual" params="fileName x y z col r g b roll:=0 pitch:=0 yaw:=0">
         <visual>
@@ -22,4 +25,10 @@
         </inertial>
     </xacro:macro>
+    <xacro:macro name="box_inertia" params="m w h d">
+    <inertial>
+      <mass value="${m}" />
+      <inertia ixx="${m / 12.0 * (d*d + h*h)}" ixy="0.0" ixz="0.0" iyy="${m / 12.0 * (w*w + h*h)}" iyz="0.0" izz="${m / 12.0 * (w*w + d*d)}" />
+    </inertial>
+  </xacro:macro>
     <!-- defines a cylinder collision object with two endpoints -->
     <xacro:macro name="link-collision-cylinder" params="radius x1 y1 z1 x2 y2 z2 roll:=0 pitch:=0 yaw:=0">
@@ -55,5 +64,5 @@
         </collision>
     </xacro:macro>
-    <xacro:macro name="joints" params="name type:=revolute parent child origin_x origin_y origin_z axis_x:=0 axis_y:=0 axis_z:=0 lower upper damp:=1">
+    <xacro:macro name="joints" params="name type:=revolute parent child origin_x origin_y origin_z axis_x:=0 axis_y:=0 axis_z:=0 lower upper damp:=1.0">
         <joint name="${name}" type="${type}">
             <origin xyz="${origin_x} ${origin_y} ${origin_z}" rpy="0 0 0" />
@@ -79,12 +88,30 @@
             <type>transmission_interface/SimpleTransmission</type>
             <joint name="${name}">
-                <hardwareInterface>hardware_interface/EffortJointInterface</hardwareInterface>
+                <hardwareInterface>hardware_interface/PositionJointInterface</hardwareInterface>
             </joint>
             <actuator name="${name}_motor">
-                <hardwareInterface>hardware_interface/EffortJointInterface</hardwareInterface>
+                <hardwareInterface>hardware_interface/PositionJointInterface</hardwareInterface>
                 <mechanicalReduction>1</mechanicalReduction>
             </actuator>
         </transmission>
     </xacro:macro>
+    <link name="base_link">
+        <xacro:box_inertia m="3.0" w="${base_len}" h="${base_width}" d="${base_height}" />
+        <visual>
+            <origin rpy="0 0 0" xyz="0 0 0" />
+            <geometry>
+                <box size="${base_len} ${base_width} ${base_height}" />
+            </geometry>
+            <material name="dark grey">
+                <color rgba="0.1 0.1 0.1 1" />
+            </material>
+        </visual>
+        <collision>
+            <origin rpy="0 0 0" xyz="0 0 0" />
+            <geometry>
+                <box size="${base_len} ${base_width} ${base_height}" />
+            </geometry>
+        </collision>
+    </link>
     <link name="chassisToa">
         <xacro:link-visual fileName="chassis-a.stl" x="0" y="0" z="0" col="red" r="1" g="0" b="0" />
@@ -137,7 +164,8 @@
     <joint name="virtual_joint" type="fixed">
         <parent link="world" />
-        <child link="chassisToa" />
-        <origin xyz="0 0 0" rpy="0 0 0" />
+        <child link="base_link" />
+        <origin xyz="0 0 ${base_height/2.0}" rpy="0 0 0" />
     </joint>
+    <xacro:joints name="base_link_connection" type="fixed" parent="base_link" child="chassisToa" origin_x="0" origin_y="5" origin_z="4" axis_z="0" lower="0" upper="0" />
     <xacro:joints name="joint_a" type="continuous" parent="chassisToa" child="aTob" origin_x="0" origin_y="0" origin_z="0" axis_z="1" lower="-3.14" upper="3.14" />
     <xacro:joints name="joint_b" parent="aTob" child="bToc" origin_x="0" origin_y="1.41293" origin_z="1.13303" axis_x="1" lower="0.035" upper="1.09" />

File: src/teleop/mrover_arm/config/gazebo_mrover_arm.urdf (robot description, URDF)
Before this commit: robot mrover_arm, 7 links, 6 joints
Links:
- added link base_link, mass 3.0; collision box size=7 7 7; visual box size=7 7 7
- added link world
- link aTob: mass 0.1 -> 0.5
- link bToc: mass 0.1 -> 0.5
- link cTod: mass 0.1 -> 0.5
- link chassisToa: mass 0.1 -> 0.5
- link dToe: mass 0.1 -> 0.5
- link eTof: mass 0.1 -> 0.5
- link hand: mass 0.1 -> 0.5
Joints:
- added joint base_link_connection: type fixed, parent base_link, child chassisToa, origin xyz=0 5 4 rpy=0 0 0, axis 0 0 0, limit lower=0 upper=0 effort=30 velocity=1
- added joint virtual_joint: type fixed, parent world, child base_link, origin xyz=0 0 3.5 rpy=0 0 0
