Commit message: Clean up new_arm stuff

File: rover_description/arm/arm.xacro (robot description, xacro)
@@ -64,7 +64,7 @@
         </collision>
     </xacro:macro>
-    <xacro:macro name="joints" params="name type:=revolute parent child origin_x origin_y origin_z axis_x:=0 axis_y:=0 axis_z:=0 lower upper damp:=1.0">
+    <xacro:macro name="joints" params="name type:=revolute parent child roll:=0 pitch:=0 yaw:=0 origin_x origin_y origin_z axis_x:=0 axis_y:=0 axis_z:=0 lower upper damp:=1.0" >
         <joint name="${name}" type="${type}">
-            <origin xyz="${origin_x} ${origin_y} ${origin_z}" rpy="0 0 0" />
+            <origin xyz="${origin_x} ${origin_y} ${origin_z}" rpy="${roll} ${pitch} ${yaw}" />
             <parent link="${parent}" />
             <child link="${child}" />
@@ -96,67 +96,46 @@
         </transmission>
     </xacro:macro>
-    <link name="base_link">
-        <xacro:box_inertia m="3.0" w="${base_len}" h="${base_width}" d="${base_height}" />
-        <visual>
-            <origin rpy="0 0 0" xyz="0 0 0" />
-            <geometry>
-                <box size="${base_len} ${base_width} ${base_height}" />
-            </geometry>
-            <material name="dark grey">
-                <color rgba="0.1 0.1 0.1 1" />
-            </material>
-        </visual>
-        <collision>
-            <origin rpy="0 0 0" xyz="0 0 0" />
-            <geometry>
-                <box size="${base_len} ${base_width} ${base_height}" />
-            </geometry>
-        </collision>
-    </link>
     <link name="chassisToa">
-        <xacro:link-visual fileName="chassis-a.stl" x="0" y="0" z="0" col="red" r="1" g="0" b="0" />
+        <xacro:link-visual fileName="chassis-a.stl" x="0" y="0" z="0" col="red" r="1" g="0" b="0"/>
         <xacro:link-collision-cylinder radius="3.75" x1="0" y1="0" z1="-1.25" x2="0" y2="0" z2="-3.75" />
-        <xacro:link-collision-cylinder radius="1.75" x1="-3.6467207" y1="3.6590503" z1="-0.6913988" x2="-3.6467207" y2="3.6590503" z2="-2.6913988" />
+        <xacro:link-collision-cylinder radius="1.75" x1="3.6467207" y1="3.6590503" z1="1" x2="3.6467207" y2="3.6590503" z2="-2.6913988" />
         <!-- calculated based on cylinder1 -->
         <xacro:link-inertial z="-2.5" mass="0.5" ixx="2.3" iyy="2.3" izz="3.5" />
     </link>
     <link name="aTob">
-        <xacro:link-visual fileName="a-b.stl" x="0" y="0" z="0" col="orange" r="1" g="0.43" b="0" />
+        <xacro:link-visual fileName="a-b.stl" x="0" y="0" z="0" col="orange" r="1" g="0.43" b="0" roll="0"/>
         <xacro:link-collision-box y="-1.75" z="3" lx="2" ly="3" lz="6" />
         <xacro:link-collision-cylinder radius="2" x1="0" y1="0" z1="-0.25" x2="0" y2="0" z2="0.75" />
-        <!-- box -->
         <xacro:link-inertial y="-1.75" z="3" mass="0.5" ixx="1.9" iyy="0.7" izz="0.5" />
     </link>
     <link name="bToc">
         <xacro:link-visual fileName="b-c.stl" x="0" y="0" z="0" col="yellow" r="1" g="1" b="0" roll="0"/>
-        <xacro:link-collision-box y="12" lx="3" ly="24" lz="3" />
-        <xacro:link-collision-cylinder radius="1" x1="0" y1="23" z1="0" x2="5" y2="23" z2="0" />
-        <xacro:link-collision-cylinder radius="1" x1="0" y1="0" z1="3.75" x2="0" y2="17" z2="3.75" roll="-0.3"/>
-        <!-- box -->
+        <xacro:link-collision-box y="9" z="5" lx="3" ly="24" lz="3" roll="0.48" />
+        <xacro:link-collision-cylinder radius="2" x1="-2" y1="20.25" z1="10.75" x2="4.5" y2="20.25" z2="10.75" />
+        <xacro:link-collision-cylinder radius="1" x1="0" y1="-2" z1="8.5" x2="0" y2="17" z2="8.5" roll="0.3" />
         <xacro:link-inertial y="12" mass="0.5" ixx="24" iyy="0.75" izz="24" />
     </link>
     <link name="cTod">
-        <xacro:link-visual fileName="c-d-blender.stl" x="0" y="0" z="0" col="green" r="0.43" g="1" b="0"/>
-        <xacro:link-collision-cylinder radius="2" x1="3" y1="0" z1="0" x2="-5" y2="0" z2="0" />
+        <xacro:link-visual fileName="c-d.stl" x="0" y="0" z="0" col="green" r="0.43" g="1" b="0"/>
+        <xacro:link-collision-cylinder radius="3.75" x1="-4.5" y1="0" z1="-2.5" x2="-4.5" y2="0" z2="3" roll="-0.17"/>
         <xacro:link-inertial x="-1" mass="0.5" ixx="3.2" iyy="3.2" izz="16" />
     </link>
     <link name="dToe">
-        <xacro:link-visual fileName="d-e-blender.stl" x="0" y="0" z="0" col="blue" r="0" g="0" b="1"/>
-        <xacro:link-collision-box y="-7.6324" z="4.7693" lx="2.5" ly="20" lz="2.5" roll="-0.558505" />
-        <xacro:link-collision-box x="1" y="-13.75" z="9.5" lx="3" ly="3" lz="6" roll="-0.558505" />
-        <!-- box1 -->
+        <xacro:link-visual fileName="d-e.stl" x="0" y="0" z="0" col="blue" r="0" g="0" b="1" pitch="0" roll="0"/>
+        <xacro:link-collision-box y="0" z="-7" lx="4" ly="20" lz="4" roll="${(-PI/2.0)+0.05}"/>
+        <xacro:link-collision-cylinder radius="2.5" x1="-3" y1="0" z1="-17" x2="3" y2="0" z2="-17" />
         <xacro:link-inertial y="-7.6324" z="4.7693" roll="-0.558505" mass="0.5" ixx="17" iyy="0.5" izz="17" />
     </link>
     <link name="eTof">
-        <xacro:link-visual fileName="e-f-blender.stl" x="0" y="0" z="0" col="violet" r="0.5" g="0" b="1" roll="1.67552" />
-        <xacro:link-collision-cylinder radius="1" x1="-0.75" y1="0" z1="0" x2="-0.75" y2="0" z2="-6" />
+        <xacro:link-visual fileName="e-f.stl" x="0" y="0" z="0" col="violet" r="0.5" g="0" b="1" roll="0" />
+        <xacro:link-collision-cylinder radius="3" x1="3" y1="1.8" z1="0" x2="-6.5" y2="1.8" z2="0" />
         <xacro:link-inertial z="-3" mass="0.5" ixx="1.6" iyy="1.6" izz="0.25" />
     </link>
     <link name="hand">
-        <xacro:link-visual fileName="hand.stl" x="0" y="0" z="0" col="pink" r="1" g="0" b="1" yaw="${PI}" roll="-1.67552"/>
-        <xacro:link-collision-box z="-2.5" lx="7" ly="2" lz="7" />
-        <xacro:link-collision-box y="-8" lx="3" ly="2" lz="4" />
-        <xacro:link-collision-cylinder radius="0.75" x1="-1.5" y1="0" z1="-0.5" x2="-1.5" y2="-9" z2="-0.5" />
-        <!-- box1 -->
+        <xacro:link-visual fileName="hand.stl" x="0" y="0" z="0" col="pink" r="1" g="0" b="1"/>
+        <xacro:link-collision-box x="-2.25" y="1" z="0.5" lx="8" ly="3.5" lz="8.5" roll="${PI/2.0}"/>
+        <xacro:link-collision-box z="8.75" y="3.5" x="-1" lx="3.5" ly="3.5" lz="5" roll="${PI/2.0}"/>
+        <xacro:link-collision-cylinder radius="0.75" x1="0" y1="2.3" z1="0" x2="0" y2="2.3" z2="9"/>
+        <xacro:link-collision-box x="-1.6" y="-1.5" z="-2" lx="1" ly="2.5" lz="2.5"/>
         <xacro:link-inertial z="-2.5" mass="0.5" ixx="2.2" iyy="4" izz="2.2" />
     </link>
@@ -164,14 +143,13 @@
     <joint name="virtual_joint" type="fixed">
         <parent link="world" />
-        <child link="base_link" />
+        <child link="chassisToa" />
         <origin xyz="0 0 ${base_height/2.0}" rpy="0 0 0" />
     </joint>
-    <xacro:joints name="base_link_connection" type="fixed" parent="base_link" child="chassisToa" origin_x="0" origin_y="5" origin_z="4" axis_z="0" lower="0" upper="0" />
     <xacro:joints name="joint_a" type="continuous" parent="chassisToa" child="aTob" origin_x="0" origin_y="0" origin_z="0" axis_z="1" lower="-3.14" upper="3.14" />
-    <xacro:joints name="joint_b" parent="aTob" child="bToc" origin_x="0" origin_y="1.41293" origin_z="1.13303" axis_x="1" lower="0.035" upper="1.09" />
-    <xacro:joints name="joint_c" parent="bToc" child="cTod" origin_x="-4.59961" origin_y="22.83397" origin_z="0.38119" axis_x="1" lower="-3.01" upper="2.73" />
-    <xacro:joints name="joint_d" parent="cTod" child="dToe" origin_x="0" origin_y="-1.4699" origin_z="0.963976" axis_z="-0.52992" axis_y="0.84805" lower="-3.14" upper="3.14" />
-    <xacro:joints name="joint_e" parent="dToe" child="eTof" origin_x="-2.30884" origin_y="-14.2085" origin_z="9.01643" axis_x="1" lower="-2.68" upper="2.68" />
-    <xacro:joints name="joint_f" parent="eTof" child="hand" origin_x="-0.817441" origin_y="0.678501" origin_z="-6.45623" axis_z="1" lower="-3.14" upper="3.14" />
+    <xacro:joints name="joint_b" parent="aTob" child="bToc" origin_x="0" origin_y="1.33" origin_z="0.99" axis_x="1" lower="-1.064651" upper="0" roll="0.593412"/>
+    <xacro:joints name="joint_c" parent="bToc" child="cTod" origin_x="0" origin_y="20.11" origin_z="10.75" axis_x="1" lower="-0.087267" upper="4.886922" roll="-0.436332"/>
+    <xacro:joints name="joint_d" parent="cTod" child="dToe" origin_x="-4.4" origin_y="-0.42" origin_z="-2.535" axis_z="1" axis_y="0" lower="-3.14" upper="3.14" roll="-0.15708" pitch="-0.0174533" yaw="0" />
+    <xacro:joints name="joint_e" parent="dToe" child="eTof" origin_x="2.55" origin_y="0.2" origin_z="-17" axis_y="1" lower="-3.59538" upper="0.610865" roll="0" pitch="0" yaw="-1.649336"/>
+    <xacro:joints name="joint_f" parent="eTof" child="hand" origin_x="-6.3" origin_y="1.75" origin_z="0" axis_x="1" lower="-0.523599" upper="6.28" />
     <xacro:transmissions name="joint_a" />
     <xacro:transmissions name="joint_b" />

Commit message: Add pedestal to bottom of arm for now, set up new mrover_arm package and remove joint_f from motion planning since it has no encoder

File: rover_description/arm/arm.xacro (robot description, xacro)
@@ -5,5 +5,5 @@
     <xacro:property name="base_width" value="7" />
     <xacro:property name="base_len" value="7" />
-    <xacro:property name="base_height" value="7" />
+    <xacro:property name="base_height" value="19" />
     <xacro:macro name="link-visual" params="fileName x y z col r g b roll:=0 pitch:=0 yaw:=0">
         <visual>
@@ -96,4 +96,22 @@
         </transmission>
     </xacro:macro>
+    <link name="base_link">
+        <xacro:box_inertia m="3.0" w="${base_len}" h="${base_width}" d="${base_height}" />
+        <visual>
+            <origin rpy="0 0 0" xyz="0 0 0" />
+            <geometry>
+                <box size="${base_len} ${base_width} ${base_height}" />
+            </geometry>
+            <material name="dark grey">
+                <color rgba="0.1 0.1 0.1 1" />
+            </material>
+        </visual>
+        <collision>
+            <origin rpy="0 0 0" xyz="0 0 0" />
+            <geometry>
+                <box size="${base_len} ${base_width} ${base_height}" />
+            </geometry>
+        </collision>
+    </link>
     <link name="chassisToa">
         <xacro:link-visual fileName="chassis-a.stl" x="0" y="0" z="0" col="red" r="1" g="0" b="0"/>
@@ -143,7 +161,8 @@
     <joint name="virtual_joint" type="fixed">
         <parent link="world" />
-        <child link="chassisToa" />
+        <child link="base_link" />
         <origin xyz="0 0 ${base_height/2.0}" rpy="0 0 0" />
     </joint>
+    <xacro:joints name="base_link_connection" type="fixed" parent="base_link" child="chassisToa" origin_x="0" origin_y="5" origin_z="10" axis_z="0" lower="0" upper="0" />
     <xacro:joints name="joint_a" type="continuous" parent="chassisToa" child="aTob" origin_x="0" origin_y="0" origin_z="0" axis_z="1" lower="-3.14" upper="3.14" />
     <xacro:joints name="joint_b" parent="aTob" child="bToc" origin_x="0" origin_y="1.33" origin_z="0.99" axis_x="1" lower="-1.064651" upper="0" roll="0.593412"/>

File: src/teleop/mrover_arm/config/gazebo_mrover_arm.urdf (robot description, URDF)
Before this commit: robot mrover_arm, 9 links, 8 joints
Links:
- link bToc: geometry collision box size=3 24 3; collision cylinder length=19.0 radius=1
- link base_link: geometry collision box size=7 7 19; visual box size=7 7 19
- link cTod: geometry collision cylinder length=5.5 radius=3.75; visual mesh filename=package://mrover/rover_description/arm/c-d.stl
- link chassisToa: geometry collision cylinder length=2.5 radius=3.75; collision cylinder length=3.6913988 radius=1.75
- link dToe: geometry collision box size=4 20 4; collision cylinder length=6.0 radius=2.5
- link eTof: geometry collision cylinder length=9.5 radius=3; visual mesh filename=package://mrover/rover_description/arm/e-f.stl
- link hand: geometry collision box size=1 2.5 2.5; collision box size=3.5 3.5 5
Joints:
- joint base_link_connection: origin xyz=0 5 4 rpy=0 0 0 -> xyz=0 5 10 rpy=0 0 0
- joint joint_b: limit lower=0.035 upper=1.09 effort=30 velocity=1 -> lower=-1.064651 upper=0 effort=30 velocity=1; origin xyz=0 1.41293 1.13303 rpy=0 0 0 -> xyz=0 1.33 0.99 rpy=0.593412 0 0
- joint joint_c: limit lower=-3.01 upper=2.73 effort=30 velocity=1 -> lower=-0.087267 upper=4.886922 effort=30 velocity=1; origin xyz=-4.59961 22.83397 0.38119 rpy=0 0 0 -> xyz=0 20.11 10.75 rpy=-0.436332 0 0
- joint joint_d: axis 0 0.84805 -0.52992 -> 0 0 1; origin xyz=0 -1.4699 0.963976 rpy=0 0 0 -> xyz=-4.4 -0.42 -2.535 rpy=-0.15708 -0.0174533 0
- joint joint_e: axis 1 0 0 -> 0 1 0; limit lower=-2.68 upper=2.68 effort=30 velocity=1 -> lower=-3.59538 upper=0.610865 effort=30 velocity=1; origin xyz=-2.30884 -14.2085 9.01643 rpy=0 0 0 -> xyz=2.55 0.2 -17 rpy=0 0 -1.649336
- joint joint_f: axis 0 0 1 -> 1 0 0; limit lower=-3.14 upper=3.14 effort=30 velocity=1 -> lower=-0.523599 upper=6.28 effort=30 velocity=1; origin xyz=-0.817441 0.678501 -6.45623 rpy=0 0 0 -> xyz=-6.3 1.75 0 rpy=0 0 0
- joint virtual_joint: origin xyz=0 0 3.5 rpy=0 0 0 -> xyz=0 0 9.5 rpy=0 0 0

Commit message: Add rover to URDF

File: rover_description/arm/arm.xacro (robot description, xacro)
@@ -98,17 +98,9 @@
     <link name="base_link">
         <xacro:box_inertia m="3.0" w="${base_len}" h="${base_width}" d="${base_height}" />
-        <visual>
-            <origin rpy="0 0 0" xyz="0 0 0" />
+        <xacro:link-visual fileName="rover.stl" x="0" y="0" z="-9.5" col="red" r="1" g="1" b="1"/>
+        <collision>
+            <origin rpy="0 0 0" xyz="0 0 -9.5" />
             <geometry>
-                <box size="${base_len} ${base_width} ${base_height}" />
-            </geometry>
-            <material name="dark grey">
-                <color rgba="0.1 0.1 0.1 1" />
-            </material>
-        </visual>
-        <collision>
-            <origin rpy="0 0 0" xyz="0 0 0" />
-            <geometry>
-                <box size="${base_len} ${base_width} ${base_height}" />
+                <mesh filename="package://mrover/rover_description/arm/rover.stl" />
             </geometry>
         </collision>
@@ -164,5 +156,5 @@
         <origin xyz="0 0 ${base_height/2.0}" rpy="0 0 0" />
     </joint>
-    <xacro:joints name="base_link_connection" type="fixed" parent="base_link" child="chassisToa" origin_x="0" origin_y="5" origin_z="10" axis_z="0" lower="0" upper="0" />
+    <xacro:joints name="base_link_connection" type="fixed" parent="base_link" child="chassisToa" origin_x="0" origin_y="15.55" origin_z="11" axis_z="0" lower="0" upper="0" />
     <xacro:joints name="joint_a" type="continuous" parent="chassisToa" child="aTob" origin_x="0" origin_y="0" origin_z="0" axis_z="1" lower="-3.14" upper="3.14" />
     <xacro:joints name="joint_b" parent="aTob" child="bToc" origin_x="0" origin_y="1.33" origin_z="0.99" axis_x="1" lower="-1.064651" upper="0" roll="0.593412"/>

Commit message: low res rover model

File: rover_description/arm/arm.xacro (robot description, xacro)
@@ -98,9 +98,9 @@
     <link name="base_link">
         <xacro:box_inertia m="3.0" w="${base_len}" h="${base_width}" d="${base_height}" />
-        <xacro:link-visual fileName="rover.stl" x="0" y="0" z="-9.5" col="red" r="1" g="1" b="1"/>
+        <xacro:link-visual fileName="rover_low_poly.stl" x="0" y="0" z="-9.5" col="red" r="1" g="1" b="1"/>
         <collision>
             <origin rpy="0 0 0" xyz="0 0 -9.5" />
             <geometry>
-                <mesh filename="package://mrover/rover_description/arm/rover.stl" />
+                <mesh filename="package://mrover/rover_description/arm/rover_low_poly.stl" />
             </geometry>
         </collision>

Commit message: Generate package for arm with rover viz, need to fix bc link collisions:

File: rover_description/arm/arm.xacro (robot description, xacro)
@@ -98,9 +98,9 @@
     <link name="base_link">
         <xacro:box_inertia m="3.0" w="${base_len}" h="${base_width}" d="${base_height}" />
-        <xacro:link-visual fileName="rover_low_poly.stl" x="0" y="0" z="-9.5" col="red" r="1" g="1" b="1"/>
+        <xacro:link-visual fileName="rover.stl" x="0" y="0" z="-9.5" col="red" r="1" g="1" b="1"/>
         <collision>
             <origin rpy="0 0 0" xyz="0 0 -9.5" />
             <geometry>
-                <mesh filename="package://mrover/rover_description/arm/rover_low_poly.stl" />
+                <mesh filename="package://mrover/rover_description/arm/rover.stl" />
             </geometry>
         </collision>

File: src/teleop/mrover_arm/config/gazebo_mrover_arm.urdf (robot description, URDF)
Before this commit: robot mrover_arm, 9 links, 8 joints
Links:
- link base_link: geometry collision mesh filename=package://mrover/rover_description/arm/rover.stl; visual mesh filename=package://mrover/rover_description/arm/rover.stl
Joints:
- joint base_link_connection: origin xyz=0 5 10 rpy=0 0 0 -> xyz=0 15.55 11 rpy=0 0 0

Commit message: Fix issues with bc link colliding/not colliding with the rover.

File: rover_description/arm/arm.xacro (robot description, xacro)
@@ -109,5 +109,5 @@
         <xacro:link-visual fileName="chassis-a.stl" x="0" y="0" z="0" col="red" r="1" g="0" b="0"/>
         <xacro:link-collision-cylinder radius="3.75" x1="0" y1="0" z1="-1.25" x2="0" y2="0" z2="-3.75" />
-        <xacro:link-collision-cylinder radius="1.75" x1="3.6467207" y1="3.6590503" z1="0" x2="3.6467207" y2="3.6590503" z2="-2.6913988" />
+        <xacro:link-collision-cylinder radius="1.75" x1="3.6467207" y1="3.6590503" z1="-0.75" x2="3.6467207" y2="3.6590503" z2="-2.6913988" />
         <!-- calculated based on cylinder1 -->
         <xacro:link-inertial z="-2.5" mass="0.5" ixx="2.3" iyy="2.3" izz="3.5" />

File: src/teleop/mrover_arm/config/gazebo_mrover_arm.urdf (robot description, URDF)
Before this commit: robot mrover_arm, 9 links, 8 joints
Links:
- link bToc: geometry collision box size=2 20 2; collision cylinder length=19.0 radius=1
- link chassisToa: geometry collision cylinder length=1.9413988 radius=1.75; collision cylinder length=2.5 radius=3.75
