Commit message: MoveIt Code for 2023 Arm URDF with Rover Model (#355)
* Arm xacro urdf

* Got arm components to display in rviz, still messed up, need to blenderize stl files bc axes are weird

* Commit progress

* Urdf up to joint E

* visuals of URDF complete

* Define cylinder and box collision xacros

* Add collision models

* Add one collision box and adjust some other, add moveit to Cmake and package.xml

* Clean up old blends and stl files, clean up rviz arm config

* Add stl files to lfs

* Fix moveit dependencies I think

* Fix moveit dependencies this time maybe

* Revert back to having all rospack list-names packages in cmake and package.xml

* Add cylinder for linear actuator to arm urdf

* Change stl files to lfs objects I think

* generated arm package

* xacro link name changes

* Rebuild mrover_arm package

* Regenerated moveit package with controllers for joint groups

* define urdf macro for inertial

* define transmissions in urdf

* Add untested action server for arm joint trajectories

* gazebo integration with arm

* add arm_trajectory server and fake arm launch file, not working/tested rn

* disable self collision gazebo

* update inertials

* Update arm.xacro with box and no collision with world link, regenerate package, set up position control in gazebo with action server

* Update launch file for arm, regenerate package again with new config files and such

* Add lots of comments

* remove unused arg from arm_gazebo launch

* Remove unused arg in arm_gazebo_sim

* remove mrover_arm2

* Make changes based on Cam's suggestions. Add params to arm_gazebo_sim.launch file

* Added some things

* Align all visual geometry

* collision models for links b-c and c-d

* adjust c-d collision

* Finish 2023 URDF.

* Clean up new_arm stuff

* Add pedestal to bottom of arm for now, set up new mrover_arm package and remove joint_f from motion planning since it has no encoder

* Add rover to URDF

* low res rover model

* Generate package for arm with rover viz, need to fix bc link collisions:

* Make bc link collision box tighter

* Fix issues with bc link colliding/not colliding with the rover.

* Style and rviz config file for moveit package fixed

* minor changes to action server

* make mypy happy

* Delete test.txt

---------

Co-authored-by: bli76 <32941474+bli76@users.noreply.github.com>

File: rover_description/arm/arm.xacro (robot description, xacro)
@@ -3,4 +3,7 @@
     <virtual_joint name="" type="fixed" parent_frame="world" child_link="chassis-a" />
     <xacro:property name="PI" value="3.141592" />
+    <xacro:property name="base_width" value="7" />
+    <xacro:property name="base_len" value="7" />
+    <xacro:property name="base_height" value="19" />
     <xacro:macro name="link-visual" params="fileName x y z col r g b roll:=0 pitch:=0 yaw:=0">
         <visual>
@@ -14,4 +17,18 @@
         </visual>
     </xacro:macro>
+    <xacro:macro name="link-inertial" params="x:=0 y:=0 z:=0 roll:=0 pitch:=0 yaw:=0 mass ixx iyy izz ixy:=0 iyz:=0 ixz:=0">
+        <inertial>
+            <origin xyz="${x} ${y} ${z}" rpy="${roll} ${pitch} ${yaw}" />
+            <!-- mass in kg -->
+            <mass value="${mass}" />
+            <inertia ixx="${ixx}" iyy="${iyy}" izz="${izz}" ixy="${ixy}" iyz="${iyz}" ixz="${ixz}" />
+        </inertial>
+    </xacro:macro>
+    <xacro:macro name="box_inertia" params="m w h d">
+    <inertial>
+      <mass value="${m}" />
+      <inertia ixx="${m / 12.0 * (d*d + h*h)}" ixy="0.0" ixz="0.0" iyy="${m / 12.0 * (w*w + h*h)}" iyz="0.0" izz="${m / 12.0 * (w*w + d*d)}" />
+    </inertial>
+  </xacro:macro>
     <!-- defines a cylinder collision object with two endpoints -->
     <xacro:macro name="link-collision-cylinder" params="radius x1 y1 z1 x2 y2 z2 roll:=0 pitch:=0 yaw:=0">
@@ -47,7 +64,7 @@
         </collision>
     </xacro:macro>
-    <xacro:macro name="joints" params="name type:=revolute parent child origin_x origin_y origin_z axis_x:=0 axis_y:=0 axis_z:=0 lower upper">
+    <xacro:macro name="joints" params="name type:=revolute parent child roll:=0 pitch:=0 yaw:=0 origin_x origin_y origin_z axis_x:=0 axis_y:=0 axis_z:=0 lower upper damp:=1.0" >
         <joint name="${name}" type="${type}">
-            <origin xyz="${origin_x} ${origin_y} ${origin_z}" rpy="0 0 0" />
+            <origin xyz="${origin_x} ${origin_y} ${origin_z}" rpy="${roll} ${pitch} ${yaw}" />
             <parent link="${parent}" />
             <child link="${child}" />
@@ -55,46 +72,110 @@
             <!-- effort in N-m, velocity in rad/s -->
             <limit lower="${lower}" upper="${upper}" effort="30" velocity="1" />
+            <!-- damping in N-m-s/rad -->
+            <dynamics damping="${damp}" />
         </joint>
     </xacro:macro>
-    <link name="chassis-a">
-        <xacro:link-visual fileName="chassis-a.stl" x="0" y="0" z="0" col="red" r="1" g="0" b="0" />
+    <xacro:macro name="gazebo_ref" params="link">
+        <gazebo reference="${link}">
+            <material>Gazebo/White</material>
+            <mu1>0.2</mu1>
+            <mu2>0.2</mu2>
+            <selfCollide>false</selfCollide>
+        </gazebo>
+   </xacro:macro>
+    <xacro:macro name="transmissions" params="name">
+        <transmission name="trans_${name}">
+            <type>transmission_interface/SimpleTransmission</type>
+            <joint name="${name}">
+                <hardwareInterface>hardware_interface/PositionJointInterface</hardwareInterface>
+            </joint>
+            <actuator name="${name}_motor">
+                <hardwareInterface>hardware_interface/PositionJointInterface</hardwareInterface>
+                <mechanicalReduction>1</mechanicalReduction>
+            </actuator>
+        </transmission>
+    </xacro:macro>
+    <link name="base_link">
+        <xacro:box_inertia m="3.0" w="${base_len}" h="${base_width}" d="${base_height}" />
+        <xacro:link-visual fileName="rover.stl" x="0" y="0" z="-9.5" col="red" r="1" g="1" b="1"/>
+        <collision>
+            <origin rpy="0 0 0" xyz="0 0 -9.5" />
+            <geometry>
+                <mesh filename="package://mrover/rover_description/arm/rover.stl" />
+            </geometry>
+        </collision>
+    </link>
+    <link name="chassisToa">
+        <xacro:link-visual fileName="chassis-a.stl" x="0" y="0" z="0" col="red" r="1" g="0" b="0"/>
         <xacro:link-collision-cylinder radius="3.75" x1="0" y1="0" z1="-1.25" x2="0" y2="0" z2="-3.75" />
-        <xacro:link-collision-cylinder radius="1.75" x1="-3.6467207" y1="3.6590503" z1="-0.6913988" x2="-3.6467207" y2="3.6590503" z2="-2.6913988" />
+        <xacro:link-collision-cylinder radius="1.75" x1="3.6467207" y1="3.6590503" z1="-0.75" x2="3.6467207" y2="3.6590503" z2="-2.6913988" />
+        <!-- calculated based on cylinder1 -->
+        <xacro:link-inertial z="-2.5" mass="0.5" ixx="2.3" iyy="2.3" izz="3.5" />
     </link>
-    <link name="a-b">
-        <xacro:link-visual fileName="a-b.stl" x="0" y="0" z="0" col="orange" r="1" g="0.43" b="0" />
+    <link name="aTob">
+        <xacro:link-visual fileName="a-b.stl" x="0" y="0" z="0" col="orange" r="1" g="0.43" b="0" roll="0"/>
         <xacro:link-collision-box y="-1.75" z="3" lx="2" ly="3" lz="6" />
         <xacro:link-collision-cylinder radius="2" x1="0" y1="0" z1="-0.25" x2="0" y2="0" z2="0.75" />
+        <xacro:link-inertial y="-1.75" z="3" mass="0.5" ixx="1.9" iyy="0.7" izz="0.5" />
     </link>
-    <link name="b-c">
+    <link name="bToc">
         <xacro:link-visual fileName="b-c.stl" x="0" y="0" z="0" col="yellow" r="1" g="1" b="0" roll="0"/>
-        <xacro:link-collision-box y="12" lx="3" ly="24" lz="3" />
-        <xacro:link-collision-cylinder radius="1" x1="0" y1="23" z1="0" x2="5" y2="23" z2="0" />
-        <xacro:link-collision-cylinder radius="1" x1="0" y1="0" z1="3.75" x2="0" y2="17" z2="3.75" roll="-0.3"/>
+        <xacro:link-collision-box y="9" z="5" lx="2" ly="20" lz="2" roll="0.48" />
+        <xacro:link-collision-cylinder radius="2" x1="-2" y1="20.25" z1="10.75" x2="4.5" y2="20.25" z2="10.75" />
+        <xacro:link-collision-cylinder radius="1" x1="0" y1="-2" z1="8.5" x2="0" y2="17" z2="8.5" roll="0.3" />
+        <xacro:link-inertial y="12" mass="0.5" ixx="24" iyy="0.75" izz="24" />
     </link>
-    <link name="c-d">
-        <xacro:link-visual fileName="c-d-blender.stl" x="0" y="0" z="0" col="green" r="0.43" g="1" b="0"/>
-        <xacro:link-collision-cylinder radius="2" x1="3" y1="0" z1="0" x2="-5" y2="0" z2="0" />
+    <link name="cTod">
+        <xacro:link-visual fileName="c-d.stl" x="0" y="0" z="0" col="green" r="0.43" g="1" b="0"/>
+        <xacro:link-collision-cylinder radius="3.75" x1="-4.5" y1="0" z1="-2.5" x2="-4.5" y2="0" z2="3" roll="-0.17"/>
+        <xacro:link-inertial x="-1" mass="0.5" ixx="3.2" iyy="3.2" izz="16" />
     </link>
-    <link name="d-e">
-        <xacro:link-visual fileName="d-e-blender.stl" x="0" y="0" z="0" col="blue" r="0" g="0" b="1"/>
-        <xacro:link-collision-box y="-7.6324" z="4.7693" lx="2.5" ly="20" lz="2.5" roll="-0.558505" />
-        <xacro:link-collision-box x="1" y="-13.75" z="9.5" lx="3" ly="3" lz="6" roll="-0.558505" />
+    <link name="dToe">
+        <xacro:link-visual fileName="d-e.stl" x="0" y="0" z="0" col="blue" r="0" g="0" b="1" pitch="0" roll="0"/>
+        <xacro:link-collision-box y="0" z="-7" lx="4" ly="20" lz="4" roll="${(-PI/2.0)+0.05}"/>
+        <xacro:link-collision-cylinder radius="2.5" x1="-3" y1="0" z1="-17" x2="3" y2="0" z2="-17" />
+        <xacro:link-inertial y="-7.6324" z="4.7693" roll="-0.558505" mass="0.5" ixx="17" iyy="0.5" izz="17" />
     </link>
-    <link name="e-f">
-        <xacro:link-visual fileName="e-f-blender.stl" x="0" y="0" z="0" col="violet" r="0.5" g="0" b="1" roll="1.67552" />
-        <xacro:link-collision-cylinder radius="1" x1="-0.75" y1="0" z1="0" x2="-0.75" y2="0" z2="-6" />
+    <link name="eTof">
+        <xacro:link-visual fileName="e-f.stl" x="0" y="0" z="0" col="violet" r="0.5" g="0" b="1" roll="0" />
+        <xacro:link-collision-cylinder radius="3" x1="3" y1="1.8" z1="0" x2="-6.5" y2="1.8" z2="0" />
+        <xacro:link-inertial z="-3" mass="0.5" ixx="1.6" iyy="1.6" izz="0.25" />
     </link>
     <link name="hand">
-        <xacro:link-visual fileName="hand.stl" x="0" y="0" z="0" col="pink" r="1" g="0" b="1" yaw="${PI}" roll="-1.67552"/>
-        <xacro:link-collision-box z="-2.5" lx="7" ly="2" lz="7" />
-        <xacro:link-collision-box y="-8" lx="3" ly="2" lz="4" />
-        <xacro:link-collision-cylinder radius="0.75" x1="-1.5" y1="0" z1="-0.5" x2="-1.5" y2="-9" z2="-0.5" />
+        <xacro:link-visual fileName="hand.stl" x="0" y="0" z="0" col="pink" r="1" g="0" b="1"/>
+        <xacro:link-collision-box x="-2.25" y="1" z="0.5" lx="8" ly="3.5" lz="8.5" roll="${PI/2.0}"/>
+        <xacro:link-collision-box z="8.75" y="3.5" x="-1" lx="3.5" ly="3.5" lz="5" roll="${PI/2.0}"/>
+        <xacro:link-collision-cylinder radius="0.75" x1="0" y1="2.3" z1="0" x2="0" y2="2.3" z2="9"/>
+        <xacro:link-collision-box x="-1.6" y="-1.5" z="-2" lx="1" ly="2.5" lz="2.5"/>
+        <xacro:link-inertial z="-2.5" mass="0.5" ixx="2.2" iyy="4" izz="2.2" />
     </link>
-    <xacro:joints name="joint_a" type="continuous" parent="chassis-a" child="a-b" origin_x="0" origin_y="0" origin_z="0" axis_z="1" lower="-3.14" upper="3.14" />
-    <xacro:joints name="joint_b" parent="a-b" child="b-c" origin_x="0" origin_y="1.41293" origin_z="1.13303" axis_x="1" lower="0.035" upper="1.09" />
-    <xacro:joints name="joint_c" parent="b-c" child="c-d" origin_x="-4.59961" origin_y="22.83397" origin_z="0.38119" axis_x="1" lower="-3.01" upper="2.73" />
-    <xacro:joints name="joint_d" parent="c-d" child="d-e" origin_x="0" origin_y="-1.4699" origin_z="0.963976" axis_z="-0.52992" axis_y="0.84805" lower="-3.14" upper="3.14" />
-    <xacro:joints name="joint_e" parent="d-e" child="e-f" origin_x="-2.30884" origin_y="-14.2085" origin_z="9.01643" axis_x="1" lower="-2.68" upper="2.68" />
-    <xacro:joints name="joint_f" parent="e-f" child="hand" origin_x="-0.817441" origin_y="0.678501" origin_z="-6.45623" axis_z="1" lower="-3.14" upper="3.14" />
+    <link name="world" />
+    <joint name="virtual_joint" type="fixed">
+        <parent link="world" />
+        <child link="base_link" />
+        <origin xyz="0 0 ${base_height/2.0}" rpy="0 0 0" />
+    </joint>
+    <xacro:joints name="base_link_connection" type="fixed" parent="base_link" child="chassisToa" origin_x="0" origin_y="15.55" origin_z="11" axis_z="0" lower="0" upper="0" />
+    <xacro:joints name="joint_a" type="continuous" parent="chassisToa" child="aTob" origin_x="0" origin_y="0" origin_z="0" axis_z="1" lower="-3.14" upper="3.14" />
+    <xacro:joints name="joint_b" parent="aTob" child="bToc" origin_x="0" origin_y="1.33" origin_z="0.99" axis_x="1" lower="-1.064651" upper="0" roll="0.593412"/>
+    <xacro:joints name="joint_c" parent="bToc" child="cTod" origin_x="0" origin_y="20.11" origin_z="10.75" axis_x="1" lower="-0.087267" upper="4.886922" roll="-0.436332"/>
+    <xacro:joints name="joint_d" parent="cTod" child="dToe" origin_x="-4.4" origin_y="-0.42" origin_z="-2.535" axis_z="1" axis_y="0" lower="-3.14" upper="3.14" roll="-0.15708" pitch="-0.0174533" yaw="0" />
+    <xacro:joints name="joint_e" parent="dToe" child="eTof" origin_x="2.55" origin_y="0.2" origin_z="-17" axis_y="1" lower="-3.59538" upper="0.610865" roll="0" pitch="0" yaw="-1.649336"/>
+    <xacro:joints name="joint_f" parent="eTof" child="hand" origin_x="-6.3" origin_y="1.75" origin_z="0" axis_x="1" lower="-0.523599" upper="6.28" />
+    <xacro:transmissions name="joint_a" />
+    <xacro:transmissions name="joint_b" />
+    <xacro:transmissions name="joint_c" />
+    <xacro:transmissions name="joint_d" />
+    <xacro:transmissions name="joint_e" />
+    <xacro:transmissions name="joint_f" />
+    <xacro:gazebo_ref link="chassisToa" />
+    <xacro:gazebo_ref link="aTob" />
+    <xacro:gazebo_ref link="bToc" />
+    <xacro:gazebo_ref link="cTod" />
+    <xacro:gazebo_ref link="dToe" />
+    <xacro:gazebo_ref link="eTof" />
+    <xacro:gazebo_ref link="hand" />
+    <gazebo>
+        <plugin name="gazebo_ros_control" filename="libgazebo_ros_control.so" />
+    </gazebo>
 </robot>
