Commit message: Add throttle and vel subs for arm, fix drive code thanks wisabel

File: urdf/world/bottle.urdf.xacro (robot description, xacro)
@@ -21,5 +21,11 @@
         <collision>
             <geometry>
-                <cylinder radius="0.08" length="0.25"/>
+                <cylinder radius="0.09" length="0.31"/>
+            </geometry>
+        </collision>
+        <collision>
+            <origin rpy="0 0 0" xyz="0 0 0.16"/>
+            <geometry>
+                <cylinder radius="0.07" length="0.05"/>
             </geometry>
         </collision>
