Commit message: MDRS! :o

File: urdf/world/mdrs.urdf.xacro (robot description, xacro)
@@ -8,10 +8,10 @@
     <visual>
       <geometry>
-        <mesh filename="package://mrover/urdf/meshes/ground.fbx"/>
+        <mesh filename="package://mrover/urdf/meshes/mdrs.fbx"/>
       </geometry>
     </visual>
     <collision>
       <geometry>
-        <mesh filename="package://mrover/urdf/meshes/ground.fbx"/>
+        <mesh filename="package://mrover/urdf/meshes/mdrs.fbx"/>
       </geometry>
     </collision>
