Commit message: Working Align

File: urdf/world/lander.urdf.xacro (robot description, xacro)
@@ -3,6 +3,6 @@
   <link name="base_link">
     <inertial>
-      <mass value="0" />
-      <inertia ixx="0" ixy="0" ixz="0" iyy="0" iyz="0" izz="0" />
+      <mass value="1" />
+      <inertia ixx="1" ixy="1" ixz="1" iyy="1" iyz="1" izz="1" />
     </inertial>
     <visual>

Commit message: lander fat

File: urdf/world/lander.urdf.xacro (robot description, xacro)
@@ -3,6 +3,6 @@
   <link name="base_link">
     <inertial>
-      <mass value="1" />
-      <inertia ixx="1" ixy="1" ixz="1" iyy="1" iyz="1" izz="1" />
+      <mass value="100" />
+      <inertia ixx="10" ixy="10" ixz="10" iyy="10" iyz="10" izz="10" />
     </inertial>
     <visual>
