Commit message: Switch to FBX, textures!

File: urdf/world/world.urdf.xacro (robot description, xacro)
@@ -8,10 +8,10 @@
     <visual>
       <geometry>
-        <mesh filename="package://mrover/urdf/meshes/ground.glb"/>
+        <mesh filename="package://mrover/urdf/meshes/ground.fbx"/>
       </geometry>
     </visual>
     <collision>
       <geometry>
-        <mesh filename="package://mrover/urdf/meshes/ground.glb"/>
+        <mesh filename="package://mrover/urdf/meshes/ground.fbx"/>
       </geometry>
     </collision>

Commit message: Decrease number of things requested from IMU, remove some printing in nav, do dilating in percep, add avoidance when target is not very close, add max iter count on raycast, paramaterize costmap generator better, add timeout on imu for costmap, add spiral search to tag detector

File: urdf/world/world.urdf.xacro (robot description, xacro)
@@ -8,10 +8,10 @@
     <visual>
       <geometry>
-        <mesh filename="package://mrover/urdf/meshes/ground.fbx"/>
+        <mesh filename="package://mrover/urdf/meshes/ground_boulders.fbx"/>
       </geometry>
     </visual>
     <collision>
       <geometry>
-        <mesh filename="package://mrover/urdf/meshes/ground.fbx"/>
+        <mesh filename="package://mrover/urdf/meshes/ground_boulders.fbx"/>
       </geometry>
     </collision>

Commit message: fix world mesh

File: urdf/world/world.urdf.xacro (robot description, xacro)
@@ -8,10 +8,10 @@
     <visual>
       <geometry>
-        <mesh filename="package://mrover/urdf/meshes/ground_boulders.fbx"/>
+        <mesh filename="package://mrover/urdf/meshes/groundflat.fbx"/>
       </geometry>
     </visual>
     <collision>
       <geometry>
-        <mesh filename="package://mrover/urdf/meshes/ground_boulders.fbx"/>
+        <mesh filename="package://mrover/urdf/meshes/groundflat.fbx"/>
       </geometry>
     </collision>
