Commit message: Why is the light so big :(

File: urdf/world/light.urdf.xacro (robot description, xacro)
@@ -1,33 +1,22 @@
 <?xml version="1.0"?>
 <robot xmlns:xacro="http://www.ros.org/wiki/xacro" name="rover">
-    <xacro:property name="mass" value="1.36078"/>\
-    <xacro:property name="TAU" value="6.2831855"/>
-    <xacro:macro name="cylinder_inertia" params="m r h xyz">
-        <inertial>
-            <origin xyz="${xyz}"/>
-            <mass value="${m}"/>
-            <inertia ixx="${m*(3*r*r+h*h)/12}" ixy="0" ixz="0"
-                     iyy="${m*(3*r*r+h*h)/12}" iyz="0"
-                     izz="${m*r*r/2}"/>
-        </inertial>
-    </xacro:macro>
-    <link name="base_link">
-        <xacro:cylinder_inertia m="${mass}" r="0.025" h="0.5" xyz="0 0 0.25"/>
-        <visual>
-            <geometry>
-                <mesh filename="package://mrover/urdf/meshes/light.fbx"/>
-            </geometry>
-        </visual>
-        <collision>
-            <geometry>
-                <cylinder radius="0.024" length="0.5"/>
-            </geometry>
-        </collision>
-        <collision>
-            <origin rpy="${TAU / 4} 0 0" xyz="0 0 0.28"/>
-            <geometry>
-                <cylinder radius="0.057" length="0.185"/>
-            </geometry>
-        </collision>
-    </link>
+  <xacro:property name="mass" value="1.36078"/>\
+  <link name="base_link">
+    <inertial>
+      <mass value="${mass}"/>
+      <inertia ixx="0.01" ixy="0" ixz="0"
+               iyy="0.01" iyz="0"
+               izz="0.01"/>
+    </inertial>
+    <visual>
+      <geometry>
+        <mesh filename="package://mrover/urdf/meshes/light.fbx"/>
+      </geometry>
+    </visual>
+    <collision>
+      <geometry>
+        <mesh filename="package://mrover/urdf/meshes/light.fbx"/>
+      </geometry>
+    </collision>
+  </link>
 </robot>

Commit message: Add load perception nodelet manager

File: urdf/world/light.urdf.xacro (robot description, xacro)
@@ -1,5 +1,5 @@
 <?xml version="1.0"?>
 <robot xmlns:xacro="http://www.ros.org/wiki/xacro" name="rover">
-  <xacro:property name="mass" value="1.36078"/>\
+  <xacro:property name="mass" value="0"/>\
   <link name="base_link">
     <inertial>
