Commit message: Fix wheels

File: urdf/rover/rover.urdf.xacro (robot description, xacro)
@@ -43,9 +43,9 @@
     </collision>
   </link>
-  <xacro:macro name="wheel" params="side reflect">
+  <xacro:macro name="wheel" params="side reflect rotate">
     <link name="front_${side}_wheel_link">
       <xacro:sphere_inertia m="${wheel_mass}" r="${wheel_radius}"/>
       <visual>
-        <origin rpy="${reflect * PI/2} 0 0" xyz="0.0 0.0 0.0"/>
+        <origin rpy="0 0 ${rotate * PI}" xyz="0.0 0.0 0.0"/>
         <geometry>
           <mesh filename="package://mrover/urdf/meshes/rover.wheel.dae"/>
@@ -61,5 +61,5 @@
       <xacro:cylinder_inertia m="${wheel_mass}" r="${wheel_radius}" h="${wheel_width}"/>
       <visual>
-        <origin rpy="${reflect * PI/2} 0 0" xyz="0.0 0.0 0.0"/>
+        <origin rpy="0 0 ${rotate * PI}" xyz="0.0 0.0 0.0"/>
         <geometry>
           <mesh filename="package://mrover/urdf/meshes/rover.wheel.dae"/>
@@ -75,5 +75,5 @@
       <xacro:sphere_inertia m="${wheel_mass}" r="${wheel_radius}"/>
       <visual>
-        <origin rpy="${reflect * PI/2} 0 0" xyz="0.0 0.0 0.0"/>
+        <origin rpy="0 0 ${rotate * PI}" xyz="0.0 0.0 0.0"/>
         <geometry>
           <mesh filename="package://mrover/urdf/meshes/rover.wheel.dae"/>
@@ -89,5 +89,5 @@
       <parent link="chassis_link"/>
       <child link="front_${side}_wheel_link"/>
-      <origin xyz="0.435 ${reflect * (base_width/2 + 0.06)} -0.373" rpy="${-PI/2} 0 0"/>
+      <origin xyz="0.435 ${reflect * (base_width/2 + 0.06)} -0.373" rpy="0 0 0"/>
       <axis xyz="0 0 1"/>
     </joint>
@@ -95,5 +95,5 @@
       <parent link="chassis_link"/>
       <child link="center_${side}_wheel_link"/>
-      <origin xyz="0 ${reflect * (base_width/2 + 0.06)} -0.373" rpy="${-PI/2} 0 0"/>
+      <origin xyz="0 ${reflect * (base_width/2 + 0.06)} -0.373" rpy="0 0 0"/>
       <axis xyz="0 0 1"/>
     </joint>
@@ -101,5 +101,5 @@
       <parent link="chassis_link"/>
       <child link="back_${side}_wheel_link"/>
-      <origin xyz="-0.435 ${reflect*(base_width/2 + 0.06)} -0.373" rpy="${-PI/2} 0 0"/>
+      <origin xyz="-0.435 ${reflect * (base_width/2 + 0.06)} -0.373" rpy="0 0 0"/>
       <axis xyz="0 0 1"/>
     </joint>
@@ -163,5 +163,5 @@
   </link>
   <xacro:include filename="$(find mrover)/urdf/rover/rover_gazebo_plugins.urdf.xacro"/>
-  <xacro:wheel side="left" reflect="1"/>
-  <xacro:wheel side="right" reflect="-1"/>
+  <xacro:wheel side="left" reflect="1" rotate="1"/>
+  <xacro:wheel side="right" reflect="-1" rotate="0"/>
 </robot>

Commit message: fix rotations

File: urdf/rover/rover.urdf.xacro (robot description, xacro)
@@ -43,9 +43,9 @@
     </collision>
   </link>
-  <xacro:macro name="wheel" params="side reflect rotate">
+  <xacro:macro name="wheel" params="side reflect">
     <link name="front_${side}_wheel_link">
       <xacro:sphere_inertia m="${wheel_mass}" r="${wheel_radius}"/>
       <visual>
-        <origin rpy="0 0 ${rotate * PI}" xyz="0.0 0.0 0.0"/>
+        <origin rpy="0 ${min(0, reflect) * PI} 0" xyz="0 0 0"/>
         <geometry>
           <mesh filename="package://mrover/urdf/meshes/rover.wheel.dae"/>
@@ -61,5 +61,5 @@
       <xacro:cylinder_inertia m="${wheel_mass}" r="${wheel_radius}" h="${wheel_width}"/>
       <visual>
-        <origin rpy="0 0 ${rotate * PI}" xyz="0.0 0.0 0.0"/>
+        <origin rpy="0 ${min(0, reflect) * PI} 0" xyz="0 0 0"/>
         <geometry>
           <mesh filename="package://mrover/urdf/meshes/rover.wheel.dae"/>
@@ -75,5 +75,5 @@
       <xacro:sphere_inertia m="${wheel_mass}" r="${wheel_radius}"/>
       <visual>
-        <origin rpy="0 0 ${rotate * PI}" xyz="0.0 0.0 0.0"/>
+        <origin rpy="0 ${min(0, reflect) * PI} 0" xyz="0 0 0"/>
         <geometry>
           <mesh filename="package://mrover/urdf/meshes/rover.wheel.dae"/>
@@ -89,5 +89,5 @@
       <parent link="chassis_link"/>
       <child link="front_${side}_wheel_link"/>
-      <origin xyz="0.435 ${reflect * (base_width/2 + 0.06)} -0.373" rpy="0 0 0"/>
+      <origin xyz="0.42 ${reflect * (base_width/2 + 0.06)} -0.373" rpy="${-PI/2} 0 0"/>
       <axis xyz="0 0 1"/>
     </joint>
@@ -95,5 +95,5 @@
       <parent link="chassis_link"/>
       <child link="center_${side}_wheel_link"/>
-      <origin xyz="0 ${reflect * (base_width/2 + 0.06)} -0.373" rpy="0 0 0"/>
+      <origin xyz="0 ${reflect * (base_width/2 + 0.06)} -0.373" rpy="${-PI/2} 0 0"/>
       <axis xyz="0 0 1"/>
     </joint>
@@ -101,5 +101,5 @@
       <parent link="chassis_link"/>
       <child link="back_${side}_wheel_link"/>
-      <origin xyz="-0.435 ${reflect * (base_width/2 + 0.06)} -0.373" rpy="0 0 0"/>
+      <origin xyz="-0.42 ${reflect * (base_width/2 + 0.06)} -0.373" rpy="${-PI/2} 0 0"/>
       <axis xyz="0 0 1"/>
     </joint>
@@ -163,5 +163,5 @@
   </link>
   <xacro:include filename="$(find mrover)/urdf/rover/rover_gazebo_plugins.urdf.xacro"/>
-  <xacro:wheel side="left" reflect="1" rotate="1"/>
-  <xacro:wheel side="right" reflect="-1" rotate="0"/>
+  <xacro:wheel side="left" reflect="1"/>
+  <xacro:wheel side="right" reflect="-1"/>
 </robot>

Commit message: Fix camera links, don't use odom frame by default since we are going to rtk

File: urdf/rover/rover.urdf.xacro (robot description, xacro)
@@ -143,11 +143,11 @@
     </inertial>
   </link>
-  <!-- Right Camera -->
-  <joint name="right_camera_joint" type="fixed">
+  <!-- Left Camera -->
+  <joint name="left_camera_joint" type="fixed">
     <origin xyz="0 -0.05 0.1"/>
     <parent link="chassis_link"/>
-    <child link="right_camera_link"/>
+    <child link="left_camera_link"/>
   </joint>
-  <link name="right_camera_link">
+  <link name="left_camera_link">
     <collision>
       <origin xyz="0 0 0" rpy="0 0 0"/>

File: urdf/rover/rover_gazebo_plugins.urdf.xacro (robot description, xacro)
@@ -99,5 +99,5 @@
         <depthImageInfoTopicName>camera_info</depthImageInfoTopicName>
         <pointCloudTopicName>points</pointCloudTopicName>
-        <frameName>camera_link</frameName>
+        <frameName>left_camera_link</frameName>
         <pointCloudCutoff>0.3</pointCloudCutoff>
         <pointCloudCutoffMax>20.0</pointCloudCutoffMax>

Commit message: Arm URDF, updated rover URDF, remove some unneeded packages (#530)
* Add arm blend file

* In progress update

* Ooops

* Fix loading model

* Get the arm imported properly as a urdf. arm_rviz_display.launch works now

* start at zeros

* Get rid of image transport, this links old opencv which is bad for when we use new opencv. also if we ever transport image it is over custom stream anyways.

* Fix wheels

* Actually push files

* Show image properly

* fix rotations

* Fix camera links, don't use odom frame by default since we are going to rtk

File: urdf/rover/rover.urdf.xacro (robot description, xacro)
@@ -7,7 +7,6 @@
   <xacro:property name="wheel_width" value="0.1"/>
   <xacro:property name="wheel_mass" value="2"/>
-  <!-- <xacro:property name="mesh_scale" value="0.0254 0.0254 0.0254" /> -->
   <xacro:property name="PI" value="3.141592"/>
-  <!--Interial macros-->
+  <!-- Inertial macros-->
   <xacro:macro name="cylinder_inertia" params="m r h">
     <inertial>
@@ -28,11 +27,12 @@
     </inertial>
   </xacro:macro>
-  <!--Base link-->
-  <link name="base_link">
+  <!-- Links -->
+  <link name="base_link"/>
+  <link name="chassis_link">
     <xacro:box_inertia m="3.0" w="${base_len}" h="${base_width}" d="${base_height}"/>
     <visual>
-      <origin rpy="0 0 0" xyz="-0.25 0.0 0.2"/>
+      <origin rpy="0 0 0" xyz="0 0 0"/>
       <geometry>
-        <mesh filename="package://mrover/rover_description/meshes/rover.dae" scale="1 1 1"/>
+        <mesh filename="package://mrover/urdf/meshes/rover.dae"/>
       </geometry>
     </visual>
@@ -47,7 +47,7 @@
       <xacro:sphere_inertia m="${wheel_mass}" r="${wheel_radius}"/>
       <visual>
-        <origin rpy="${reflect * PI/2} 0 0" xyz="0.0 0.0 0.0"/>
+        <origin rpy="0 ${min(0, reflect) * PI} 0" xyz="0 0 0"/>
         <geometry>
-          <mesh filename="package://mrover/rover_description/meshes/wheel.dae" scale="1 1 1"/>
+          <mesh filename="package://mrover/urdf/meshes/rover.wheel.dae"/>
         </geometry>
       </visual>
@@ -61,7 +61,7 @@
       <xacro:cylinder_inertia m="${wheel_mass}" r="${wheel_radius}" h="${wheel_width}"/>
       <visual>
-        <origin rpy="${reflect * PI/2} 0 0" xyz="0.0 0.0 0.0"/>
+        <origin rpy="0 ${min(0, reflect) * PI} 0" xyz="0 0 0"/>
         <geometry>
-          <mesh filename="package://mrover/rover_description/meshes/wheel.dae" scale="1 1 1"/>
+          <mesh filename="package://mrover/urdf/meshes/rover.wheel.dae"/>
         </geometry>
       </visual>
@@ -75,7 +75,7 @@
       <xacro:sphere_inertia m="${wheel_mass}" r="${wheel_radius}"/>
       <visual>
-        <origin rpy="${reflect * PI/2} 0 0" xyz="0.0 0.0 0.0"/>
+        <origin rpy="0 ${min(0, reflect) * PI} 0" xyz="0 0 0"/>
         <geometry>
-          <mesh filename="package://mrover/rover_description/meshes/wheel.dae" scale="1 1 1"/>
+          <mesh filename="package://mrover/urdf/meshes/rover.wheel.dae"/>
         </geometry>
       </visual>
@@ -87,33 +87,39 @@
     </link>
     <joint name="front_${side}_wheel_joint" type="continuous">
-      <parent link="base_link"/>
+      <parent link="chassis_link"/>
       <child link="front_${side}_wheel_link"/>
-      <origin xyz="0.42 ${reflect * (base_width/2 + 0.06)} -0.27" rpy="${-PI/2} 0 0"/>
+      <origin xyz="0.42 ${reflect * (base_width/2 + 0.06)} -0.373" rpy="${-PI/2} 0 0"/>
       <axis xyz="0 0 1"/>
     </joint>
     <joint name="center_${side}_wheel_joint" type="continuous">
-      <parent link="base_link"/>
+      <parent link="chassis_link"/>
       <child link="center_${side}_wheel_link"/>
-      <origin xyz="0 ${reflect * (base_width/2 + 0.06)} -0.27" rpy="${-PI/2} 0 0"/>
+      <origin xyz="0 ${reflect * (base_width/2 + 0.06)} -0.373" rpy="${-PI/2} 0 0"/>
       <axis xyz="0 0 1"/>
     </joint>
     <joint name="back_${side}_wheel_joint" type="continuous">
-      <parent link="base_link"/>
+      <parent link="chassis_link"/>
       <child link="back_${side}_wheel_link"/>
-      <origin xyz="-0.42 ${reflect*(base_width/2 + 0.06)} -0.27" rpy="${-PI/2} 0 0"/>
+      <origin xyz="-0.42 ${reflect * (base_width/2 + 0.06)} -0.373" rpy="${-PI/2} 0 0"/>
       <axis xyz="0 0 1"/>
     </joint>
   </xacro:macro>
+  <!-- Joints -->
+  <joint name="base_link_to_chassis" type="fixed">
+    <origin xyz="0 0 0.5"/>
+    <parent link="base_link"/>
+    <child link="chassis_link"/>
+  </joint>
   <!-- IMU -->
   <joint name="imu_joint" type="fixed">
     <origin xyz="0 0 0.2"/>
-    <parent link="base_link"/>
+    <parent link="chassis_link"/>
     <child link="imu_link"/>
   </joint>
-  <link name="imu_link"></link>
+  <link name="imu_link"/>
   <!-- Camera -->
   <joint name="camera_joint" type="fixed">
-    <origin xyz="0 0 0.2"/>
-    <parent link="base_link"/>
+    <origin xyz="0 0 0.1"/>
+    <parent link="chassis_link"/>
     <child link="camera_link"/>
   </joint>
@@ -128,5 +134,5 @@
       <origin xyz="0 0 0" rpy="0 0 0"/>
       <geometry>
-        <mesh filename="package://mrover/rover_description/meshes/zed2i.dae" scale="1 1 1"/>
+        <mesh filename="package://mrover/urdf/meshes/zed2i.dae"/>
       </geometry>
     </visual>
@@ -137,8 +143,8 @@
     </inertial>
   </link>
-  <!-- Left Stereoscopic Camera -->
+  <!-- Left Camera -->
   <joint name="left_camera_joint" type="fixed">
-    <origin xyz="0 0.05 0.2"/>
-    <parent link="base_link"/>
+    <origin xyz="0 -0.05 0.1"/>
+    <parent link="chassis_link"/>
     <child link="left_camera_link"/>
   </joint>
@@ -150,10 +156,4 @@
       </geometry>
     </collision>
-    <visual>
-      <origin xyz="0 0 0" rpy="0 0 0"/>
-      <geometry>
-        <box size="0.06 0.01 0.06"/>
-      </geometry>
-    </visual>
     <inertial>
       <mass value="1e-5"/>
@@ -162,30 +162,5 @@
     </inertial>
   </link>
-  <!-- Right Stereoscopic Camera -->
-  <joint name="right_camera_joint" type="fixed">
-    <origin xyz="0 -0.05 0.2"/>
-    <parent link="base_link"/>
-    <child link="right_camera_link"/>
-  </joint>
-  <link name="right_camera_link">
-    <collision>
-      <origin xyz="0 0 0" rpy="0 0 0"/>
-      <geometry>
-        <box size="0.06 0.01 0.06"/>
-      </geometry>
-    </collision>
-    <visual>
-      <origin xyz="0 0 0" rpy="0 0 0"/>
-      <geometry>
-        <box size="0.06 0.01 0.06"/>
-      </geometry>
-    </visual>
-    <inertial>
-      <mass value="1e-5"/>
-      <origin xyz="0 0 0" rpy="0 0 0"/>
-      <inertia ixx="1e-6" ixy="0" ixz="0" iyy="1e-6" iyz="0" izz="1e-6"/>
-    </inertial>
-  </link>
-  <xacro:include filename="$(find mrover)/rover_description/rover_gazebo_plugins.xacro"/>
+  <xacro:include filename="$(find mrover)/urdf/rover/rover_gazebo_plugins.urdf.xacro"/>
   <xacro:wheel side="left" reflect="1"/>
   <xacro:wheel side="right" reflect="-1"/>

File: urdf/rover/rover_gazebo_plugins.urdf.xacro (robot description, xacro)
@@ -38,5 +38,4 @@
   <!-- IMU -->
   <gazebo reference="imu_link">
-    <gravity>false</gravity>
     <sensor name="imu_sensor" type="imu">
       <always_on>true</always_on>
@@ -77,10 +76,10 @@
   <gazebo reference="camera_link">
     <sensor name="camera_link_camera" type="depth">
-      <update_rate>20</update_rate>
+      <update_rate>15</update_rate>
       <camera>
         <horizontal_fov>1.919862</horizontal_fov>
         <image>
-          <width>640</width>
-          <height>480</height>
+          <width>320</width>
+          <height>240</height>
           <format>R8G8B8</format>
         </image>
@@ -91,7 +90,7 @@
       </camera>
       <plugin name="gazebo_ros_openni_kinect_plugin" filename="libkinect_plugin.so">
-        <baseline>0.2</baseline>
+        <baseline>0</baseline> <!-- Publish same rate as camera -->
         <alwaysOn>true</alwaysOn>
-        <updateRate>1.0</updateRate>
+        <updateRate>5</updateRate>
         <cameraName>camera/left</cameraName>
         <imageTopicName>image</imageTopicName>
@@ -100,5 +99,5 @@
         <depthImageInfoTopicName>camera_info</depthImageInfoTopicName>
         <pointCloudTopicName>points</pointCloudTopicName>
-        <frameName>camera_link</frameName>
+        <frameName>left_camera_link</frameName>
         <pointCloudCutoff>0.3</pointCloudCutoff>
         <pointCloudCutoffMax>20.0</pointCloudCutoffMax>
@@ -116,65 +115,3 @@
     </sensor>
   </gazebo>
-  <gazebo reference="left_camera_link">
-    <sensor name="left_camera_link_camera" type="camera">
-      <update_rate>20</update_rate>
-      <camera>
-        <horizontal_fov>1.919862</horizontal_fov>
-        <image>
-          <width>640</width>
-          <height>480</height>
-          <format>R8G8B8</format>
-        </image>
-        <clip>
-          <near>0.2</near>
-          <far>20</far>
-        </clip>
-      </camera>
-      <plugin name="left_camera_controller" filename="libgazebo_ros_camera.so">
-        <alwaysOn>true</alwaysOn>
-        <updateRate>20</updateRate>
-        <cameraName>camera/left</cameraName>
-        <imageTopicName>image</imageTopicName>
-        <cameraInfoTopicName>camera_info</cameraInfoTopicName>
-        <frameName>base_link</frameName>
-        <hackBaseline>0.02</hackBaseline>
-        <distortionK1>0.0</distortionK1>
-        <distortionK2>0.0</distortionK2>
-        <distortionK3>0.0</distortionK3>
-        <distortionT1>0.0</distortionT1>
-        <distortionT2>0.0</distortionT2>
-      </plugin>
-    </sensor>
-  </gazebo>
-  <gazebo reference="right_camera_link">
-    <sensor name="right_camera_link_camera" type="camera">
-      <update_rate>20</update_rate>
-      <camera>
-        <horizontal_fov>1.919862</horizontal_fov>
-        <image>
-          <width>640</width>
-          <height>480</height>
-          <format>R8G8B8</format>
-        </image>
-        <clip>
-          <near>0.2</near>
-          <far>20</far>
-        </clip>
-      </camera>
-      <plugin name="right_camera_controller" filename="libgazebo_ros_camera.so">
-        <alwaysOn>true</alwaysOn>
-        <updateRate>20</updateRate>
-        <cameraName>camera/right</cameraName>
-        <imageTopicName>image</imageTopicName>
-        <cameraInfoTopicName>camera_info</cameraInfoTopicName>
-        <frameName>base_link</frameName>
-        <hackBaseline>0.07</hackBaseline>
-        <distortionK1>0.0</distortionK1>
-        <distortionK2>0.0</distortionK2>
-        <distortionK3>0.0</distortionK3>
-        <distortionT1>0.0</distortionT1>
-        <distortionT2>0.0</distortionT2>
-      </plugin>
-    </sensor>
-  </gazebo>
 </robot>

File: urdf/zed/zed_descr.urdf.xacro (robot description, xacro)
@@ -25,5 +25,5 @@
     <xacro:arg name="cam_pitch" default="0.0"/>
     <xacro:arg name="cam_yaw" default="0.0"/>
-    <xacro:include filename="$(find mrover)/rover_description/zed/zed_macro.urdf.xacro"/>
+    <xacro:include filename="$(find mrover)/urdf/zed/zed_macro.urdf.xacro"/>
     <xacro:zed_camera name="$(arg camera_name)" model="$(arg camera_model)" parent="$(arg base_frame)">
         <origin xyz="$(arg cam_pos_x) $(arg cam_pos_y) $(arg cam_pos_z)" rpy="$(arg cam_roll) $(arg cam_pitch) $(arg cam_yaw)"/>

File: urdf/zed/zed_macro.urdf.xacro (robot description, xacro)
@@ -16,5 +16,5 @@
 -->
 <robot xmlns:xacro="http://wiki.ros.org/xacro">
-    <xacro:include filename="$(find mrover)/rover_description/zed/include/materials.urdf.xacro"/>
+    <xacro:include filename="$(find mrover)/urdf/zed/include/materials.urdf.xacro"/>
     <xacro:property name="M_PI" value="3.1415926535897931"/>
     <!--
@@ -66,5 +66,5 @@
                 <origin xyz="${screw_offset_x} 0 0" rpy="0 0 0"/>
                 <geometry>
-                    <mesh filename="package://mrover/rover_description/meshes/${model}.dae"/>
+                    <mesh filename="package://mrover/urdf/meshes/${model}.dae"/>
                 </geometry>
                 <material name="${model}_mat"/>
@@ -72,5 +72,5 @@
             <collision>
                 <geometry>
-                    <mesh filename="package://mrover/rover_description/meshes/${model}.dae"/>
+                    <mesh filename="package://mrover/urdf/meshes/${model}.dae"/>
                 </geometry>
             </collision>

Commit message: started adding gps to gazebo

File: urdf/rover/rover.urdf.xacro (robot description, xacro)
@@ -29,4 +29,14 @@
   <!-- Links -->
   <link name="base_link"/>
+  <link name="rover_gps_left">
+    <visual>
+      <origin rpy="0 0 0" xyz="0.5 0 0"/>
+    </visual>
+  </link>
+  <link name="rover_gps_right">
+    <visual>
+      <origin rpy="0 0 0" xyz="-0.5 0 0"/>
+    </visual>
+  </link>
   <link name="chassis_link">
     <xacro:box_inertia m="3.0" w="${base_len}" h="${base_width}" d="${base_height}"/>

File: urdf/rover/rover_gazebo_plugins.urdf.xacro (robot description, xacro)
@@ -18,8 +18,8 @@
       <bodyName>base_link</bodyName>
     </plugin>
-    <!-- GPS -->
-    <plugin name="gazebo_ros_gps" filename="libhector_gazebo_ros_gps.so">
+    <!-- Rover GPS Left -->
+    <plugin name="rover_gps_left" filename="libhector_gazebo_ros_gps.so">
       <updateRate>100.0</updateRate>
-      <bodyName>base_link</bodyName>
+      <bodyName>rover_gps_left</bodyName>
       <frameId>base_link</frameId>
       <topicName>gps/fix</topicName>
@@ -34,4 +34,19 @@
       <velocityDrift>0.0 0.0 0.0</velocityDrift>
       <velocityGaussianNoise>0.2 0.2 0.2</velocityGaussianNoise>
+    </plugin>
+    <!-- Rover GPS Right -->
+    <plugin name="rover_gps_right" filename="libhector_gazebo_ros_gps.so">
+      <updateRate>100.0</updateRate>
+      <bodyName>rover_gps_right</bodyName>
+      <frameId></frameId>
+      <velocityTopicName>gps/fix_velocity</velocityTopicName>
+      <referenceLatitude></referenceLatitude>
+      <referenceLongitude></referenceLongitude>
+      <referenceAltitude></referenceAltitude>
+      <offset></offset>
+      <drift></droft>
+      <gaussianNoise></gaussianNoise>
+      <velocityDrift></velocityDrift>
+      <velocityGaussianNoise></velocityGaussianNoise>
     </plugin>
   </gazebo>

Commit message: edited links

File: urdf/rover/rover.urdf.xacro (robot description, xacro)
@@ -29,14 +29,4 @@
   <!-- Links -->
   <link name="base_link"/>
-  <link name="rover_gps_left">
-    <visual>
-      <origin rpy="0 0 0" xyz="0.5 0 0"/>
-    </visual>
-  </link>
-  <link name="rover_gps_right">
-    <visual>
-      <origin rpy="0 0 0" xyz="-0.5 0 0"/>
-    </visual>
-  </link>
   <link name="chassis_link">
     <xacro:box_inertia m="3.0" w="${base_len}" h="${base_width}" d="${base_height}"/>
@@ -128,4 +118,17 @@
   </joint>
   <link name="imu_link"/>
+  <!-- GPS -->
+  <joint name="rover_gps_left_joint" type="fixed">
+    <origin xyz="-0.5 0 0"/>
+    <parent link="chassis_link"/>
+    <child link="rover_gps_left_link"/>
+  </joint>
+  <link name="rover_gps_left_link"/>
+  <joint name="rover_gps_right_joint" type="fixed">
+    <origin xyz="0.5 0 0"/>
+    <parent link="chassis_link"/>
+    <child link="rover_gps_right_link"/>
+  </joint>
+  <link name="rover_gps_right_link"/>
   <!-- Camera -->
   <joint name="camera_joint" type="fixed">

File: urdf/rover/rover_gazebo_plugins.urdf.xacro (robot description, xacro)
@@ -21,5 +21,5 @@
     <plugin name="rover_gps_left" filename="libhector_gazebo_ros_gps.so">
       <updateRate>100.0</updateRate>
-      <bodyName>rover_gps_left</bodyName>
+      <bodyName>rover_gps_left_link</bodyName>
       <frameId></frameId>
       <topicName>gps/fix_gps_left</topicName>
@@ -38,5 +38,5 @@
     <plugin name="rover_gps_right" filename="libhector_gazebo_ros_gps.so">
       <updateRate>100.0</updateRate>
-      <bodyName>rover_gps_right</bodyName>
+      <bodyName>rover_gps_right_link</bodyName>
       <frameId></frameId>
       <topicName>gps/fix_gps_right</topicName>
@@ -47,5 +47,5 @@
       <referenceAltitude>0.0</referenceAltitude>
       <offset>0 0 0</offset>
-      <drift>0.0 0.0 0.0</droft>
+      <drift>0.0 0.0 0.0</drift>
       <gaussianNoise>0.3 0.3 0.3</gaussianNoise>
       <velocityDrift>0.0 0.0 0.0</velocityDrift>

Commit message: added links

File: urdf/rover/rover.urdf.xacro (robot description, xacro)
@@ -119,16 +119,16 @@
   <link name="imu_link"/>
   <!-- GPS -->
+  <link name="rover_gps_left_link"/>
   <joint name="rover_gps_left_joint" type="fixed">
-    <origin xyz="-0.5 0 0"/>
+    <origin xyz="0 -0.5 0"/>
     <parent link="chassis_link"/>
     <child link="rover_gps_left_link"/>
   </joint>
-  <link name="rover_gps_left_link"/>
+  <link name="rover_gps_right_link"/>
   <joint name="rover_gps_right_joint" type="fixed">
-    <origin xyz="0.5 0 0"/>
+    <origin xyz="0 0.5 0"/>
     <parent link="chassis_link"/>
     <child link="rover_gps_right_link"/>
   </joint>
-  <link name="rover_gps_right_link"/>
   <!-- Camera -->
   <joint name="camera_joint" type="fixed">
