Commit message: try to debug plugins and make test subscriber file

File: urdf/rover/rover.urdf.xacro (robot description, xacro)
@@ -1,43 +1,46 @@
 <?xml version="1.0"?>
 <robot xmlns:xacro="http://www.ros.org/wiki/xacro" name="rover">
-  <xacro:property name="base_width" value="0.7357"/>
-  <xacro:property name="base_len" value="1.0"/>
-  <xacro:property name="base_height" value="0.6"/>
-  <xacro:property name="wheel_radius" value="0.13"/>
-  <xacro:property name="wheel_width" value="0.1"/>
-  <xacro:property name="wheel_mass" value="2"/>
-  <xacro:property name="PI" value="3.141592"/>
+  <xacro:property name="base_width" value="0.7357" />
+  <xacro:property name="base_len" value="1.0" />
+  <xacro:property name="base_height" value="0.6" />
+  <xacro:property name="wheel_radius" value="0.13" />
+  <xacro:property name="wheel_width" value="0.1" />
+  <xacro:property name="wheel_mass" value="2" />
+  <xacro:property name="PI" value="3.141592" />
   <!-- Inertial macros-->
   <xacro:macro name="cylinder_inertia" params="m r h">
     <inertial>
-      <mass value="${m}"/>
-      <inertia ixx="${m*(3*r*r+h*h)/12}" ixy="0" ixz="0" iyy="${m*(3*r*r+h*h)/12}" iyz="0" izz="${m*r*r/2}"/>
+      <mass value="${m}" />
+      <inertia ixx="${m*(3*r*r+h*h)/12}" ixy="0" ixz="0" iyy="${m*(3*r*r+h*h)/12}" iyz="0"
+        izz="${m*r*r/2}" />
     </inertial>
   </xacro:macro>
   <xacro:macro name="box_inertia" params="m w h d">
     <inertial>
-      <mass value="${m}"/>
-      <inertia ixx="${m / 12.0 * (d*d + h*h)}" ixy="0.0" ixz="0.0" iyy="${m / 12.0 * (w*w + h*h)}" iyz="0.0" izz="${m / 12.0 * (w*w + d*d)}"/>
+      <mass value="${m}" />
+      <inertia ixx="${m / 12.0 * (d*d + h*h)}" ixy="0.0" ixz="0.0" iyy="${m / 12.0 * (w*w + h*h)}"
+        iyz="0.0" izz="${m / 12.0 * (w*w + d*d)}" />
     </inertial>
   </xacro:macro>
   <xacro:macro name="sphere_inertia" params="m r">
     <inertial>
-      <mass value="${m}"/>
-      <inertia ixx="${2.0*m*(r*r)/5.0}" ixy="0.0" ixz="0.0" iyy="${2.0*m*(r*r)/5.0}" iyz="0.0" izz="${2.0*m*(r*r)/5.0}"/>
+      <mass value="${m}" />
+      <inertia ixx="${2.0*m*(r*r)/5.0}" ixy="0.0" ixz="0.0" iyy="${2.0*m*(r*r)/5.0}" iyz="0.0"
+        izz="${2.0*m*(r*r)/5.0}" />
     </inertial>
   </xacro:macro>
   <!-- Links -->
-  <link name="base_link"/>
+  <link name="base_link" />
   <link name="chassis_link">
-    <xacro:box_inertia m="3.0" w="${base_len}" h="${base_width}" d="${base_height}"/>
+    <xacro:box_inertia m="3.0" w="${base_len}" h="${base_width}" d="${base_height}" />
     <visual>
-      <origin rpy="0 0 0" xyz="0 0 0"/>
+      <origin rpy="0 0 0" xyz="0 0 0" />
       <geometry>
-        <mesh filename="package://mrover/urdf/meshes/rover.dae"/>
+        <mesh filename="package://mrover/urdf/meshes/rover.dae" />
       </geometry>
     </visual>
     <collision>
       <geometry>
-        <box size="${base_len} ${base_width} ${base_height}"/>
+        <box size="${base_len} ${base_width} ${base_height}" />
       </geometry>
     </collision>
@@ -45,136 +48,136 @@
   <xacro:macro name="wheel" params="side reflect">
     <link name="front_${side}_wheel_link">
-      <xacro:sphere_inertia m="${wheel_mass}" r="${wheel_radius}"/>
+      <xacro:sphere_inertia m="${wheel_mass}" r="${wheel_radius}" />
       <visual>
-        <origin rpy="0 ${min(0, reflect) * PI} 0" xyz="0 0 0"/>
+        <origin rpy="0 ${min(0, reflect) * PI} 0" xyz="0 0 0" />
         <geometry>
-          <mesh filename="package://mrover/urdf/meshes/rover.wheel.dae"/>
+          <mesh filename="package://mrover/urdf/meshes/rover.wheel.dae" />
         </geometry>
       </visual>
       <collision>
         <geometry>
-          <sphere radius="${wheel_radius}"/>
+          <sphere radius="${wheel_radius}" />
         </geometry>
       </collision>
     </link>
     <link name="center_${side}_wheel_link">
-      <xacro:cylinder_inertia m="${wheel_mass}" r="${wheel_radius}" h="${wheel_width}"/>
+      <xacro:cylinder_inertia m="${wheel_mass}" r="${wheel_radius}" h="${wheel_width}" />
       <visual>
-        <origin rpy="0 ${min(0, reflect) * PI} 0" xyz="0 0 0"/>
+        <origin rpy="0 ${min(0, reflect) * PI} 0" xyz="0 0 0" />
         <geometry>
-          <mesh filename="package://mrover/urdf/meshes/rover.wheel.dae"/>
+          <mesh filename="package://mrover/urdf/meshes/rover.wheel.dae" />
         </geometry>
       </visual>
       <collision>
         <geometry>
-          <cylinder length="${wheel_width}" radius="${wheel_radius}"/>
+          <cylinder length="${wheel_width}" radius="${wheel_radius}" />
         </geometry>
       </collision>
     </link>
     <link name="back_${side}_wheel_link">
-      <xacro:sphere_inertia m="${wheel_mass}" r="${wheel_radius}"/>
+      <xacro:sphere_inertia m="${wheel_mass}" r="${wheel_radius}" />
       <visual>
-        <origin rpy="0 ${min(0, reflect) * PI} 0" xyz="0 0 0"/>
+        <origin rpy="0 ${min(0, reflect) * PI} 0" xyz="0 0 0" />
         <geometry>
-          <mesh filename="package://mrover/urdf/meshes/rover.wheel.dae"/>
+          <mesh filename="package://mrover/urdf/meshes/rover.wheel.dae" />
         </geometry>
       </visual>
       <collision>
         <geometry>
-          <sphere radius="${wheel_radius}"/>
+          <sphere radius="${wheel_radius}" />
         </geometry>
       </collision>
     </link>
     <joint name="front_${side}_wheel_joint" type="continuous">
-      <parent link="chassis_link"/>
-      <child link="front_${side}_wheel_link"/>
-      <origin xyz="0.42 ${reflect * (base_width/2 + 0.06)} -0.373" rpy="${-PI/2} 0 0"/>
-      <axis xyz="0 0 1"/>
+      <parent link="chassis_link" />
+      <child link="front_${side}_wheel_link" />
+      <origin xyz="0.42 ${reflect * (base_width/2 + 0.06)} -0.373" rpy="${-PI/2} 0 0" />
+      <axis xyz="0 0 1" />
     </joint>
     <joint name="center_${side}_wheel_joint" type="continuous">
-      <parent link="chassis_link"/>
-      <child link="center_${side}_wheel_link"/>
-      <origin xyz="0 ${reflect * (base_width/2 + 0.06)} -0.373" rpy="${-PI/2} 0 0"/>
-      <axis xyz="0 0 1"/>
+      <parent link="chassis_link" />
+      <child link="center_${side}_wheel_link" />
+      <origin xyz="0 ${reflect * (base_width/2 + 0.06)} -0.373" rpy="${-PI/2} 0 0" />
+      <axis xyz="0 0 1" />
     </joint>
     <joint name="back_${side}_wheel_joint" type="continuous">
-      <parent link="chassis_link"/>
-      <child link="back_${side}_wheel_link"/>
-      <origin xyz="-0.42 ${reflect * (base_width/2 + 0.06)} -0.373" rpy="${-PI/2} 0 0"/>
-      <axis xyz="0 0 1"/>
+      <parent link="chassis_link" />
+      <child link="back_${side}_wheel_link" />
+      <origin xyz="-0.42 ${reflect * (base_width/2 + 0.06)} -0.373" rpy="${-PI/2} 0 0" />
+      <axis xyz="0 0 1" />
     </joint>
   </xacro:macro>
   <!-- Joints -->
   <joint name="base_link_to_chassis" type="fixed">
-    <origin xyz="0 0 0.5"/>
-    <parent link="base_link"/>
-    <child link="chassis_link"/>
+    <origin xyz="0 0 0.5" />
+    <parent link="base_link" />
+    <child link="chassis_link" />
   </joint>
   <!-- IMU -->
   <joint name="imu_joint" type="fixed">
-    <origin xyz="0 0 0.2"/>
-    <parent link="chassis_link"/>
-    <child link="imu_link"/>
+    <origin xyz="0 0 0.2" />
+    <parent link="chassis_link" />
+    <child link="imu_link" />
   </joint>
-  <link name="imu_link"/>
+  <link name="imu_link" />
   <!-- GPS -->
-  <link name="rover_gps_left_link"/>
-  <joint name="rover_gps_left_joint" type="fixed">
-    <origin xyz="0 -0.5 0"/>
-    <parent link="chassis_link"/>
-    <child link="rover_gps_left_link"/>
+  <joint name="rover_gps_left" type="fixed">
+    <origin xyz="0 -0.5 0" />
+    <parent link="chassis_link" />
+    <child link="gps_link" />
   </joint>
-  <link name="rover_gps_right_link"/>
-  <joint name="rover_gps_right_joint" type="fixed">
-    <origin xyz="0 0.5 0"/>
-    <parent link="chassis_link"/>
-    <child link="rover_gps_right_link"/>
+  <!-- <link name="rover_gps_right_link"/> -->
+  <joint name="rover_gps_right" type="fixed">
+    <origin xyz="0 0.5 0" />
+    <parent link="chassis_link" />
+    <child link="gps_link" />
   </joint>
+  <link name="gps_link" />
   <!-- Camera -->
   <joint name="camera_joint" type="fixed">
-    <origin xyz="0 0 0.1"/>
-    <parent link="chassis_link"/>
-    <child link="camera_link"/>
+    <origin xyz="0 0 0.1" />
+    <parent link="chassis_link" />
+    <child link="camera_link" />
   </joint>
   <link name="camera_link">
     <collision>
-      <origin xyz="0 0 0" rpy="0 0 0"/>
+      <origin xyz="0 0 0" rpy="0 0 0" />
       <geometry>
-        <box size="0.01 0.1 0.01"/>
+        <box size="0.01 0.1 0.01" />
       </geometry>
     </collision>
     <visual>
-      <origin xyz="0 0 0" rpy="0 0 0"/>
+      <origin xyz="0 0 0" rpy="0 0 0" />
       <geometry>
-        <mesh filename="package://mrover/urdf/meshes/zed2i.dae"/>
+        <mesh filename="package://mrover/urdf/meshes/zed2i.dae" />
       </geometry>
     </visual>
     <inertial>
-      <mass value="1e-5"/>
-      <origin xyz="0 0 0" rpy="0 0 0"/>
-      <inertia ixx="1e-6" ixy="0" ixz="0" iyy="1e-6" iyz="0" izz="1e-6"/>
+      <mass value="1e-5" />
+      <origin xyz="0 0 0" rpy="0 0 0" />
+      <inertia ixx="1e-6" ixy="0" ixz="0" iyy="1e-6" iyz="0" izz="1e-6" />
     </inertial>
   </link>
   <!-- Left Camera -->
   <joint name="left_camera_joint" type="fixed">
-    <origin xyz="0 -0.05 0.1"/>
-    <parent link="chassis_link"/>
-    <child link="left_camera_link"/>
+    <origin xyz="0 -0.05 0.1" />
+    <parent link="chassis_link" />
+    <child link="left_camera_link" />
   </joint>
   <link name="left_camera_link">
     <collision>
-      <origin xyz="0 0 0" rpy="0 0 0"/>
+      <origin xyz="0 0 0" rpy="0 0 0" />
       <geometry>
-        <box size="0.06 0.01 0.06"/>
+        <box size="0.06 0.01 0.06" />
       </geometry>
     </collision>
     <inertial>
-      <mass value="1e-5"/>
-      <origin xyz="0 0 0" rpy="0 0 0"/>
-      <inertia ixx="1e-6" ixy="0" ixz="0" iyy="1e-6" iyz="0" izz="1e-6"/>
+      <mass value="1e-5" />
+      <origin xyz="0 0 0" rpy="0 0 0" />
+      <inertia ixx="1e-6" ixy="0" ixz="0" iyy="1e-6" iyz="0" izz="1e-6" />
     </inertial>
   </link>
-  <xacro:include filename="$(find mrover)/urdf/rover/rover_gazebo_plugins.urdf.xacro"/>
-  <xacro:wheel side="left" reflect="1"/>
-  <xacro:wheel side="right" reflect="-1"/>
+  <xacro:include filename="$(find mrover)/urdf/rover/rover_gazebo_plugins.urdf.xacro" />
+  <xacro:wheel side="left" reflect="1" />
+  <xacro:wheel side="right" reflect="-1" />
 </robot>

File: urdf/rover/rover_gazebo_plugins.urdf.xacro (robot description, xacro)
@@ -21,5 +21,5 @@
     <plugin name="rover_gps_left" filename="libhector_gazebo_ros_gps.so">
       <updateRate>100.0</updateRate>
-      <bodyName>rover_gps_left_link</bodyName>
+      <bodyName>rover_gps_left</bodyName>
       <frameId></frameId>
       <topicName>gps/fix_gps_left</topicName>
@@ -38,5 +38,5 @@
     <plugin name="rover_gps_right" filename="libhector_gazebo_ros_gps.so">
       <updateRate>100.0</updateRate>
-      <bodyName>rover_gps_right_link</bodyName>
+      <bodyName>rover_gps_right</bodyName>
       <frameId></frameId>
       <topicName>gps/fix_gps_right</topicName>

Commit message: gps creation and subscribers

File: urdf/rover/rover.urdf.xacro (robot description, xacro)
@@ -133,5 +133,6 @@
     <child link="gps_link" />
   </joint>
-  <link name="gps_link" />
+  <link name="gps_link">
+  </link>
   <!-- Camera -->
   <joint name="camera_joint" type="fixed">

File: urdf/rover/rover_gazebo_plugins.urdf.xacro (robot description, xacro)
@@ -19,8 +19,8 @@
     </plugin>
     <!-- Rover GPS Left -->
-    <plugin name="rover_gps_left" filename="libhector_gazebo_ros_gps.so">
+    <plugin name="gazebo_ros_gps" filename="libhector_gazebo_ros_gps.so">
       <updateRate>100.0</updateRate>
-      <bodyName>rover_gps_left</bodyName>
-      <frameId></frameId>
+      <bodyName>base_link</bodyName>
+      <frameId>base_link</frameId>
       <topicName>gps/fix_gps_left</topicName>
       <velocityTopicName>gps/fix_velocity</velocityTopicName>
@@ -36,8 +36,8 @@
     </plugin>
     <!-- Rover GPS Right -->
-    <plugin name="rover_gps_right" filename="libhector_gazebo_ros_gps.so">
+    <plugin name="gazebo_ros_gps" filename="libhector_gazebo_ros_gps.so">
       <updateRate>100.0</updateRate>
-      <bodyName>rover_gps_right</bodyName>
-      <frameId></frameId>
+      <bodyName>base_link</bodyName>
+      <frameId>base_link</frameId>
       <topicName>gps/fix_gps_right</topicName>
       <velocityTopicName>gps/fix_velocity</velocityTopicName>

Commit message: gps now put in sim

File: urdf/rover/rover.urdf.xacro (robot description, xacro)
@@ -120,19 +120,18 @@
     <child link="imu_link" />
   </joint>
-  <link name="imu_link" />
+  <link name="imu_link"/>
   <!-- GPS -->
+  <link name="rover_gps_left_link"/>
   <joint name="rover_gps_left" type="fixed">
+    <origin xyz="0 0.5 0" />
+    <parent link="chassis_link" />
+    <child link="rover_gps_left_link" />
+  </joint>
+  <link name="rover_gps_right_link"/>
+  <joint name="rover_gps_right" type="fixed">
     <origin xyz="0 -0.5 0" />
     <parent link="chassis_link" />
-    <child link="gps_link" />
+    <child link="rover_gps_right_link" />
   </joint>
-  <!-- <link name="rover_gps_right_link"/> -->
-  <joint name="rover_gps_right" type="fixed">
-    <origin xyz="0 0.5 0" />
-    <parent link="chassis_link" />
-    <child link="gps_link" />
-  </joint>
-  <link name="gps_link">
-  </link>
   <!-- Camera -->
   <joint name="camera_joint" type="fixed">

File: urdf/rover/rover_gazebo_plugins.urdf.xacro (robot description, xacro)
@@ -18,10 +18,10 @@
       <bodyName>base_link</bodyName>
     </plugin>
-    <!-- GPS -->
+    <!-- Rover GPS Left -->
     <plugin name="gazebo_ros_gps" filename="libhector_gazebo_ros_gps.so">
       <updateRate>100.0</updateRate>
-      <bodyName>base_link</bodyName>
-      <frameId>base_link</frameId>
-      <topicName>gps/fix</topicName>
+      <bodyName>rover_gps_left_link</bodyName>
+      <frameId>rover_gps_left_link</frameId>
+      <topicName>gps/fix/rover_gps_left</topicName>
       <velocityTopicName>gps/fix_velocity</velocityTopicName>
       <referenceLatitude>42.293195</referenceLatitude>
@@ -35,10 +35,10 @@
       <velocityGaussianNoise>0.2 0.2 0.2</velocityGaussianNoise>
     </plugin>
-    <!-- Rover GPS Left -->
+    <!-- Rover GPS Right -->
     <plugin name="gazebo_ros_gps" filename="libhector_gazebo_ros_gps.so">
       <updateRate>100.0</updateRate>
-      <bodyName>base_link</bodyName>
-      <frameId>base_link</frameId>
-      <topicName>gps/fix_gps_left</topicName>
+      <bodyName>rover_gps_right_link</bodyName>
+      <frameId>rover_gps_right_link</frameId>
+      <topicName>gps/fix/rover_gps_right</topicName>
       <velocityTopicName>gps/fix_velocity</velocityTopicName>
       <referenceLatitude>42.293195</referenceLatitude>
@@ -47,21 +47,4 @@
       <referenceAltitude>0.0</referenceAltitude>
       <offset>0 0.5 0</offset>
-      <drift>0.0 0.0 0.0</drift>
-      <gaussianNoise>0 0 0</gaussianNoise>
-      <velocityDrift>0.0 0.0 0.0</velocityDrift>
-      <velocityGaussianNoise>0.2 0.2 0.2</velocityGaussianNoise>
-    </plugin>
-    <!-- Rover GPS Right -->
-    <plugin name="gazebo_ros_gps" filename="libhector_gazebo_ros_gps.so">
-      <updateRate>100.0</updateRate>
-      <bodyName>base_link</bodyName>
-      <frameId>base_link</frameId>
-      <topicName>gps/fix_gps_right</topicName>
-      <velocityTopicName>gps/fix_velocity</velocityTopicName>
-      <referenceLatitude>42.293195</referenceLatitude>
-      <referenceLongitude>-83.7096706</referenceLongitude>
-      <referenceHeading>90.0</referenceHeading>
-      <referenceAltitude>0.0</referenceAltitude>
-      <offset>0 -0.5 0</offset>
       <drift>0.0 0.0 0.0</drift>
       <gaussianNoise>0 0 0</gaussianNoise>

Commit message: tests for offset

File: urdf/rover/rover.urdf.xacro (robot description, xacro)
@@ -120,15 +120,15 @@
     <child link="imu_link" />
   </joint>
-  <link name="imu_link"/>
+  <link name="imu_link" />
   <!-- GPS -->
-  <link name="rover_gps_left_link"/>
+  <link name="rover_gps_left_link" />
   <joint name="rover_gps_left" type="fixed">
-    <origin xyz="0 0.5 0" />
+    <origin xyz="0 0 0" />
     <parent link="chassis_link" />
     <child link="rover_gps_left_link" />
   </joint>
-  <link name="rover_gps_right_link"/>
+  <link name="rover_gps_right_link" />
   <joint name="rover_gps_right" type="fixed">
-    <origin xyz="0 -0.5 0" />
+    <origin xyz="0 1 0" />
     <parent link="chassis_link" />
     <child link="rover_gps_right_link" />

File: urdf/rover/rover_gazebo_plugins.urdf.xacro (robot description, xacro)
@@ -25,6 +25,6 @@
       <topicName>gps/fix/rover_gps_left</topicName>
       <velocityTopicName>gps/fix_velocity</velocityTopicName>
-      <referenceLatitude>42.293195</referenceLatitude>
-      <referenceLongitude>-83.7096706</referenceLongitude>
+      <referenceLatitude>42.2931950000000000000000</referenceLatitude>
+      <referenceLongitude>-83.80967060000000000000000</referenceLongitude>
       <referenceHeading>90.0</referenceHeading>
       <referenceAltitude>0.0</referenceAltitude>
@@ -42,6 +42,6 @@
       <topicName>gps/fix/rover_gps_right</topicName>
       <velocityTopicName>gps/fix_velocity</velocityTopicName>
-      <referenceLatitude>42.293195</referenceLatitude>
-      <referenceLongitude>-83.7096706</referenceLongitude>
+      <referenceLatitude>42.2931950000000000000000</referenceLatitude>
+      <referenceLongitude>-83.80967060000000000000000</referenceLongitude>
       <referenceHeading>90.0</referenceHeading>
       <referenceAltitude>0.0</referenceAltitude>

Commit message: offset is 10?

File: urdf/rover/rover.urdf.xacro (robot description, xacro)
@@ -130,5 +130,5 @@
   <link name="rover_gps_right_link" />
   <joint name="rover_gps_right" type="fixed">
-    <origin xyz="0 1 0" />
+    <origin xyz="0 10 0" />
     <parent link="chassis_link" />
     <child link="rover_gps_right_link" />

File: urdf/rover/rover_gazebo_plugins.urdf.xacro (robot description, xacro)
@@ -46,5 +46,5 @@
       <referenceHeading>90.0</referenceHeading>
       <referenceAltitude>0.0</referenceAltitude>
-      <offset>0 0 0</offset>
+      <offset>0 10 0</offset>
       <drift>0.0 0.0 0.0</drift>
       <gaussianNoise>0 0 0</gaussianNoise>

Commit message: chanegd offset to 1 and modified testing code

File: urdf/rover/rover.urdf.xacro (robot description, xacro)
@@ -130,5 +130,5 @@
   <link name="rover_gps_right_link" />
   <joint name="rover_gps_right" type="fixed">
-    <origin xyz="0 10 0" />
+    <origin xyz="0 1 0" />
     <parent link="chassis_link" />
     <child link="rover_gps_right_link" />

File: urdf/rover/rover_gazebo_plugins.urdf.xacro (robot description, xacro)
@@ -46,5 +46,5 @@
       <referenceHeading>90.0</referenceHeading>
       <referenceAltitude>0.0</referenceAltitude>
-      <offset>0 10 0</offset>
+      <offset>0 1 0</offset>
       <drift>0.0 0.0 0.0</drift>
       <gaussianNoise>0 0 0</gaussianNoise>

Commit message: Bind buffers

File: urdf/rover/rover.urdf.xacro (robot description, xacro)
@@ -18,5 +18,6 @@
     <inertial>
       <mass value="${m}"/>
-      <inertia ixx="${m / 12.0 * (d*d + h*h)}" ixy="0.0" ixz="0.0" iyy="${m / 12.0 * (w*w + h*h)}" iyz="0.0" izz="${m / 12.0 * (w*w + d*d)}"/>
+      <inertia ixx="${m / 12.0 * (d*d + h*h)}" ixy="0.0" ixz="0.0" iyy="${m / 12.0 * (w*w + h*h)}" iyz="0.0"
+               izz="${m / 12.0 * (w*w + d*d)}"/>
     </inertial>
   </xacro:macro>
@@ -24,5 +25,6 @@
     <inertial>
       <mass value="${m}"/>
-      <inertia ixx="${2.0*m*(r*r)/5.0}" ixy="0.0" ixz="0.0" iyy="${2.0*m*(r*r)/5.0}" iyz="0.0" izz="${2.0*m*(r*r)/5.0}"/>
+      <inertia ixx="${2.0*m*(r*r)/5.0}" ixy="0.0" ixz="0.0" iyy="${2.0*m*(r*r)/5.0}" iyz="0.0"
+               izz="${2.0*m*(r*r)/5.0}"/>
     </inertial>
   </xacro:macro>
@@ -162,5 +164,5 @@
     </inertial>
   </link>
-  <xacro:include filename="$(find mrover)/urdf/rover/rover_gazebo_plugins.urdf.xacro"/>
+  <!--  <xacro:include filename="$(find mrover)/urdf/rover/rover_gazebo_plugins.urdf.xacro"/>-->
   <xacro:wheel side="left" reflect="1"/>
   <xacro:wheel side="right" reflect="-1"/>

Commit message: GLB testing

File: urdf/rover/rover.urdf.xacro (robot description, xacro)
@@ -36,5 +36,5 @@
       <origin rpy="0 0 0" xyz="0 0 0"/>
       <geometry>
-        <mesh filename="package://mrover/urdf/meshes/rover.dae"/>
+        <mesh filename="package://mrover/urdf/meshes/rover2.glb"/>
       </geometry>
     </visual>
@@ -48,10 +48,10 @@
     <link name="front_${side}_wheel_link">
       <xacro:sphere_inertia m="${wheel_mass}" r="${wheel_radius}"/>
-      <visual>
-        <origin rpy="0 ${min(0, reflect) * PI} 0" xyz="0 0 0"/>
-        <geometry>
-          <mesh filename="package://mrover/urdf/meshes/rover.wheel.dae"/>
-        </geometry>
-      </visual>
+<!--      <visual>-->
+<!--        <origin rpy="0 ${min(0, reflect) * PI} 0" xyz="0 0 0"/>-->
+<!--        <geometry>-->
+<!--          <mesh filename="package://mrover/urdf/meshes/rover.wheel.dae"/>-->
+<!--        </geometry>-->
+<!--      </visual>-->
       <collision>
         <geometry>
@@ -62,10 +62,10 @@
     <link name="center_${side}_wheel_link">
       <xacro:cylinder_inertia m="${wheel_mass}" r="${wheel_radius}" h="${wheel_width}"/>
-      <visual>
-        <origin rpy="0 ${min(0, reflect) * PI} 0" xyz="0 0 0"/>
-        <geometry>
-          <mesh filename="package://mrover/urdf/meshes/rover.wheel.dae"/>
-        </geometry>
-      </visual>
+<!--      <visual>-->
+<!--        <origin rpy="0 ${min(0, reflect) * PI} 0" xyz="0 0 0"/>-->
+<!--        <geometry>-->
+<!--          <mesh filename="package://mrover/urdf/meshes/rover.wheel.dae"/>-->
+<!--        </geometry>-->
+<!--      </visual>-->
       <collision>
         <geometry>
@@ -76,10 +76,10 @@
     <link name="back_${side}_wheel_link">
       <xacro:sphere_inertia m="${wheel_mass}" r="${wheel_radius}"/>
-      <visual>
-        <origin rpy="0 ${min(0, reflect) * PI} 0" xyz="0 0 0"/>
-        <geometry>
-          <mesh filename="package://mrover/urdf/meshes/rover.wheel.dae"/>
-        </geometry>
-      </visual>
+<!--      <visual>-->
+<!--        <origin rpy="0 ${min(0, reflect) * PI} 0" xyz="0 0 0"/>-->
+<!--        <geometry>-->
+<!--          <mesh filename="package://mrover/urdf/meshes/rover.wheel.dae"/>-->
+<!--        </geometry>-->
+<!--      </visual>-->
       <collision>
         <geometry>
@@ -133,10 +133,10 @@
       </geometry>
     </collision>
-    <visual>
-      <origin xyz="0 0 0" rpy="0 0 0"/>
-      <geometry>
-        <mesh filename="package://mrover/urdf/meshes/zed2i.dae"/>
-      </geometry>
-    </visual>
+<!--    <visual>-->
+<!--      <origin xyz="0 0 0" rpy="0 0 0"/>-->
+<!--      <geometry>-->
+<!--        <mesh filename="package://mrover/urdf/meshes/zed2i.dae"/>-->
+<!--      </geometry>-->
+<!--    </visual>-->
     <inertial>
       <mass value="1e-5"/>
