Commit message: Kinda working

File: urdf/rover/rover.urdf.xacro (robot description, xacro)
@@ -1,11 +1,11 @@
 <?xml version="1.0"?>
 <robot xmlns:xacro="http://www.ros.org/wiki/xacro" name="rover">
-  <xacro:property name="base_width" value="0.7357"/>
-  <xacro:property name="base_len" value="1.0"/>
-  <xacro:property name="base_height" value="0.4"/>
+  <xacro:property name="base_width" value="0.553"/>
+  <xacro:property name="base_len" value="0.482"/>
+  <xacro:property name="base_height" value="0.186"/>
   <xacro:property name="wheel_radius" value="0.13"/>
   <xacro:property name="wheel_width" value="0.1"/>
   <xacro:property name="wheel_mass" value="1"/>
-  <xacro:property name="chassis_mass" value="30"/>
+  <xacro:property name="chassis_mass" value="10"/>
   <xacro:property name="PI" value="3.141592"/>
   <!-- Inertial macros-->
@@ -19,5 +19,5 @@
     <inertial>
       <mass value="${m}"/>
-      <inertia ixx="${m / 12.0 * (d*d + h*h)}" ixy="0.0" ixz="0.0" iyy="${m / 12.0 * (w*w + h*h)}" iyz="0.0"
+      <inertia ixx="${m / 12.0 * (d*d + h*h)}" ixy="0" ixz="0" iyy="${m / 12.0 * (w*w + h*h)}" iyz="0"
                izz="${m / 12.0 * (w*w + d*d)}"/>
     </inertial>
@@ -26,5 +26,5 @@
     <inertial>
       <mass value="${m}"/>
-      <inertia ixx="${2.0*m*(r*r)/5.0}" ixy="0.0" ixz="0.0" iyy="${2.0*m*(r*r)/5.0}" iyz="0.0"
+      <inertia ixx="${2.0*m*(r*r)/5.0}" ixy="0" ixz="0" iyy="${2.0*m*(r*r)/5.0}" iyz="0"
                izz="${2.0*m*(r*r)/5.0}"/>
     </inertial>
@@ -35,9 +35,9 @@
   <link name="chassis_link">
     <xacro:box_inertia m="${chassis_mass}" w="${base_len}" h="${base_width}" d="${base_height}"/>
-    <visual>
-      <geometry>
-        <mesh filename="package://mrover/urdf/meshes/cube.glb"/>
-      </geometry>
-    </visual>
+    <!--    <visual>-->
+    <!--      <geometry>-->
+    <!--        <mesh filename="package://mrover/urdf/meshes/cube.glb"/>-->
+    <!--      </geometry>-->
+    <!--    </visual>-->
     <collision>
       <geometry>
@@ -46,5 +46,5 @@
     </collision>
   </link>
-  <xacro:macro name="wheel" params="name reflect xyz">
+  <xacro:macro name="wheel" params="name reflect">
     <link name="${name}_wheel_link">
       <xacro:cylinder_inertia m="${wheel_mass}" r="${wheel_radius}" h="${wheel_width}"/>
@@ -69,25 +69,82 @@
       </collision>
     </link>
-    <joint name="${name}_axle_joint" type="continuous">
-      <parent link="chassis_link"/>
-      <child link="${name}_axle_link"/>
-      <origin xyz="${xyz}" rpy="${-PI/2} 0 0"/>
-      <axis xyz="0 0 1"/>
-    </joint>
-    <joint name="${name}_wheel_joint" type="continuous">
+    <joint name="${name}_axle_link_to_${name}_wheel_link" type="continuous">
       <parent link="${name}_axle_link"/>
       <child link="${name}_wheel_link"/>
-      <origin xyz="0 0 0" rpy="0 0 0"/>
-      <axis xyz="0 0 1"/>
+      <axis xyz="0 0 1"/>
+      <limit effort="2.68" velocity="0"/>
     </joint>
   </xacro:macro>
   <xacro:macro name="wheels" params="side reflect">
-    <xacro:wheel name="front_${side}" reflect="${reflect}" xyz="0.42 ${reflect * (base_width/2 + 0.06)} -0.373"/>
-    <xacro:wheel name="center_${side}" reflect="${reflect}" xyz="0 ${reflect * (base_width/2 + 0.06)} -0.373"/>
-    <xacro:wheel name="back_${side}" reflect="${reflect}" xyz="-0.42 ${reflect * (base_width/2 + 0.06)} -0.373"/>
+    <xacro:wheel name="front_${side}" reflect="${reflect}"/>
+    <xacro:wheel name="center_${side}" reflect="${reflect}"/>
+    <xacro:wheel name="back_${side}" reflect="${reflect}"/>
+    <link name="${side}_bogie_link">
+      <xacro:box_inertia m="2" w="0.5" h="0.5" d="0.5"/>
+      <collision>
+        <origin xyz="-0.14 0.1 0" rpy="0 0 -0.734"/>
+        <geometry>
+          <box size="0.2 0.025 0.025"/>
+        </geometry>
+      </collision>
+      <collision>
+        <origin xyz="0.1 0.088 0" rpy="0 0 0.734"/>
+        <geometry>
+          <box size="0.2 0.025 0.025"/>
+        </geometry>
+      </collision>
+    </link>
+    <link name="${side}_rocker_link">
+      <xacro:box_inertia m="2" w="0.5" h="0.5" d="0.5"/>
+      <collision>
+        <origin xyz="-0.11 0.077 0" rpy="0 0 -0.585"/>
+        <geometry>
+          <box size="0.2 0.025 0.025"/>
+        </geometry>
+      </collision>
+      <collision>
+        <origin xyz="0.22 0.15 0" rpy="0 0 0.585"/>
+        <geometry>
+          <box size="0.5 0.025 0.025"/>
+        </geometry>
+      </collision>
+    </link>
+    <joint name="chassis_link_to_${side}_rocker_link" type="revolute">
+      <parent link="chassis_link"/>
+      <child link="${side}_rocker_link"/>
+      <origin xyz="0.17 ${reflect * (base_width/2 + 0.05)} 0" rpy="${-PI/2} 0 0"/>
+      <axis xyz="0 0 1"/>
+      0.349066
+      <limit lower="-0.122173" upper="0.523599" effort="0" velocity="0"/>
+    </joint>
+    <joint name="${side}_rocker_link_to_front_${side}_axle_link" type="continuous">
+      <parent link="${side}_rocker_link"/>
+      <child link="front_${side}_axle_link"/>
+      <origin xyz="0.42 0.286 ${reflect * 0.05}"/>
+      <axis xyz="0 0 1"/>
+    </joint>
+    <joint name="${side}_rocker_link_to_${side}_bogie_link" type="revolute">
+      <parent link="${side}_rocker_link"/>
+      <child link="${side}_bogie_link"/>
+      <origin xyz="-0.202 0.134 0"/>
+      <axis xyz="0 0 1"/>
+      <limit lower="-0.349066" upper="0.349066" effort="0" velocity="0"/>
+    </joint>
+    <joint name="${side}_bogie_link_to_center_${side}_axle_link" type="continuous">
+      <parent link="${side}_bogie_link"/>
+      <child link="center_${side}_axle_link"/>
+      <origin xyz="0.174 0.157 ${reflect * 0.05}"/>
+      <axis xyz="0 0 1"/>
+    </joint>
+    <joint name="${side}_bogie_link_to_back_${side}_axle_link" type="continuous">
+      <parent link="${side}_bogie_link"/>
+      <child link="back_${side}_axle_link"/>
+      <origin xyz="-0.221 0.157 ${reflect * 0.05}"/>
+      <axis xyz="0 0 1"/>
+    </joint>
   </xacro:macro>
   <!-- Joints -->
-  <joint name="base_link_to_chassis" type="fixed">
-    <origin xyz="0 0 0.5"/>
+  <joint name="base_link_to_chassis_link" type="fixed">
+    <origin xyz="0 0 0.42"/>
     <parent link="base_link"/>
     <child link="chassis_link"/>

Commit message: Tweak mass values

File: urdf/rover/rover.urdf.xacro (robot description, xacro)
@@ -7,5 +7,5 @@
   <xacro:property name="wheel_width" value="0.1"/>
   <xacro:property name="wheel_mass" value="1"/>
-  <xacro:property name="chassis_mass" value="10"/>
+  <xacro:property name="chassis_mass" value="15"/>
   <xacro:property name="PI" value="3.141592"/>
   <!-- Inertial macros-->
@@ -62,5 +62,5 @@
     </link>
     <link name="${name}_axle_link">
-      <xacro:cylinder_inertia m="1.0" r="0.01" h="0.1"/>
+      <xacro:cylinder_inertia m="1" r="0.01" h="0.1"/>
       <collision>
         <geometry>
@@ -81,5 +81,5 @@
     <xacro:wheel name="back_${side}" reflect="${reflect}"/>
     <link name="${side}_bogie_link">
-      <xacro:box_inertia m="2" w="0.5" h="0.5" d="0.5"/>
+      <xacro:box_inertia m="3" w="0.5" h="0.5" d="0.5"/>
       <collision>
         <origin xyz="-0.14 0.1 0" rpy="0 0 -0.734"/>
@@ -96,5 +96,5 @@
     </link>
     <link name="${side}_rocker_link">
-      <xacro:box_inertia m="2" w="0.5" h="0.5" d="0.5"/>
+      <xacro:box_inertia m="3" w="0.5" h="0.5" d="0.5"/>
       <collision>
         <origin xyz="-0.11 0.077 0" rpy="0 0 -0.585"/>

Commit message: Switch rocker and bogie

File: urdf/rover/rover.urdf.xacro (robot description, xacro)
@@ -98,5 +98,5 @@
       <xacro:box_inertia m="3" w="0.5" h="0.5" d="0.5"/>
       <collision>
-        <origin xyz="-0.11 0.077 0" rpy="0 0 -0.585"/>
+        <origin xyz="0.11 0.077 0" rpy="0 0 0.585"/>
         <geometry>
           <box size="0.2 0.025 0.025"/>
@@ -104,5 +104,5 @@
       </collision>
       <collision>
-        <origin xyz="0.22 0.15 0" rpy="0 0 0.585"/>
+        <origin xyz="-0.22 0.15 0" rpy="0 0 -0.585"/>
         <geometry>
           <box size="0.5 0.025 0.025"/>
@@ -113,13 +113,12 @@
       <parent link="chassis_link"/>
       <child link="${side}_rocker_link"/>
-      <origin xyz="0.17 ${reflect * (base_width/2 + 0.05)} 0" rpy="${-PI/2} 0 0"/>
-      <axis xyz="0 0 1"/>
-      0.349066
+      <origin xyz="0.17 ${reflect * (base_width/2 + 0.03)} 0" rpy="${-PI/2} 0 0"/>
+      <axis xyz="0 0 1"/>
       <limit lower="-0.122173" upper="0.523599" effort="0" velocity="0"/>
     </joint>
-    <joint name="${side}_rocker_link_to_front_${side}_axle_link" type="continuous">
+    <joint name="${side}_rocker_link_to_back_${side}_axle_link" type="continuous">
       <parent link="${side}_rocker_link"/>
-      <child link="front_${side}_axle_link"/>
-      <origin xyz="0.42 0.286 ${reflect * 0.05}"/>
+      <child link="back_${side}_axle_link"/>
+      <origin xyz="-0.42 0.286 ${reflect * 0.07}"/>
       <axis xyz="0 0 1"/>
     </joint>
@@ -127,18 +126,18 @@
       <parent link="${side}_rocker_link"/>
       <child link="${side}_bogie_link"/>
-      <origin xyz="-0.202 0.134 0"/>
+      <origin xyz="0.202 0.134 0"/>
       <axis xyz="0 0 1"/>
       <limit lower="-0.349066" upper="0.349066" effort="0" velocity="0"/>
+    </joint>
+    <joint name="${side}_bogie_link_to_front_${side}_axle_link" type="continuous">
+      <parent link="${side}_bogie_link"/>
+      <child link="front_${side}_axle_link"/>
+      <origin xyz="0.174 0.157 ${reflect * 0.07}"/>
+      <axis xyz="0 0 1"/>
     </joint>
     <joint name="${side}_bogie_link_to_center_${side}_axle_link" type="continuous">
       <parent link="${side}_bogie_link"/>
       <child link="center_${side}_axle_link"/>
-      <origin xyz="0.174 0.157 ${reflect * 0.05}"/>
-      <axis xyz="0 0 1"/>
-    </joint>
-    <joint name="${side}_bogie_link_to_back_${side}_axle_link" type="continuous">
-      <parent link="${side}_bogie_link"/>
-      <child link="back_${side}_axle_link"/>
-      <origin xyz="-0.221 0.157 ${reflect * 0.05}"/>
+      <origin xyz="-0.221 0.157 ${reflect * 0.07}"/>
       <axis xyz="0 0 1"/>
     </joint>

Commit message: Sigh

File: urdf/rover/rover.urdf.xacro (robot description, xacro)
@@ -120,5 +120,5 @@
       <parent link="${side}_rocker_link"/>
       <child link="back_${side}_axle_link"/>
-      <origin xyz="-0.42 0.286 ${reflect * 0.07}"/>
+      <origin xyz="-0.42 0.286 ${reflect * 0.08}"/>
       <axis xyz="0 0 1"/>
     </joint>
@@ -133,5 +133,5 @@
       <parent link="${side}_bogie_link"/>
       <child link="front_${side}_axle_link"/>
-      <origin xyz="0.174 0.157 ${reflect * 0.07}"/>
+      <origin xyz="0.174 0.157 ${reflect * 0.08}"/>
       <axis xyz="0 0 1"/>
     </joint>
@@ -139,5 +139,5 @@
       <parent link="${side}_bogie_link"/>
       <child link="center_${side}_axle_link"/>
-      <origin xyz="-0.221 0.157 ${reflect * 0.07}"/>
+      <origin xyz="-0.221 0.157 ${reflect * 0.08}"/>
       <axis xyz="0 0 1"/>
     </joint>

Commit message: Tune mass

File: urdf/rover/rover.urdf.xacro (robot description, xacro)
@@ -6,5 +6,5 @@
   <xacro:property name="wheel_radius" value="0.13"/>
   <xacro:property name="wheel_width" value="0.1"/>
-  <xacro:property name="wheel_mass" value="1"/>
+  <xacro:property name="wheel_mass" value="0.8"/>
   <xacro:property name="chassis_mass" value="15"/>
   <xacro:property name="PI" value="3.141592"/>
@@ -62,8 +62,8 @@
     </link>
     <link name="${name}_axle_link">
-      <xacro:cylinder_inertia m="1" r="0.01" h="0.1"/>
-      <collision>
-        <geometry>
-          <cylinder length="0.1" radius="0.01"/>
+      <xacro:cylinder_inertia m="2" r="0.01" h="0.075"/>
+      <collision>
+        <geometry>
+          <cylinder length="0.075" radius="0.01"/>
         </geometry>
       </collision>
@@ -113,5 +113,5 @@
       <parent link="chassis_link"/>
       <child link="${side}_rocker_link"/>
-      <origin xyz="0.17 ${reflect * (base_width/2 + 0.03)} 0" rpy="${-PI/2} 0 0"/>
+      <origin xyz="0.17 ${reflect * (base_width/2 + 0.05)} 0" rpy="${-PI/2} 0 0"/>
       <axis xyz="0 0 1"/>
       <limit lower="-0.122173" upper="0.523599" effort="0" velocity="0"/>
@@ -120,5 +120,5 @@
       <parent link="${side}_rocker_link"/>
       <child link="back_${side}_axle_link"/>
-      <origin xyz="-0.42 0.286 ${reflect * 0.08}"/>
+      <origin xyz="-0.42 0.286 ${reflect * 0.09}"/>
       <axis xyz="0 0 1"/>
     </joint>
@@ -133,5 +133,5 @@
       <parent link="${side}_bogie_link"/>
       <child link="front_${side}_axle_link"/>
-      <origin xyz="0.174 0.157 ${reflect * 0.08}"/>
+      <origin xyz="0.174 0.157 ${reflect * 0.09}"/>
       <axis xyz="0 0 1"/>
     </joint>
@@ -139,5 +139,5 @@
       <parent link="${side}_bogie_link"/>
       <child link="center_${side}_axle_link"/>
-      <origin xyz="-0.221 0.157 ${reflect * 0.08}"/>
+      <origin xyz="-0.221 0.157 ${reflect * 0.09}"/>
       <axis xyz="0 0 1"/>
     </joint>
