Commit message: Add arm

File: urdf/rover/rover.urdf.xacro (robot description, xacro)
@@ -1,7 +1,8 @@
 <?xml version="1.0"?>
 <robot xmlns:xacro="http://www.ros.org/wiki/xacro" name="rover">
-  <xacro:property name="base_width" value="0.553"/>
-  <xacro:property name="base_len" value="0.482"/>
-  <xacro:property name="base_height" value="0.186"/>
+  <!-- Constants -->
+  <xacro:property name="base_width" value="0.63"/>
+  <xacro:property name="base_len" value="0.478"/>
+  <xacro:property name="base_height" value="0.183"/>
   <xacro:property name="wheel_radius" value="0.13"/>
   <xacro:property name="wheel_width" value="0.1"/>
@@ -10,16 +11,19 @@
   <xacro:property name="wheel_torque" value="2.68"/>
   <xacro:property name="TAU" value="6.2831855"/>
-  <!-- Inertial macros-->
+  <!-- Inertial Macros-->
   <xacro:macro name="cylinder_inertia" params="m r h">
     <inertial>
       <mass value="${m}"/>
-      <inertia ixx="${m*(3*r*r+h*h)/12}" ixy="0" ixz="0" iyy="${m*(3*r*r+h*h)/12}" iyz="0" izz="${m*r*r/2}"/>
+      <inertia ixx="${m*(3*r*r+h*h)/12}" ixy="0" ixz="0"
+               iyy="${m*(3*r*r+h*h)/12}" iyz="0"
+               izz="${m*r*r/2}"/>
     </inertial>
   </xacro:macro>
-  <xacro:macro name="box_inertia" params="m w h d">
+  <xacro:macro name="box_inertia" params="m d w h">
     <inertial>
       <mass value="${m}"/>
-      <inertia ixx="${m / 12.0 * (d*d + h*h)}" ixy="0" ixz="0" iyy="${m / 12.0 * (w*w + h*h)}" iyz="0"
-               izz="${m / 12.0 * (w*w + d*d)}"/>
+      <inertia ixx="${m / 12.0 * (w*w + h*h)}" ixy="0" ixz="0"
+               iyy="${m / 12.0 * (d*d + h*h)}" iyz="0"
+               izz="${m / 12.0 * (d*d + w*w)}"/>
     </inertial>
   </xacro:macro>
@@ -27,13 +31,145 @@
     <inertial>
       <mass value="${m}"/>
-      <inertia ixx="${2.0*m*(r*r)/5.0}" ixy="0" ixz="0" iyy="${2.0*m*(r*r)/5.0}" iyz="0"
+      <inertia ixx="${2.0*m*(r*r)/5.0}" ixy="0" ixz="0"
+               iyy="${2.0*m*(r*r)/5.0}" iyz="0"
                izz="${2.0*m*(r*r)/5.0}"/>
     </inertial>
   </xacro:macro>
-  <!-- Links -->
+  <!-- Joints/Links Macros -->
+  <xacro:macro name="arm_link" params="name m x y z">
+    <link name="arm_${name}_link">
+      <xacro:box_inertia m="${m}" d="${y}" w="${x}" h="${z}"/>
+      <visual>
+        <geometry>
+          <mesh filename="package://mrover/urdf/meshes/arm_${name}.fbx"/>
+        </geometry>
+      </visual>
+      <collision>
+        <geometry>
+          <box size="${x} ${y} ${z}"/>
+        </geometry>
+      </collision>
+    </link>
+  </xacro:macro>
+  <xacro:macro name="arm_revolute_joint" params="parent child x y z">
+    <joint name="${parent}_link_to_${child}_link" type="revolute">
+      <origin xyz="${x} ${y} ${z}"/>
+      <parent link="${parent}_link"/>
+      <child link="${child}_link"/>
+      <axis xyz="0 1 0"/>
+      <limit lower="-0.523599" upper="0.523599" effort="0" velocity="0"/>
+    </joint>
+  </xacro:macro>
+  <xacro:macro name="wheel" params="pos side reflect">
+    <link name="${pos}_${side}_wheel_link">
+      <xacro:cylinder_inertia m="${wheel_mass}" r="${wheel_radius}" h="${wheel_width}"/>
+      <visual>
+        <geometry>
+          <mesh filename="package://mrover/urdf/meshes/rover_${side}_wheel.fbx"/>
+        </geometry>
+      </visual>
+      <collision>
+        <geometry>
+          <cylinder length="${wheel_width}" radius="${wheel_radius}"/>
+        </geometry>
+      </collision>
+    </link>
+    <link name="${pos}_${side}_axle_link">
+      <xacro:cylinder_inertia m="2.5" r="0.05" h="0.075"/>
+      <collision>
+        <geometry>
+          <cylinder length="0.075" radius="0.05"/>
+        </geometry>
+      </collision>
+    </link>
+    <joint name="${pos}_${side}_axle_link_to_${pos}_${side}_wheel_link" type="continuous">
+      <parent link="${pos}_${side}_axle_link"/>
+      <child link="${pos}_${side}_wheel_link"/>
+      <axis xyz="0 0 1"/>
+      <limit effort="${wheel_torque}" velocity="0"/>
+    </joint>
+  </xacro:macro>
+  <xacro:macro name="wheels" params="side reflect">
+    <xacro:wheel pos="front" side="${side}" reflect="${reflect}"/>
+    <xacro:wheel pos="center" side="${side}" reflect="${reflect}"/>
+    <xacro:wheel pos="back" side="${side}" reflect="${reflect}"/>
+    <link name="${side}_bogie_link">
+      <xacro:box_inertia m="3" d="0.5" w="0.5" h="0.5"/>
+      <visual>
+        <geometry>
+          <mesh filename="package://mrover/urdf/meshes/rover_${side}_bogie.fbx"/>
+        </geometry>
+      </visual>
+      <collision>
+        <origin xyz="-0.14 0.1 0" rpy="0 0 -0.734"/>
+        <geometry>
+          <box size="0.2 0.025 0.025"/>
+        </geometry>
+      </collision>
+      <collision>
+        <origin xyz="0.1 0.088 0" rpy="0 0 0.734"/>
+        <geometry>
+          <box size="0.2 0.025 0.025"/>
+        </geometry>
+      </collision>
+    </link>
+    <link name="${side}_rocker_link">
+      <xacro:box_inertia m="3" d="0.5" w="0.5" h="0.5"/>
+      <visual>
+        <geometry>
+          <mesh filename="package://mrover/urdf/meshes/rover_${side}_rocker.fbx"/>
+        </geometry>
+      </visual>
+      <collision>
+        <origin xyz="0.11 0.077 0" rpy="0 0 0.585"/>
+        <geometry>
+          <box size="0.2 0.025 0.025"/>
+        </geometry>
+      </collision>
+      <collision>
+        <origin xyz="-0.22 0.15 0" rpy="0 0 -0.585"/>
+        <geometry>
+          <box size="0.5 0.025 0.025"/>
+        </geometry>
+      </collision>
+    </link>
+    <joint name="chassis_link_to_${side}_rocker_link" type="revolute">
+      <parent link="chassis_link"/>
+      <child link="${side}_rocker_link"/>
+      <origin xyz="0.164665 ${reflect * (base_width/2 + 0.05)} 0" rpy="${-TAU/4} 0 0"/>
+      <axis xyz="0 0 1"/>
+      <limit lower="-0.122173" upper="0.523599" effort="0" velocity="0"/>
+    </joint>
+    <joint name="${side}_rocker_link_to_back_${side}_axle_link" type="continuous">
+      <parent link="${side}_rocker_link"/>
+      <child link="back_${side}_axle_link"/>
+      <origin xyz="-0.417094 0.28513 ${reflect * 0.09}"/>
+      <axis xyz="0 0 1"/>
+    </joint>
+    <joint name="${side}_rocker_link_to_${side}_bogie_link" type="revolute">
+      <parent link="${side}_rocker_link"/>
+      <child link="${side}_bogie_link"/>
+      <origin xyz="0.198948 0.138674 0"/>
+      <axis xyz="0 0 1"/>
+      <limit lower="-0.349066" upper="0.349066" effort="0" velocity="0"/>
+    </joint>
+    <joint name="${side}_bogie_link_to_front_${side}_axle_link" type="continuous">
+      <parent link="${side}_bogie_link"/>
+      <child link="front_${side}_axle_link"/>
+      <origin xyz="0.215233 0.147933 ${reflect * 0.09}"/>
+      <axis xyz="0 0 1"/>
+    </joint>
+    <joint name="${side}_bogie_link_to_center_${side}_axle_link" type="continuous">
+      <parent link="${side}_bogie_link"/>
+      <child link="center_${side}_axle_link"/>
+      <origin xyz="-0.173532 0.147659 ${reflect * 0.09}"/>
+      <axis xyz="0 0 1"/>
+    </joint>
+  </xacro:macro>
+  <!-- Joints/Links -->
   <link name="base_link">
   </link>
   <link name="chassis_link">
-    <xacro:box_inertia m="${chassis_mass}" w="${base_len}" h="${base_width}" d="${base_height}"/>
+    <xacro:box_inertia m="${chassis_mass}" d="${base_len}" w="${base_width}" h="${base_height}"/>
     <visual>
       <geometry>
@@ -47,116 +183,28 @@
     </collision>
   </link>
-  <xacro:macro name="wheel" params="pos side reflect">
-    <link name="${pos}_${side}_wheel_link">
-      <xacro:cylinder_inertia m="${wheel_mass}" r="${wheel_radius}" h="${wheel_width}"/>
-      <visual>
-        <geometry>
-          <mesh filename="package://mrover/urdf/meshes/rover_${side}_wheel.fbx"/>
-        </geometry>
-      </visual>
-      <collision>
-        <geometry>
-          <cylinder length="${wheel_width}" radius="${wheel_radius}"/>
-        </geometry>
-      </collision>
-    </link>
-    <link name="${pos}_${side}_axle_link">
-      <xacro:cylinder_inertia m="2.5" r="0.05" h="0.075"/>
-      <collision>
-        <geometry>
-          <cylinder length="0.075" radius="0.05"/>
-        </geometry>
-      </collision>
-    </link>
-    <joint name="${pos}_${side}_axle_link_to_${pos}_${side}_wheel_link" type="continuous">
-      <parent link="${pos}_${side}_axle_link"/>
-      <child link="${pos}_${side}_wheel_link"/>
-      <axis xyz="0 0 1"/>
-      <limit effort="${wheel_torque}" velocity="0"/>
-    </joint>
-  </xacro:macro>
-  <xacro:macro name="wheels" params="side reflect">
-    <xacro:wheel pos="front" side="${side}" reflect="${reflect}"/>
-    <xacro:wheel pos="center" side="${side}" reflect="${reflect}"/>
-    <xacro:wheel pos="back" side="${side}" reflect="${reflect}"/>
-    <link name="${side}_bogie_link">
-      <xacro:box_inertia m="3" w="0.5" h="0.5" d="0.5"/>
-      <visual>
-        <geometry>
-          <mesh filename="package://mrover/urdf/meshes/rover_${side}_bogie.fbx"/>
-        </geometry>
-      </visual>
-      <collision>
-        <origin xyz="-0.14 0.1 0" rpy="0 0 -0.734"/>
-        <geometry>
-          <box size="0.2 0.025 0.025"/>
-        </geometry>
-      </collision>
-      <collision>
-        <origin xyz="0.1 0.088 0" rpy="0 0 0.734"/>
-        <geometry>
-          <box size="0.2 0.025 0.025"/>
-        </geometry>
-      </collision>
-    </link>
-    <link name="${side}_rocker_link">
-      <xacro:box_inertia m="3" w="0.5" h="0.5" d="0.5"/>
-      <visual>
-        <geometry>
-          <mesh filename="package://mrover/urdf/meshes/rover_${side}_rocker.fbx"/>
-        </geometry>
-      </visual>
-      <collision>
-        <origin xyz="0.11 0.077 0" rpy="0 0 0.585"/>
-        <geometry>
-          <box size="0.2 0.025 0.025"/>
-        </geometry>
-      </collision>
-      <collision>
-        <origin xyz="-0.22 0.15 0" rpy="0 0 -0.585"/>
-        <geometry>
-          <box size="0.5 0.025 0.025"/>
-        </geometry>
-      </collision>
-    </link>
-    <joint name="chassis_link_to_${side}_rocker_link" type="revolute">
-      <parent link="chassis_link"/>
-      <child link="${side}_rocker_link"/>
-      <origin xyz="0.17 ${reflect * (base_width/2 + 0.05)} 0" rpy="${-TAU/4} 0 0"/>
-      <axis xyz="0 0 1"/>
-      <limit lower="-0.122173" upper="0.523599" effort="0" velocity="0"/>
-    </joint>
-    <joint name="${side}_rocker_link_to_back_${side}_axle_link" type="continuous">
-      <parent link="${side}_rocker_link"/>
-      <child link="back_${side}_axle_link"/>
-      <origin xyz="-0.42 0.286 ${reflect * 0.09}"/>
-      <axis xyz="0 0 1"/>
-    </joint>
-    <joint name="${side}_rocker_link_to_${side}_bogie_link" type="revolute">
-      <parent link="${side}_rocker_link"/>
-      <child link="${side}_bogie_link"/>
-      <origin xyz="0.202 0.134 0"/>
-      <axis xyz="0 0 1"/>
-      <limit lower="-0.349066" upper="0.349066" effort="0" velocity="0"/>
-    </joint>
-    <joint name="${side}_bogie_link_to_front_${side}_axle_link" type="continuous">
-      <parent link="${side}_bogie_link"/>
-      <child link="front_${side}_axle_link"/>
-      <origin xyz="0.174 0.157 ${reflect * 0.09}"/>
-      <axis xyz="0 0 1"/>
-    </joint>
-    <joint name="${side}_bogie_link_to_center_${side}_axle_link" type="continuous">
-      <parent link="${side}_bogie_link"/>
-      <child link="center_${side}_axle_link"/>
-      <origin xyz="-0.221 0.157 ${reflect * 0.09}"/>
-      <axis xyz="0 0 1"/>
-    </joint>
-  </xacro:macro>
-  <!-- Joints -->
   <joint name="base_link_to_chassis_link" type="fixed">
-    <origin xyz="0 0 0.42"/>
+    <origin xyz="0 0 0.439675"/>
     <parent link="base_link"/>
     <child link="chassis_link"/>
   </joint>
+  <xacro:arm_link name="a" m="2" x="0.1" y="0.1" z="0.1"/>
+  <xacro:arm_link name="b" m="2" x="0.58" y="0.04" z="0.04"/>
+  <xacro:arm_link name="c" m="2" x="0.61" y="0.04" z="0.04"/>
+  <xacro:arm_link name="d" m="2" x="0.065" y="0.15" z="0.065"/>
+  <xacro:arm_link name="e" m="2" x="0.172" y="0.155" z="0.145"/>
+  <joint name="chassis_link_to_arm_a_link" type="fixed">
+    <origin xyz="0.164882 0.200235 0.051497"/>
+    <parent link="chassis_link"/>
+    <child link="arm_a_link"/>
+    <axis xyz="0 1 0"/>
+    <limit lower="0" upper="0.5" effort="0" velocity="0"/>
+  </joint>
+  <xacro:arm_revolute_joint parent="arm_a" child="arm_b" x="0.034346" y="0" z="0.049024"/>
+  <xacro:arm_revolute_joint parent="arm_b" child="arm_c" x="0.534365" y="0" z="0.009056"/>
+  <xacro:arm_revolute_joint parent="arm_c" child="arm_d" x="0.546033" y="0" z="0.088594"/>
+  <xacro:arm_revolute_joint parent="arm_d" child="arm_e" x="0.044886" y="0" z="0"/>
+  <xacro:wheels side="left" reflect="1"/>
+  <xacro:wheels side="right" reflect="-1"/>
+  <!-- TODO(quintin): Add IMU -->
   <!-- IMU -->
   <!--  <joint name="imu_joint" type="fixed">-->
@@ -166,5 +214,5 @@
   <!--  </joint>-->
   <!--  <link name="imu_link"/>-->
-  <!-- Camera -->
+  <!-- TODO(quintin): Import the ZED URDF here -->
   <joint name="chassis_link_to_camera_link" type="fixed">
     <origin xyz="0.3 0 0"/>
@@ -179,35 +227,4 @@
     </collision>
   </link>
-  <!--    <visual>-->
-  <!--      <origin xyz="0 0 0" rpy="0 0 0"/>-->
-  <!--      <geometry>-->
-  <!--        <mesh filename="package://mrover/urdf/meshes/zed2i.dae"/>-->
-  <!--      </geometry>-->
-  <!--    </visual>-->
-  <!--    <inertial>-->
-  <!--      <mass value="1e-5"/>-->
-  <!--      <origin xyz="0 0 0" rpy="0 0 0"/>-->
-  <!--      <inertia ixx="1e-6" ixy="0" ixz="0" iyy="1e-6" iyz="0" izz="1e-6"/>-->
-  <!--    </inertial>-->
-  <!--  </link>-->
-  <!-- Left Camera -->
-  <!--  <joint name="left_camera_joint" type="fixed">-->
-  <!--    <origin xyz="0 -0.05 0.1"/>-->
-  <!--    <parent link="chassis_link"/>-->
-  <!--    <child link="left_camera_link"/>-->
-  <!--  </joint>-->
-  <!--  <link name="left_camera_link">-->
-  <!--    <collision>-->
-  <!--      <geometry>-->
-  <!--        <box size="0.06 0.01 0.06"/>-->
-  <!--      </geometry>-->
-  <!--    </collision>-->
-  <!--    <inertial>-->
-  <!--      <mass value="1e-5"/>-->
-  <!--      <inertia ixx="1e-6" ixy="0" ixz="0" iyy="1e-6" iyz="0" izz="1e-6"/>-->
-  <!--    </inertial>-->
-  <!--  </link>-->
   <!--  <xacro:include filename="$(find mrover)/urdf/rover/rover_gazebo_plugins.urdf.xacro"/>-->
-  <xacro:wheels side="left" reflect="1"/>
-  <xacro:wheels side="right" reflect="-1"/>
 </robot>

Commit message: Arm begin whacky

File: urdf/rover/rover.urdf.xacro (robot description, xacro)
@@ -37,5 +37,13 @@
   </xacro:macro>
   <!-- Joints/Links Macros -->
-  <xacro:macro name="arm_link" params="name m x y z">
+  <xacro:macro name="arm_link" params="name m x y z dz:=0">
+<!--    <link name="arm_${name}_axle_link">-->
+<!--      <xacro:cylinder_inertia m="${m}" r="0.05" h="0.075"/>-->
+<!--      <collision>-->
+<!--        <geometry>-->
+<!--          <cylinder length="0.075" radius="0.05"/>-->
+<!--        </geometry>-->
+<!--      </collision>-->
+<!--    </link>-->
     <link name="arm_${name}_link">
       <xacro:box_inertia m="${m}" d="${y}" w="${x}" h="${z}"/>
@@ -46,6 +54,7 @@
       </visual>
       <collision>
-        <geometry>
-          <box size="${x} ${y} ${z}"/>
+        <origin xyz="${x / 2} 0 ${dz}"/>
+        <geometry>
+          <box size="${x * 0.85} ${y} ${z}"/>
         </geometry>
       </collision>
@@ -190,7 +199,7 @@
   <xacro:arm_link name="a" m="2" x="0.1" y="0.1" z="0.1"/>
   <xacro:arm_link name="b" m="2" x="0.58" y="0.04" z="0.04"/>
-  <xacro:arm_link name="c" m="2" x="0.61" y="0.04" z="0.04"/>
+  <xacro:arm_link name="c" m="2" x="0.61" y="0.04" z="0.04" dz="0.1"/>
   <xacro:arm_link name="d" m="2" x="0.065" y="0.15" z="0.065"/>
-  <xacro:arm_link name="e" m="2" x="0.172" y="0.155" z="0.145"/>
+  <xacro:arm_link name="e" m="2" x="0.172" y="0.155" z="0.032"/>
   <joint name="chassis_link_to_arm_a_link" type="fixed">
     <origin xyz="0.164882 0.200235 0.051497"/>

Commit message: Wip

File: urdf/rover/rover.urdf.xacro (robot description, xacro)
@@ -61,5 +61,5 @@
     </link>
   </xacro:macro>
-  <xacro:macro name="arm_revolute_joint" params="parent child x y z">
+  <xacro:macro name="arm_revolute_joint" params="parent child x y z lower upper">
     <joint name="${parent}_link_to_${child}_link" type="revolute">
       <origin xyz="${x} ${y} ${z}"/>
@@ -67,5 +67,5 @@
       <child link="${child}_link"/>
       <axis xyz="0 1 0"/>
-      <limit lower="-0.523599" upper="0.523599" effort="0" velocity="0"/>
+      <limit lower="${lower}" upper="${upper}" effort="0" velocity="0"/>
     </joint>
   </xacro:macro>
@@ -187,6 +187,13 @@
     </visual>
     <collision>
-      <geometry>
-        <box size="${base_len} ${base_width} ${base_height}"/>
+      <origin xyz="-0.085906 0 0"/>
+      <geometry>
+        <box size="0.277 ${base_width} ${base_height}"/>
+      </geometry>
+    </collision>
+    <collision>
+      <origin xyz="0.163609 0 -0.049449"/>
+      <geometry>
+        <box size="0.167 ${base_width} 0.0891 "/>
       </geometry>
     </collision>
@@ -197,9 +204,9 @@
     <child link="chassis_link"/>
   </joint>
-  <xacro:arm_link name="a" m="2" x="0.1" y="0.1" z="0.1"/>
-  <xacro:arm_link name="b" m="2" x="0.58" y="0.04" z="0.04"/>
-  <xacro:arm_link name="c" m="2" x="0.61" y="0.04" z="0.04" dz="0.1"/>
-  <xacro:arm_link name="d" m="2" x="0.065" y="0.15" z="0.065"/>
-  <xacro:arm_link name="e" m="2" x="0.172" y="0.155" z="0.032"/>
+  <xacro:arm_link name="a" m="1" x="0.1" y="0.1" z="0.1"/>
+  <xacro:arm_link name="b" m="1" x="0.58" y="0.04" z="0.04"/>
+  <xacro:arm_link name="c" m="1" x="0.55" y="0.04" z="0.04" dz="0.1"/>
+  <xacro:arm_link name="d" m="1" x="0.065" y="0.15" z="0.065"/>
+  <xacro:arm_link name="e" m="1" x="0.15" y="0.155" z="0.032"/>
   <joint name="chassis_link_to_arm_a_link" type="fixed">
     <origin xyz="0.164882 0.200235 0.051497"/>
@@ -209,8 +216,8 @@
     <limit lower="0" upper="0.5" effort="0" velocity="0"/>
   </joint>
-  <xacro:arm_revolute_joint parent="arm_a" child="arm_b" x="0.034346" y="0" z="0.049024"/>
-  <xacro:arm_revolute_joint parent="arm_b" child="arm_c" x="0.534365" y="0" z="0.009056"/>
-  <xacro:arm_revolute_joint parent="arm_c" child="arm_d" x="0.546033" y="0" z="0.088594"/>
-  <xacro:arm_revolute_joint parent="arm_d" child="arm_e" x="0.044886" y="0" z="0"/>
+  <xacro:arm_revolute_joint parent="arm_a" child="arm_b" x="0.034346" y="0" z="0.049024" lower="${-TAU / 4}" upper="0"/>
+  <xacro:arm_revolute_joint parent="arm_b" child="arm_c" x="0.534365" y="0" z="0.009056" lower="0" upper="${TAU / 4}"/>
+  <xacro:arm_revolute_joint parent="arm_c" child="arm_d" x="0.546033" y="0" z="0.088594" lower="0" upper="0"/>
+  <xacro:arm_revolute_joint parent="arm_d" child="arm_e" x="0.044886" y="0" z="0" lower="0" upper="0"/>
   <xacro:wheels side="left" reflect="1"/>
   <xacro:wheels side="right" reflect="-1"/>

Commit message: Checkppoint

File: urdf/rover/rover.urdf.xacro (robot description, xacro)
@@ -177,6 +177,5 @@
   </xacro:macro>
   <!-- Joints/Links -->
-  <link name="base_link">
-  </link>
+  <link name="base_link" />
   <link name="chassis_link">
     <xacro:box_inertia m="${chassis_mass}" d="${base_len}" w="${base_width}" h="${base_height}"/>

Commit message: Cant tell if things are better or worse...

File: urdf/rover/rover.urdf.xacro (robot description, xacro)
@@ -6,5 +6,5 @@
   <xacro:property name="base_height" value="0.183"/>
   <xacro:property name="wheel_radius" value="0.13"/>
-  <xacro:property name="wheel_width" value="0.1"/>
+  <xacro:property name="wheel_width" value="0.08"/>
   <xacro:property name="wheel_mass" value="0.8"/>
   <xacro:property name="chassis_mass" value="15"/>
@@ -208,5 +208,5 @@
   <xacro:arm_link name="d" m="1" x="0.065" y="0.15" z="0.065"/>
   <xacro:arm_link name="e" m="1" x="0.15" y="0.155" z="0.032"/>
-  <joint name="chassis_link_to_arm_a_link" type="fixed">
+  <joint name="chassis_link_to_arm_a_link" type="prismatic">
     <origin xyz="0.164882 0.200235 0.051497"/>
     <parent link="chassis_link"/>
