Commit message: New simulator into integration (#630)
* Refactor lol

* Add watchdog

* Fix ordering of timer

* Remove fused encoder, should be handled by controller

* some changes to brushless

* testing out websocket with vuex

* Add proper clock arr

* Wrap in extenr C

* I HATE C++

* Dont start in two modes

* Not gross

* Fixed typo

* Added SetDesiredThrottle() in brushless.cpp

* SEND WORKS HAHAHAHAHAHAHHAHAHAHAHHAH ty owen beast gl on 281 and 370 yk yeah

* Change pdlb receiving from RTOS to interrupts

* Watchdog and throttle working

* Encoder working :D

* Implement proper min and max clamping for brushless and resolve motors manager bug

* Resolve TODO

* Add more comments

* More documentation

* Use defines for timers

* added can interrupt

* Removed TODOs from brushless.cpp as they have been done

* changed brushless test bridge to use setDesiredPosition()

* initial dirt sensor commit

* Properly test pdlb code and make it build

* Fix science project to build - comment out broken spectral code

* Add FDCAN peripheral filtering

* Tested and got to work the brushless controller on the Jetson

* Change spectral code in ROS end to include errors

* Comments, make it compile

* Make projects build and make spectral FW properly call init when not init and send out error

* Remove old brushless stuff from esw.yaml

* added nav state msg

* some changes to brushless

* Delete outdated dirt sensor code

* Updated sensor code with ros

* Added updating of mCurrentPosition, mCurretnVelocity, mErrorState and mState in BrushlessController

* Add documentation for SA sensor bridge

* guthrie made me

* Update science code

* adding sempahores for I2C callbacks (wip)

* Change motor library to allow for messages that have some invalid names - prepare for Joint DE node

* Add test joint de script

* Implement better logic for adjustment - still need to implement looping

* Set up reading global revolutions

* Add globals

* Add code to change positions

* Make test joint de script use classes

* Move watchdog to controllers instead of motors manager

* Move everything to have both motor groups and individual motors

* Add joint DE bridge node - barely did anything

* Test on arm bridge with new config

* Add mission specific launch files

* Change multiplier to be an explicit float instead of an int

* Adjust motors group

* Implement joint DE code and fix minor calculation bugs

* Allow arm translator to allow position commands when received all necessary data

* Fix code to check for the correct names array for processing incoming joint data from hw bridge

* Move arm translator bridge into multiple files to be more manageable

* Rename from arm translator to joint DE

* Add offset

* Change code to make pitch and roll output at 8 RPM

* Change keyboard mapping to lowercase

* trust me

* Change

* Create make brake

* Add prints

* Rechange formatting

* Fixed the instructions for how to run the brushless controller demo on the laptop and jetson

* Add absolute encoder timer in bdcmc

* Changed BrushlessController::setDesiredVelocity() to set brake for small velocities

* Set brake when position reached

* Make code

* Recover if in fault state too

* Change comments

* Fix compile errors

* WIP science code.

* WIP Science. Builds now.

* Start changing absolute encoder transaction to I2C DMA

* Rename

* Science code builds pt2.

* changed default min and max velocity for BrushlessController

* fixed joystick mappings

* Remove uneeded things from launch file, format consumers, PDB->PDLB

* Init

* Make nodelet

* Launch file

* Update

* Update

* Update

* Bind buffers

* Update

* Shader infra

* Add shaders

* yo something renders

* Touch

* Update

* Temp

* GLB testing

* Rendering!

* Fix perspective function, bruh WHY is GLM column-major that is so silly!

* YO free look working

* Separate out fly code

* Comments

* Fix fly control ty riley, fix embarassing bug in SO3 LOL

* Refactor

* Update

* Add IMGUI, refactor moteus dep

* Enter and exit gui

* Oops

* Fix framerate

* Update

* Update

* Render coliision

* Add deps

* Fix joints??

* Naming

* Bruh moment

* Status

* Call xacro ourselves on URI

* Things rotating

* SIM3

* Omg working

* Bump

* Can init

* Bleh

* Kinda working lol

* Kinda working

* Tweak mass values

* Switch rocker and bogie

* Try generic version

* Sigh

* Tune mass

* Support meshes

* IN prog commit

* Switch to FBX, textures!

* Import meshses properly

* Make importing models concurrent

* Header refactor

* Update

* ArUco stuff

* Work on render texture

* Holy cow it actually works :D

* Refactor update loop

* Experimenting

* less magic nums

* In prog

* Checkpoint

* A bit of refactoring

* Fix nav exiting behavior

* Pub links to tf tree

* Point cloud gen working on CPU

* In progress update

* In prog commit

* Working, but for some reason tag detector misbehaving

* Fix flip

* Minor updates

* Msg consistencies in nav

* Full auton mission working!

* Comments

* In prog update for saving state

* YO REWIND WORKING!

* Update failure identification to use new state machine messaging (#628)

* print init

* Remove normal maps for now

* Update

* Add imgui settings file

* Add arm

* Arm begin whacky

* Wip

* Checkpoint

* Checkppoint

* Checkpoint

* Cant tell if things are better or worse...

* Kinda working

* Lol trying out webgpu for macs

* Magenta window lol

* imgui working :D

* Update

* Doing something

* OMG mountians rendering with vulkan in linux and metal on macos

* Color :D

* Texture working!

* Input looking good

* wip

* Update

* Constant for depth

* Render multiple modesl

* Holy it actually works

* Spaget code but camera & render texture working

* WIP compute changes

* PC compute working but inefficient and upside down

* PC as fast as possible but dont slow down render

* Auton debug course working, flip uvs, fix pc orientation, fix history

* Rate limit pc correctly

* Add eigen align directives (WTF LOL) to prevent crashing in release mode

* Changes for mac

* Update imgui to v1.90.1

* Update

* Refactor

* remove tf_id from Waypoint.msg

* Build dawn separately, spin sleep

* macos

* Add IK code that neven wrote, fix saved transform of base link, disable resize for now

* Address std::format issue

* minor cmake changes

* Start to IK

* Fix macos compile

* sky blue

* Dawn build script

* Update

* Minor updates

* Remove axle, fix compile

* Try working on wireframe

* Work on render colliders

* Collider rendering somewhat working

* Increase wheel mass

* Add orange hammer, make rover more pretty (thx chloe)

* Pick sky value

* Clean up compute shader

* Work on normal generation

* Oops

* Working?

* Normals actually working I think

* Remove misc stuff from merge

---------

Co-authored-by: Artyom Boyarov <artyom.boyarov@gmail.com>
Co-authored-by: neuenfeldttj <tjneuenfeldt@gmail.com>
Co-authored-by: qhdwight <umroverPerception@gmail.com>
Co-authored-by: Anthony Varkey <anthonyvarkey@gmail.com>
Co-authored-by: owenpark <owenpark@umich.edu>
Co-authored-by: tabiosg <gutstabios@gmail.com>
Co-authored-by: wisabel0 <wisabel@umich.edu>
Co-authored-by: Nate <nbaskins@umich.edu>
Co-authored-by: Polishdudealan <atondryk@umich.edu>
Co-authored-by: Emerson-Ramey <101608185+Emerson-Ramey@users.noreply.github.com>
Co-authored-by: Emerson-Ramey <emramey@umich.edu>

File: urdf/rover/rover.urdf.xacro (robot description, xacro)
@@ -1,22 +1,29 @@
 <?xml version="1.0"?>
 <robot xmlns:xacro="http://www.ros.org/wiki/xacro" name="rover">
-  <xacro:property name="base_width" value="0.7357"/>
-  <xacro:property name="base_len" value="1.0"/>
-  <xacro:property name="base_height" value="0.6"/>
+  <!-- Constants -->
+  <xacro:property name="base_width" value="0.63"/>
+  <xacro:property name="base_len" value="0.478"/>
+  <xacro:property name="base_height" value="0.183"/>
   <xacro:property name="wheel_radius" value="0.13"/>
-  <xacro:property name="wheel_width" value="0.1"/>
-  <xacro:property name="wheel_mass" value="2"/>
-  <xacro:property name="PI" value="3.141592"/>
-  <!-- Inertial macros-->
+  <xacro:property name="wheel_width" value="0.08"/>
+  <xacro:property name="wheel_mass" value="3"/>
+  <xacro:property name="chassis_mass" value="15"/>
+  <xacro:property name="wheel_torque" value="2.68"/>
+  <xacro:property name="TAU" value="6.2831855"/>
+  <!-- Inertial Macros-->
   <xacro:macro name="cylinder_inertia" params="m r h">
     <inertial>
       <mass value="${m}"/>
-      <inertia ixx="${m*(3*r*r+h*h)/12}" ixy="0" ixz="0" iyy="${m*(3*r*r+h*h)/12}" iyz="0" izz="${m*r*r/2}"/>
+      <inertia ixx="${m*(3*r*r+h*h)/12}" ixy="0" ixz="0"
+               iyy="${m*(3*r*r+h*h)/12}" iyz="0"
+               izz="${m*r*r/2}"/>
     </inertial>
   </xacro:macro>
-  <xacro:macro name="box_inertia" params="m w h d">
+  <xacro:macro name="box_inertia" params="m d w h">
     <inertial>
       <mass value="${m}"/>
-      <inertia ixx="${m / 12.0 * (d*d + h*h)}" ixy="0.0" ixz="0.0" iyy="${m / 12.0 * (w*w + h*h)}" iyz="0.0" izz="${m / 12.0 * (w*w + d*d)}"/>
+      <inertia ixx="${m / 12.0 * (w*w + h*h)}" ixy="0" ixz="0"
+               iyy="${m / 12.0 * (d*d + h*h)}" iyz="0"
+               izz="${m / 12.0 * (d*d + w*w)}"/>
     </inertial>
   </xacro:macro>
@@ -24,144 +31,204 @@
     <inertial>
       <mass value="${m}"/>
-      <inertia ixx="${2.0*m*(r*r)/5.0}" ixy="0.0" ixz="0.0" iyy="${2.0*m*(r*r)/5.0}" iyz="0.0" izz="${2.0*m*(r*r)/5.0}"/>
+      <inertia ixx="${2.0*m*(r*r)/5.0}" ixy="0" ixz="0"
+               iyy="${2.0*m*(r*r)/5.0}" iyz="0"
+               izz="${2.0*m*(r*r)/5.0}"/>
     </inertial>
   </xacro:macro>
-  <!-- Links -->
+  <!-- Joints/Links Macros -->
+  <xacro:macro name="arm_link" params="name m x y z dz:=0">
+    <link name="arm_${name}_link">
+      <xacro:box_inertia m="${m}" d="${y}" w="${x}" h="${z}"/>
+      <visual>
+        <geometry>
+          <mesh filename="package://mrover/urdf/meshes/arm_${name}.fbx"/>
+        </geometry>
+      </visual>
+      <collision>
+        <origin xyz="${x / 2} 0 ${dz}"/>
+        <geometry>
+          <box size="${x * 0.85} ${y} ${z}"/>
+        </geometry>
+      </collision>
+    </link>
+  </xacro:macro>
+  <xacro:macro name="arm_revolute_joint" params="parent child x y z lower upper">
+    <joint name="${parent}_link_to_${child}_link" type="revolute">
+      <origin xyz="${x} ${y} ${z}"/>
+      <parent link="${parent}_link"/>
+      <child link="${child}_link"/>
+      <axis xyz="0 1 0"/>
+      <limit lower="${lower}" upper="${upper}" effort="0" velocity="0"/>
+    </joint>
+  </xacro:macro>
+  <xacro:macro name="wheel" params="pos side reflect">
+    <link name="${pos}_${side}_wheel_link">
+      <xacro:cylinder_inertia m="${wheel_mass}" r="${wheel_radius}" h="${wheel_width}"/>
+      <visual>
+        <geometry>
+          <mesh filename="package://mrover/urdf/meshes/rover_${side}_wheel.fbx"/>
+        </geometry>
+      </visual>
+      <collision>
+        <geometry>
+          <cylinder length="${wheel_width}" radius="${wheel_radius}"/>
+        </geometry>
+      </collision>
+    </link>
+  </xacro:macro>
+  <xacro:macro name="wheels" params="side reflect">
+    <xacro:wheel pos="front" side="${side}" reflect="${reflect}"/>
+    <xacro:wheel pos="center" side="${side}" reflect="${reflect}"/>
+    <xacro:wheel pos="back" side="${side}" reflect="${reflect}"/>
+    <link name="${side}_bogie_link">
+      <xacro:box_inertia m="3" d="0.5" w="0.5" h="0.5"/>
+      <visual>
+        <geometry>
+          <mesh filename="package://mrover/urdf/meshes/rover_${side}_bogie.fbx"/>
+        </geometry>
+      </visual>
+      <collision>
+        <origin xyz="-0.14 0.1 0" rpy="0 0 -0.734"/>
+        <geometry>
+          <box size="0.2 0.025 0.025"/>
+        </geometry>
+      </collision>
+      <collision>
+        <origin xyz="0.1 0.088 0" rpy="0 0 0.734"/>
+        <geometry>
+          <box size="0.2 0.025 0.025"/>
+        </geometry>
+      </collision>
+    </link>
+    <link name="${side}_rocker_link">
+      <xacro:box_inertia m="3" d="0.5" w="0.5" h="0.5"/>
+      <visual>
+        <geometry>
+          <mesh filename="package://mrover/urdf/meshes/rover_${side}_rocker.fbx"/>
+        </geometry>
+      </visual>
+      <collision>
+        <origin xyz="0.11 0.077 0" rpy="0 0 0.585"/>
+        <geometry>
+          <box size="0.2 0.025 0.025"/>
+        </geometry>
+      </collision>
+      <collision>
+        <origin xyz="-0.22 0.15 0" rpy="0 0 -0.585"/>
+        <geometry>
+          <box size="0.5 0.025 0.025"/>
+        </geometry>
+      </collision>
+    </link>
+    <joint name="chassis_link_to_${side}_rocker_link" type="revolute">
+      <parent link="chassis_link"/>
+      <child link="${side}_rocker_link"/>
+      <origin xyz="0.164665 ${reflect * (base_width/2 + 0.05)} 0" rpy="${-TAU/4} 0 0"/>
+      <axis xyz="0 0 1"/>
+      <limit lower="-0.122173" upper="0.523599" effort="0" velocity="0"/>
+    </joint>
+    <joint name="${side}_rocker_link_to_back_${side}_wheel_link" type="continuous">
+      <parent link="${side}_rocker_link"/>
+      <child link="back_${side}_wheel_link"/>
+      <origin xyz="-0.417094 0.28513 ${reflect * 0.09}"/>
+      <axis xyz="0 0 1"/>
+      <limit effort="${wheel_torque}" velocity="0"/>
+    </joint>
+    <joint name="${side}_rocker_link_to_${side}_bogie_link" type="revolute">
+      <parent link="${side}_rocker_link"/>
+      <child link="${side}_bogie_link"/>
+      <origin xyz="0.198948 0.138674 0"/>
+      <axis xyz="0 0 1"/>
+      <limit lower="-0.349066" upper="0.349066" effort="0" velocity="0"/>
+    </joint>
+    <joint name="${side}_bogie_link_to_front_${side}_wheel_link" type="continuous">
+      <parent link="${side}_bogie_link"/>
+      <child link="front_${side}_wheel_link"/>
+      <origin xyz="0.215233 0.147933 ${reflect * 0.09}"/>
+      <axis xyz="0 0 1"/>
+      <limit effort="${wheel_torque}" velocity="0"/>
+    </joint>
+    <joint name="${side}_bogie_link_to_center_${side}_wheel_link" type="continuous">
+      <parent link="${side}_bogie_link"/>
+      <child link="center_${side}_wheel_link"/>
+      <origin xyz="-0.173532 0.147659 ${reflect * 0.09}"/>
+      <axis xyz="0 0 1"/>
+      <limit effort="${wheel_torque}" velocity="0"/>
+    </joint>
+  </xacro:macro>
+  <!-- Joints/Links -->
   <link name="base_link"/>
   <link name="chassis_link">
-    <xacro:box_inertia m="3.0" w="${base_len}" h="${base_width}" d="${base_height}"/>
+    <xacro:box_inertia m="${chassis_mass}" d="${base_len}" w="${base_width}" h="${base_height}"/>
     <visual>
-      <origin rpy="0 0 0" xyz="0 0 0"/>
-      <geometry>
-        <mesh filename="package://mrover/urdf/meshes/rover.dae"/>
+      <geometry>
+        <mesh filename="package://mrover/urdf/meshes/rover_chassis.fbx"/>
       </geometry>
     </visual>
     <collision>
-      <geometry>
-        <box size="${base_len} ${base_width} ${base_height}"/>
+      <origin xyz="-0.085906 0 0"/>
+      <geometry>
+        <box size="0.277 ${base_width} ${base_height}"/>
+      </geometry>
+    </collision>
+    <collision>
+      <origin xyz="0.163609 0 -0.049449"/>
+      <geometry>
+        <box size="0.167 ${base_width} 0.0891 "/>
       </geometry>
     </collision>
   </link>
-  <xacro:macro name="wheel" params="side reflect">
-    <link name="front_${side}_wheel_link">
-      <xacro:sphere_inertia m="${wheel_mass}" r="${wheel_radius}"/>
-      <visual>
-        <origin rpy="0 ${min(0, reflect) * PI} 0" xyz="0 0 0"/>
-        <geometry>
-          <mesh filename="package://mrover/urdf/meshes/rover.wheel.dae"/>
-        </geometry>
-      </visual>
-      <collision>
-        <geometry>
-          <sphere radius="${wheel_radius}"/>
-        </geometry>
-      </collision>
-    </link>
-    <link name="center_${side}_wheel_link">
-      <xacro:cylinder_inertia m="${wheel_mass}" r="${wheel_radius}" h="${wheel_width}"/>
-      <visual>
-        <origin rpy="0 ${min(0, reflect) * PI} 0" xyz="0 0 0"/>
-        <geometry>
-          <mesh filename="package://mrover/urdf/meshes/rover.wheel.dae"/>
-        </geometry>
-      </visual>
-      <collision>
-        <geometry>
-          <cylinder length="${wheel_width}" radius="${wheel_radius}"/>
-        </geometry>
-      </collision>
-    </link>
-    <link name="back_${side}_wheel_link">
-      <xacro:sphere_inertia m="${wheel_mass}" r="${wheel_radius}"/>
-      <visual>
-        <origin rpy="0 ${min(0, reflect) * PI} 0" xyz="0 0 0"/>
-        <geometry>
-          <mesh filename="package://mrover/urdf/meshes/rover.wheel.dae"/>
-        </geometry>
-      </visual>
-      <collision>
-        <geometry>
-          <sphere radius="${wheel_radius}"/>
-        </geometry>
-      </collision>
-    </link>
-    <joint name="front_${side}_wheel_joint" type="continuous">
-      <parent link="chassis_link"/>
-      <child link="front_${side}_wheel_link"/>
-      <origin xyz="0.42 ${reflect * (base_width/2 + 0.06)} -0.373" rpy="${-PI/2} 0 0"/>
-      <axis xyz="0 0 1"/>
-    </joint>
-    <joint name="center_${side}_wheel_joint" type="continuous">
-      <parent link="chassis_link"/>
-      <child link="center_${side}_wheel_link"/>
-      <origin xyz="0 ${reflect * (base_width/2 + 0.06)} -0.373" rpy="${-PI/2} 0 0"/>
-      <axis xyz="0 0 1"/>
-    </joint>
-    <joint name="back_${side}_wheel_joint" type="continuous">
-      <parent link="chassis_link"/>
-      <child link="back_${side}_wheel_link"/>
-      <origin xyz="-0.42 ${reflect * (base_width/2 + 0.06)} -0.373" rpy="${-PI/2} 0 0"/>
-      <axis xyz="0 0 1"/>
-    </joint>
-  </xacro:macro>
-  <!-- Joints -->
-  <joint name="base_link_to_chassis" type="fixed">
-    <origin xyz="0 0 0.5"/>
+  <joint name="base_link_to_chassis_link" type="fixed">
+    <origin xyz="0 0 0.439675"/>
     <parent link="base_link"/>
     <child link="chassis_link"/>
   </joint>
+  <xacro:arm_link name="a" m="1" x="0.1" y="0.1" z="0.1"/>
+  <xacro:arm_link name="b" m="1" x="0.58" y="0.04" z="0.04"/>
+  <xacro:arm_link name="c" m="1" x="0.55" y="0.04" z="0.04" dz="0.1"/>
+  <xacro:arm_link name="d" m="1" x="0.065" y="0.15" z="0.065"/>
+  <xacro:arm_link name="e" m="1" x="0.15" y="0.155" z="0.032"/>
+  <joint name="chassis_link_to_arm_a_link" type="prismatic">
+    <origin xyz="0.164882 0.200235 0.051497"/>
+    <parent link="chassis_link"/>
+    <child link="arm_a_link"/>
+    <axis xyz="0 1 0"/>
+    <limit lower="0" upper="0.5" effort="0" velocity="0"/>
+  </joint>
+  <xacro:arm_revolute_joint parent="arm_a" child="arm_b"
+                            x="0.034346" y="0" z="0.049024"
+                            lower="${-TAU / 8}" upper="0"/>
+  <xacro:arm_revolute_joint parent="arm_b" child="arm_c"
+                            x="0.534365" y="0" z="0.009056"
+                            lower="0" upper="${TAU / 2}"/>
+  <xacro:arm_revolute_joint parent="arm_c" child="arm_d"
+                            x="0.546033" y="0" z="0.088594"
+                            lower="0" upper="0"/>
+  <xacro:arm_revolute_joint parent="arm_d" child="arm_e"
+                            x="0.044886" y="0" z="0"
+                            lower="0" upper="0"/>
+  <xacro:wheels side="left" reflect="1"/>
+  <xacro:wheels side="right" reflect="-1"/>
+  <!-- TODO(quintin): Add IMU -->
   <!-- IMU -->
-  <joint name="imu_joint" type="fixed">
-    <origin xyz="0 0 0.2"/>
+  <!--  <joint name="imu_joint" type="fixed">-->
+  <!--    <origin xyz="0 0 0.2"/>-->
+  <!--    <parent link="chassis_link"/>-->
+  <!--    <child link="imu_link"/>-->
+  <!--  </joint>-->
+  <!--  <link name="imu_link"/>-->
+  <!-- TODO(quintin): Import the ZED URDF here -->
+  <joint name="chassis_link_to_camera_link" type="fixed">
+    <origin xyz="0.3 0 0"/>
     <parent link="chassis_link"/>
-    <child link="imu_link"/>
+    <child link="zed2i_left_camera_frame"/>
   </joint>
-  <link name="imu_link"/>
-  <!-- Camera -->
-  <joint name="camera_joint" type="fixed">
-    <origin xyz="0 0 0.1"/>
-    <parent link="chassis_link"/>
-    <child link="camera_link"/>
-  </joint>
-  <link name="camera_link">
+  <link name="zed2i_left_camera_frame">
     <collision>
-      <origin xyz="0 0 0" rpy="0 0 0"/>
       <geometry>
         <box size="0.01 0.1 0.01"/>
       </geometry>
     </collision>
-    <visual>
-      <origin xyz="0 0 0" rpy="0 0 0"/>
-      <geometry>
-        <mesh filename="package://mrover/urdf/meshes/zed2i.dae"/>
-      </geometry>
-    </visual>
-    <inertial>
-      <mass value="1e-5"/>
-      <origin xyz="0 0 0" rpy="0 0 0"/>
-      <inertia ixx="1e-6" ixy="0" ixz="0" iyy="1e-6" iyz="0" izz="1e-6"/>
-    </inertial>
   </link>
-  <!-- Left Camera -->
-  <joint name="left_camera_joint" type="fixed">
-    <origin xyz="0 -0.05 0.1"/>
-    <parent link="chassis_link"/>
-    <child link="left_camera_link"/>
-  </joint>
-  <link name="left_camera_link">
-    <collision>
-      <origin xyz="0 0 0" rpy="0 0 0"/>
-      <geometry>
-        <box size="0.06 0.01 0.06"/>
-      </geometry>
-    </collision>
-    <inertial>
-      <mass value="1e-5"/>
-      <origin xyz="0 0 0" rpy="0 0 0"/>
-      <inertia ixx="1e-6" ixy="0" ixz="0" iyy="1e-6" iyz="0" izz="1e-6"/>
-    </inertial>
-  </link>
-  <xacro:include filename="$(find mrover)/urdf/rover/rover_gazebo_plugins.urdf.xacro"/>
-  <xacro:wheel side="left" reflect="1"/>
-  <xacro:wheel side="right" reflect="-1"/>
+  <!--  <xacro:include filename="$(find mrover)/urdf/rover/rover_gazebo_plugins.urdf.xacro"/>-->
 </robot>
