Commit message: fixed reference points and removed z component for better rviz experience

File: urdf/rover/rover.urdf.xacro (robot description, xacro)
@@ -124,5 +124,5 @@
   <link name="rover_gps_left_link" />
   <joint name="rover_gps_left" type="fixed">
-    <origin xyz="0 0 0" />
+    <origin xyz="0 1 0" />
     <parent link="chassis_link" />
     <child link="rover_gps_left_link" />
@@ -130,5 +130,5 @@
   <link name="rover_gps_right_link" />
   <joint name="rover_gps_right" type="fixed">
-    <origin xyz="0 1 0" />
+    <origin xyz="0 -1 0" />
     <parent link="chassis_link" />
     <child link="rover_gps_right_link" />

File: urdf/rover/rover_gazebo_plugins.urdf.xacro (robot description, xacro)
@@ -25,6 +25,6 @@
       <topicName>left_gps_driver/fix</topicName>
       <velocityTopicName>gps/fix_velocity</velocityTopicName>
-      <referenceLatitude>42.2931950000000000000000</referenceLatitude>
-      <referenceLongitude>-83.80967060000000000000000</referenceLongitude>
+      <referenceLatitude>42.293195</referenceLatitude>
+      <referenceLongitude>-83.7096706</referenceLongitude>
       <referenceHeading>90.0</referenceHeading>
       <referenceAltitude>0.0</referenceAltitude>
@@ -42,6 +42,6 @@
       <topicName>right_gps_driver/fix</topicName>
       <velocityTopicName>gps/fix_velocity</velocityTopicName>
-      <referenceLatitude>42.2931950000000000000000</referenceLatitude>
-      <referenceLongitude>-83.80967060000000000000000</referenceLongitude>
+      <referenceLatitude>42.293195</referenceLatitude>
+      <referenceLongitude>-83.7096706</referenceLongitude>
       <referenceHeading>90.0</referenceHeading>
       <referenceAltitude>0.0</referenceAltitude>

Commit message: fixed pose publishing offset temporarily

File: urdf/rover/rover.urdf.xacro (robot description, xacro)
@@ -122,15 +122,15 @@
   <link name="imu_link" />
   <!-- GPS -->
-  <link name="rover_gps_left_link" />
-  <joint name="rover_gps_left" type="fixed">
+  <link name="left_gps_link" />
+  <joint name="left_gps" type="fixed">
     <origin xyz="0 1 0" />
     <parent link="chassis_link" />
-    <child link="rover_gps_left_link" />
+    <child link="left_gps_link" />
   </joint>
-  <link name="rover_gps_right_link" />
-  <joint name="rover_gps_right" type="fixed">
+  <link name="right_gps_link" />
+  <joint name="right_gps" type="fixed">
     <origin xyz="0 -1 0" />
     <parent link="chassis_link" />
-    <child link="rover_gps_right_link" />
+    <child link="right_gps_link" />
   </joint>
   <!-- Camera -->

Commit message: Add starter work for gps

File: urdf/rover/rover.urdf.xacro (robot description, xacro)
@@ -210,12 +210,16 @@
   <xacro:wheels side="left" reflect="1"/>
   <xacro:wheels side="right" reflect="-1"/>
-  <!-- TODO(quintin): Add IMU -->
-  <!-- IMU -->
-  <!--  <joint name="imu_joint" type="fixed">-->
-  <!--    <origin xyz="0 0 0.2"/>-->
-  <!--    <parent link="chassis_link"/>-->
-  <!--    <child link="imu_link"/>-->
-  <!--  </joint>-->
-  <!--  <link name="imu_link"/>-->
+  <joint name="chassis_link_to_left_gps" type="fixed">
+    <origin xyz="0 0.1 0"/>
+    <parent link="chassis_link"/>
+    <child link="left_gps"/>
+  </joint>
+  <link name="left_gps"/>
+  <joint name="chassis_link_to_right_gps" type="fixed">
+    <origin xyz="0 -0.1 0"/>
+    <parent link="chassis_link"/>
+    <child link="right_gps"/>
+  </joint>
+  <link name="right_gps"/>
   <!-- TODO(quintin): Import the ZED URDF here -->
   <joint name="chassis_link_to_camera_link" type="fixed">

Commit message: Yo workingin the new sim

File: urdf/rover/rover.urdf.xacro (robot description, xacro)
@@ -2,36 +2,36 @@
 <robot xmlns:xacro="http://www.ros.org/wiki/xacro" name="rover">
   <!-- Constants -->
-  <xacro:property name="base_width" value="0.63" />
-  <xacro:property name="base_len" value="0.478" />
-  <xacro:property name="base_height" value="0.183" />
-  <xacro:property name="wheel_radius" value="0.13" />
-  <xacro:property name="wheel_width" value="0.08" />
-  <xacro:property name="wheel_mass" value="3" />
-  <xacro:property name="chassis_mass" value="15" />
-  <xacro:property name="wheel_torque" value="2.68" />
-  <xacro:property name="TAU" value="6.2831855" />
+  <xacro:property name="base_width" value="0.63"/>
+  <xacro:property name="base_len" value="0.478"/>
+  <xacro:property name="base_height" value="0.183"/>
+  <xacro:property name="wheel_radius" value="0.13"/>
+  <xacro:property name="wheel_width" value="0.08"/>
+  <xacro:property name="wheel_mass" value="3"/>
+  <xacro:property name="chassis_mass" value="15"/>
+  <xacro:property name="wheel_torque" value="2.68"/>
+  <xacro:property name="TAU" value="6.2831855"/>
   <!-- Inertial Macros-->
   <xacro:macro name="cylinder_inertia" params="m r h">
     <inertial>
-      <mass value="${m}" />
+      <mass value="${m}"/>
       <inertia ixx="${m*(3*r*r+h*h)/12}" ixy="0" ixz="0"
-        iyy="${m*(3*r*r+h*h)/12}" iyz="0"
-        izz="${m*r*r/2}" />
+               iyy="${m*(3*r*r+h*h)/12}" iyz="0"
+               izz="${m*r*r/2}"/>
     </inertial>
   </xacro:macro>
   <xacro:macro name="box_inertia" params="m d w h">
     <inertial>
-      <mass value="${m}" />
+      <mass value="${m}"/>
       <inertia ixx="${m / 12.0 * (w*w + h*h)}" ixy="0" ixz="0"
-        iyy="${m / 12.0 * (d*d + h*h)}" iyz="0"
-        izz="${m / 12.0 * (d*d + w*w)}" />
+               iyy="${m / 12.0 * (d*d + h*h)}" iyz="0"
+               izz="${m / 12.0 * (d*d + w*w)}"/>
     </inertial>
   </xacro:macro>
   <xacro:macro name="sphere_inertia" params="m r">
     <inertial>
-      <mass value="${m}" />
+      <mass value="${m}"/>
       <inertia ixx="${2.0*m*(r*r)/5.0}" ixy="0" ixz="0"
-        iyy="${2.0*m*(r*r)/5.0}" iyz="0"
-        izz="${2.0*m*(r*r)/5.0}" />
+               iyy="${2.0*m*(r*r)/5.0}" iyz="0"
+               izz="${2.0*m*(r*r)/5.0}"/>
     </inertial>
   </xacro:macro>
@@ -39,14 +39,14 @@
   <xacro:macro name="arm_link" params="name m x y z dz:=0">
     <link name="arm_${name}_link">
-      <xacro:box_inertia m="${m}" d="${y}" w="${x}" h="${z}" />
-      <visual>
-        <geometry>
-          <mesh filename="package://mrover/urdf/meshes/arm_${name}.fbx" />
-        </geometry>
-      </visual>
-      <collision>
-        <origin xyz="${x / 2} 0 ${dz}" />
-        <geometry>
-          <box size="${x * 0.85} ${y} ${z}" />
+      <xacro:box_inertia m="${m}" d="${y}" w="${x}" h="${z}"/>
+      <visual>
+        <geometry>
+          <mesh filename="package://mrover/urdf/meshes/arm_${name}.fbx"/>
+        </geometry>
+      </visual>
+      <collision>
+        <origin xyz="${x / 2} 0 ${dz}"/>
+        <geometry>
+          <box size="${x * 0.85} ${y} ${z}"/>
         </geometry>
       </collision>
@@ -55,22 +55,22 @@
   <xacro:macro name="arm_revolute_joint" params="parent child x y z lower upper">
     <joint name="${parent}_link_to_${child}_link" type="revolute">
-      <origin xyz="${x} ${y} ${z}" />
-      <parent link="${parent}_link" />
-      <child link="${child}_link" />
-      <axis xyz="0 1 0" />
-      <limit lower="${lower}" upper="${upper}" effort="0" velocity="0" />
+      <origin xyz="${x} ${y} ${z}"/>
+      <parent link="${parent}_link"/>
+      <child link="${child}_link"/>
+      <axis xyz="0 1 0"/>
+      <limit lower="${lower}" upper="${upper}" effort="0" velocity="0"/>
     </joint>
   </xacro:macro>
   <xacro:macro name="wheel" params="pos side reflect">
     <link name="${pos}_${side}_wheel_link">
-      <xacro:cylinder_inertia m="${wheel_mass}" r="${wheel_radius}" h="${wheel_width}" />
-      <visual>
-        <geometry>
-          <mesh filename="package://mrover/urdf/meshes/rover_${side}_wheel.fbx" />
-        </geometry>
-      </visual>
-      <collision>
-        <geometry>
-          <cylinder length="${wheel_width}" radius="${wheel_radius}" />
+      <xacro:cylinder_inertia m="${wheel_mass}" r="${wheel_radius}" h="${wheel_width}"/>
+      <visual>
+        <geometry>
+          <mesh filename="package://mrover/urdf/meshes/rover_${side}_wheel.fbx"/>
+        </geometry>
+      </visual>
+      <collision>
+        <geometry>
+          <cylinder length="${wheel_width}" radius="${wheel_radius}"/>
         </geometry>
       </collision>
@@ -78,154 +78,164 @@
   </xacro:macro>
   <xacro:macro name="wheels" params="side reflect">
-    <xacro:wheel pos="front" side="${side}" reflect="${reflect}" />
-    <xacro:wheel pos="center" side="${side}" reflect="${reflect}" />
-    <xacro:wheel pos="back" side="${side}" reflect="${reflect}" />
+    <xacro:wheel pos="front" side="${side}" reflect="${reflect}"/>
+    <xacro:wheel pos="center" side="${side}" reflect="${reflect}"/>
+    <xacro:wheel pos="back" side="${side}" reflect="${reflect}"/>
     <link name="${side}_bogie_link">
-      <xacro:box_inertia m="3" d="0.5" w="0.5" h="0.5" />
-      <visual>
-        <geometry>
-          <mesh filename="package://mrover/urdf/meshes/rover_${side}_bogie.fbx" />
-        </geometry>
-      </visual>
-      <collision>
-        <origin xyz="-0.14 0.1 0" rpy="0 0 -0.734" />
-        <geometry>
-          <box size="0.2 0.025 0.025" />
-        </geometry>
-      </collision>
-      <collision>
-        <origin xyz="0.1 0.088 0" rpy="0 0 0.734" />
-        <geometry>
-          <box size="0.2 0.025 0.025" />
+      <xacro:box_inertia m="3" d="0.5" w="0.5" h="0.5"/>
+      <visual>
+        <geometry>
+          <mesh filename="package://mrover/urdf/meshes/rover_${side}_bogie.fbx"/>
+        </geometry>
+      </visual>
+      <collision>
+        <origin xyz="-0.14 0.1 0" rpy="0 0 -0.734"/>
+        <geometry>
+          <box size="0.2 0.025 0.025"/>
+        </geometry>
+      </collision>
+      <collision>
+        <origin xyz="0.1 0.088 0" rpy="0 0 0.734"/>
+        <geometry>
+          <box size="0.2 0.025 0.025"/>
         </geometry>
       </collision>
     </link>
     <link name="${side}_rocker_link">
-      <xacro:box_inertia m="3" d="0.5" w="0.5" h="0.5" />
-      <visual>
-        <geometry>
-          <mesh filename="package://mrover/urdf/meshes/rover_${side}_rocker.fbx" />
-        </geometry>
-      </visual>
-      <collision>
-        <origin xyz="0.11 0.077 0" rpy="0 0 0.585" />
-        <geometry>
-          <box size="0.2 0.025 0.025" />
-        </geometry>
-      </collision>
-      <collision>
-        <origin xyz="-0.22 0.15 0" rpy="0 0 -0.585" />
-        <geometry>
-          <box size="0.5 0.025 0.025" />
+      <xacro:box_inertia m="3" d="0.5" w="0.5" h="0.5"/>
+      <visual>
+        <geometry>
+          <mesh filename="package://mrover/urdf/meshes/rover_${side}_rocker.fbx"/>
+        </geometry>
+      </visual>
+      <collision>
+        <origin xyz="0.11 0.077 0" rpy="0 0 0.585"/>
+        <geometry>
+          <box size="0.2 0.025 0.025"/>
+        </geometry>
+      </collision>
+      <collision>
+        <origin xyz="-0.22 0.15 0" rpy="0 0 -0.585"/>
+        <geometry>
+          <box size="0.5 0.025 0.025"/>
         </geometry>
       </collision>
     </link>
     <joint name="chassis_link_to_${side}_rocker_link" type="revolute">
-      <parent link="chassis_link" />
-      <child link="${side}_rocker_link" />
-      <origin xyz="0.164665 ${reflect * (base_width/2 + 0.05)} 0" rpy="${-TAU/4} 0 0" />
-      <axis xyz="0 0 1" />
-      <limit lower="-0.122173" upper="0.523599" effort="0" velocity="0" />
+      <parent link="chassis_link"/>
+      <child link="${side}_rocker_link"/>
+      <origin xyz="0.164665 ${reflect * (base_width/2 + 0.05)} 0" rpy="${-TAU/4} 0 0"/>
+      <axis xyz="0 0 1"/>
+      <limit lower="-0.122173" upper="0.523599" effort="0" velocity="0"/>
     </joint>
     <joint name="${side}_rocker_link_to_back_${side}_wheel_link" type="continuous">
-      <parent link="${side}_rocker_link" />
-      <child link="back_${side}_wheel_link" />
-      <origin xyz="-0.417094 0.28513 ${reflect * 0.09}" />
-      <axis xyz="0 0 1" />
-      <limit effort="${wheel_torque}" velocity="0" />
+      <parent link="${side}_rocker_link"/>
+      <child link="back_${side}_wheel_link"/>
+      <origin xyz="-0.417094 0.28513 ${reflect * 0.09}"/>
+      <axis xyz="0 0 1"/>
+      <limit effort="${wheel_torque}" velocity="0"/>
     </joint>
     <joint name="${side}_rocker_link_to_${side}_bogie_link" type="revolute">
-      <parent link="${side}_rocker_link" />
-      <child link="${side}_bogie_link" />
-      <origin xyz="0.198948 0.138674 0" />
-      <axis xyz="0 0 1" />
-      <limit lower="-0.349066" upper="0.349066" effort="0" velocity="0" />
+      <parent link="${side}_rocker_link"/>
+      <child link="${side}_bogie_link"/>
+      <origin xyz="0.198948 0.138674 0"/>
+      <axis xyz="0 0 1"/>
+      <limit lower="-0.349066" upper="0.349066" effort="0" velocity="0"/>
     </joint>
     <joint name="${side}_bogie_link_to_front_${side}_wheel_link" type="continuous">
-      <parent link="${side}_bogie_link" />
-      <child link="front_${side}_wheel_link" />
-      <origin xyz="0.215233 0.147933 ${reflect * 0.09}" />
-      <axis xyz="0 0 1" />
-      <limit effort="${wheel_torque}" velocity="0" />
+      <parent link="${side}_bogie_link"/>
+      <child link="front_${side}_wheel_link"/>
+      <origin xyz="0.215233 0.147933 ${reflect * 0.09}"/>
+      <axis xyz="0 0 1"/>
+      <limit effort="${wheel_torque}" velocity="0"/>
     </joint>
     <joint name="${side}_bogie_link_to_center_${side}_wheel_link" type="continuous">
-      <parent link="${side}_bogie_link" />
-      <child link="center_${side}_wheel_link" />
-      <origin xyz="-0.173532 0.147659 ${reflect * 0.09}" />
-      <axis xyz="0 0 1" />
-      <limit effort="${wheel_torque}" velocity="0" />
+      <parent link="${side}_bogie_link"/>
+      <child link="center_${side}_wheel_link"/>
+      <origin xyz="-0.173532 0.147659 ${reflect * 0.09}"/>
+      <axis xyz="0 0 1"/>
+      <limit effort="${wheel_torque}" velocity="0"/>
     </joint>
   </xacro:macro>
   <!-- Joints/Links -->
-  <link name="base_link" />
+  <link name="base_link"/>
   <link name="chassis_link">
-    <xacro:box_inertia m="${chassis_mass}" d="${base_len}" w="${base_width}" h="${base_height}" />
+    <xacro:box_inertia m="${chassis_mass}" d="${base_len}" w="${base_width}" h="${base_height}"/>
     <visual>
       <geometry>
-        <mesh filename="package://mrover/urdf/meshes/rover_chassis.fbx" />
+        <mesh filename="package://mrover/urdf/meshes/rover_chassis.fbx"/>
       </geometry>
     </visual>
     <collision>
-      <origin xyz="-0.085906 0 0" />
-      <geometry>
-        <box size="0.277 ${base_width} ${base_height}" />
+      <origin xyz="-0.085906 0 0"/>
+      <geometry>
+        <box size="0.277 ${base_width} ${base_height}"/>
       </geometry>
     </collision>
     <collision>
-      <origin xyz="0.163609 0 -0.049449" />
-      <geometry>
-        <box size="0.167 ${base_width} 0.0891 " />
+      <origin xyz="0.163609 0 -0.049449"/>
+      <geometry>
+        <box size="0.167 ${base_width} 0.0891 "/>
       </geometry>
     </collision>
   </link>
   <joint name="base_link_to_chassis_link" type="fixed">
-    <origin xyz="0 0 0.439675" />
-    <parent link="base_link" />
-    <child link="chassis_link" />
-  </joint>
-  <xacro:arm_link name="a" m="1" x="0.1" y="0.1" z="0.1" />
-  <xacro:arm_link name="b" m="1" x="0.58" y="0.04" z="0.04" />
-  <xacro:arm_link name="c" m="1" x="0.55" y="0.04" z="0.04" dz="0.1" />
-  <xacro:arm_link name="d" m="1" x="0.065" y="0.15" z="0.065" />
-  <xacro:arm_link name="e" m="1" x="0.15" y="0.155" z="0.032" />
+    <origin xyz="0 0 0.439675"/>
+    <parent link="base_link"/>
+    <child link="chassis_link"/>
+  </joint>
+  <xacro:arm_link name="a" m="1" x="0.1" y="0.1" z="0.1"/>
+  <xacro:arm_link name="b" m="1" x="0.58" y="0.04" z="0.04"/>
+  <xacro:arm_link name="c" m="1" x="0.55" y="0.04" z="0.04" dz="0.1"/>
+  <xacro:arm_link name="d" m="1" x="0.065" y="0.15" z="0.065"/>
+  <xacro:arm_link name="e" m="1" x="0.15" y="0.155" z="0.032"/>
   <joint name="chassis_link_to_arm_a_link" type="prismatic">
-    <origin xyz="0.164882 0.200235 0.051497" />
-    <parent link="chassis_link" />
-    <child link="arm_a_link" />
-    <axis xyz="0 1 0" />
-    <limit lower="0" upper="0.5" effort="0" velocity="0" />
+    <origin xyz="0.164882 0.200235 0.051497"/>
+    <parent link="chassis_link"/>
+    <child link="arm_a_link"/>
+    <axis xyz="0 1 0"/>
+    <limit lower="0" upper="0.5" effort="0" velocity="0"/>
   </joint>
   <xacro:arm_revolute_joint parent="arm_a" child="arm_b"
-    x="0.034346" y="0" z="0.049024"
-    lower="${-TAU / 8}" upper="0" />
+                            x="0.034346" y="0" z="0.049024"
+                            lower="${-TAU / 8}" upper="0"/>
   <xacro:arm_revolute_joint parent="arm_b" child="arm_c"
-    x="0.534365" y="0" z="0.009056"
-    lower="0" upper="${TAU / 2}" />
+                            x="0.534365" y="0" z="0.009056"
+                            lower="0" upper="${TAU / 2}"/>
   <xacro:arm_revolute_joint parent="arm_c" child="arm_d"
-    x="0.546033" y="0" z="0.088594"
-    lower="0" upper="0" />
+                            x="0.546033" y="0" z="0.088594"
+                            lower="0" upper="0"/>
   <xacro:arm_revolute_joint parent="arm_d" child="arm_e"
-    x="0.044886" y="0" z="0"
-    lower="0" upper="0" />
-  <xacro:wheels side="left" reflect="1" />
-  <xacro:wheels side="right" reflect="-1" />
-  <!-- TODO(quintin): Add IMU -->
-  <!-- IMU -->
-  <!--  <joint name="imu_joint" type="fixed">-->
-  <!--    <origin xyz="0 0 0.2"/>-->
-  <!--    <parent link="chassis_link"/>-->
-  <!--    <child link="imu_link"/>-->
-  <!--  </joint>-->
-  <!--  <link name="imu_link"/>-->
+                            x="0.044886" y="0" z="0"
+                            lower="0" upper="0"/>
+  <xacro:wheels side="left" reflect="1"/>
+  <xacro:wheels side="right" reflect="-1"/>
+  <joint name="chassis_link_to_left_gps" type="fixed">
+    <origin xyz="0 0.1 0"/>
+    <parent link="chassis_link"/>
+    <child link="left_gps"/>
+  </joint>
+  <link name="left_gps"/>
+  <joint name="chassis_link_to_right_gps" type="fixed">
+    <origin xyz="0 -0.1 0"/>
+    <parent link="chassis_link"/>
+    <child link="right_gps"/>
+  </joint>
+  <link name="right_gps"/>
+  <joint name="chassis_link_to_imu" type="fixed">
+    <origin xyz="0 0 0"/>
+    <parent link="chassis_link"/>
+    <child link="imu"/>
+  </joint>
+  <link name="imu"/>
   <!-- TODO(quintin): Import the ZED URDF here -->
   <joint name="chassis_link_to_camera_link" type="fixed">
-    <origin xyz="0.3 0 0" />
-    <parent link="chassis_link" />
-    <child link="zed2i_left_camera_frame" />
+    <origin xyz="0.3 0 0"/>
+    <parent link="chassis_link"/>
+    <child link="zed2i_left_camera_frame"/>
   </joint>
   <link name="zed2i_left_camera_frame">
     <collision>
       <geometry>
-        <box size="0.01 0.1 0.01" />
+        <box size="0.01 0.1 0.01"/>
       </geometry>
     </collision>
